File: subsheet_100.sch (KiCad schematic (older format))
At the start: 23 parts, among them U15 ST_MMU_PHY, U22 74LS373_PHY, U23 74LS373_PHY, U26 74LS244_PHY, U27 74LS244_PHY

Commit message: reformat main sheet, start fixing directionnality of MMU signals
Changed lines of the file:
@@
 Sheet 2 2
 Title "Converted schematics of Atari 260/520 ST"
-Date "2022-07-08"
+Date "2022-07-10"
 Rev "0"
 Comp ""
-Comment1 "Original repository : ---"
-Comment2 "Reference : C070231"
-Comment3 ""
+Comment1 "…sporniket/kicad-conversions--atari-260-520-st-motherboard--c070231"
+Comment2 "Original repository : https://github.com/…"
+Comment3 "Reference : C070231"
 Comment4 ""
 $EndDescr
@@
 	1    0    0    -1
 $EndComp
-Text GLabel 1500 1000 2    50   BiDi ~ 0
+Text GLabel 1500 1000 2    50   Input ~ 0
 ADDR[1..23]
 Text Label 1250 1000 2    50   ~ 0
@@
 Wire Bus Line
 	5750 1000 6000 1000
-Text GLabel 4500 1000 2    50   BiDi ~ 0
+Text GLabel 4500 1000 2    50   Output ~ 0
 MADDR[0..8]
 Text Label 4250 1000 2    50   ~ 0
