File: subsheet_100.sch (KiCad schematic (older format))
At the start: 23 parts, among them U15 ST_MMU_PHY, U22 74LS373_PHY, U23 74LS373_PHY, U26 74LS244_PHY, U27 74LS244_PHY

Commit message: pcb session : placement ok, routing as much as possible
Parts:
- removed C?: 0.1uF, symbol Device:C_Small
- C16, C25, C29, C35: footprint (none) -> commons-passives_THT:Passive_THT_capacitor_mlcc_W2.54mm_L12.70mm
- L26, L28: footprint (none) -> commons-passives_THT:Passive_THT_ferrite_bead_W3.81mm_L15.24mm
- R118, R119, R120, R121, R122, R123, R124, R125, R126, R133, R134: footprint (none) -> commons-passives_THT:Passive_THT_resistor_W2.54mm_L12.70mm

Commit message: Schematics : shifter and video port
Changed lines of the file:
@@
 $Descr A4 8268 11693 portrait
 encoding utf-8
-Sheet 2 3
+Sheet 2 4
 Title "Converted schematics of Atari 260/520 ST"
-Date "2022-07-22"
+Date "2022-07-30"
 Rev "0"
 Comp ""
@@
 	1    0    0    -1
 $EndComp
-Text GLabel 1500 1000 2    50   Input ~ 0
+Text GLabel 1500 1000 0    50   Input ~ 0
 ADDR[1..23]
-Text Label 1250 1000 2    50   ~ 0
+Text Label 1750 1000 0    50   ~ 0
 A[1..23]
 Wire Bus Line
-	1250 1000 1500 1000
+	1750 1000 1500 1000
 Text GLabel 3000 1000 2    50   BiDi ~ 0
 DATA[0..15]
