File: motherboard.sch (KiCad schematic (older format))
At the start: 0 parts

Commit message: schematics : eproms and cartridge port
Other:
- note added: "Page 5"
Changed lines of the file:
@@
 $Descr A4 8268 11693 portrait
 encoding utf-8
-Sheet 1 4
+Sheet 1 5
 Title "Converted schematics of Atari 260/520 ST"
-Date "2022-09-08"
+Date "2022-10-20"
 Rev "0"
 Comp ""
@@
 Text Notes 6950 3150 0    50   ~ 0
 Page 4
+$Sheet
+S 1000 3450 6300 150
+U 6351BFF4
+F0 "U2-3-4-5-6-7-EPROMs ; J1-Cartridge port" 71
+F1 "subsheet_103.sch" 50
+$EndSheet
+Text Notes 6950 3550 0    50   ~ 0
+Page 5
 $EndSCHEMATC

Commit message: schematics : start adding U12 GLUE
Other:
- note added: "Page 6"
Changed lines of the file:
@@
 $Descr A4 8268 11693 portrait
 encoding utf-8
-Sheet 1 5
+Sheet 1 6
 Title "Converted schematics of Atari 260/520 ST"
-Date "2022-10-20"
+Date "2023-01-12"
 Rev "0"
 Comp ""
@@
 Text Notes 6950 3550 0    50   ~ 0
 Page 5
+$Sheet
+S 1000 3850 6300 150
+U 63C0E747
+F0 "U12-GLUE" 71
+F1 "subsheet_104.sch" 50
+$EndSheet
+Text Notes 6950 3950 0    50   ~ 0
+Page 6
 $EndSCHEMATC
