File: subsheet_101.sch (KiCad schematic (older format))
At the start: 34 parts, among them U16 DRAM_256K×1_PHY, U17 DRAM_256K×1_PHY, U18 DRAM_256K×1_PHY, U24 DRAM_256K×1_PHY, U25 DRAM_256K×1_PHY, U28 DRAM_256K×1_PHY, U29 DRAM_256K×1_PHY, U30 DRAM_256K×1_PHY, U32 DRAM_256K×1_PHY, U33 DRAM_256K×1_PHY, U34 DRAM_256K×1_PHY, U38 DRAM_256K×1_PHY, U42 DRAM_256K×1_PHY, U43 DRAM_256K×1_PHY, U44 DRAM_256K×1_PHY, U45 DRAM_256K×1_PHY

Commit message: subsheet 101 : assign footprints
Parts:
- C104: footprint (none) -> commons-passives_THT:Passive_THT_capacitor_polarized_W10.16mm_L30.48mm
- C26, C27, C28, C30, C36, C37, C38, C39, C41, C42, C44, C45, C57, C78, C79, C80: footprint (none) -> commons-passives_THT:Passive_THT_capacitor_mlcc_W2.54mm_L12.70mm
- L29: footprint (none) -> commons-passives_THT:Passive_THT_inductor_W5.08mm_L17.78mm

Commit message: Schematics : shifter and video port
Changed lines of the file:
@@
 $Descr A4 8268 11693 portrait
 encoding utf-8
-Sheet 3 3
+Sheet 3 4
 Title "Converted schematics of Atari 260/520 ST"
-Date "2022-07-22"
+Date "2022-07-30"
 Rev "0"
 Comp ""
@@
 Wire Bus Line
 	2500 10100 2750 10100
-Text GLabel 1250 10100 2    50   Input ~ 0
+Text GLabel 1250 10100 0    50   Input ~ 0
 MADDR[0..8]
-Text Label 1000 10100 2    50   ~ 0
+Text Label 1500 10100 0    50   ~ 0
 MAD[0..8]
 Wire Bus Line
-	1000 10100 1250 10100
+	1500 10100 1250 10100
 $Comp
 L power:+5V #PWR0112
