File: subsheet_102.sch (KiCad schematic (older format))
At the start: 54 parts, among them J6 DIN13S, Q2 2N3904, Q3 Q_NPN_CBE, Q4 2N3904, Q5 2N3904

Commit message: Added number to component still not numbered
Parts:
- gave numbers to parts that had none: 6
- renumbered JMOD to JMOD1
Changed lines of the file:
@@
 $EndDescr
 $Comp
-L st_shifter:ST_SHIFTER_PHY U?
+L st_shifter:ST_SHIFTER_PHY U31
 U 1 1 62E3A99D
 P 2350 3500
-F 0 "U?" H 1950 4750 50  0000 L TNN
+F 0 "U31" H 1950 4750 50  0000 L TNN
 F 1 "ST_SHIFTER_PHY" H 1950 4650 50  0000 L TNB
 F 2 "Package_DIP:DIP-40_W15.24mm_LongPads" H 1950 4850 50  0001 L TNN
@@
 P 2750 2250
 AR Path="/62C842FF/62EBBDFE" Ref="#PWR?"  Part="1"
-AR Path="/62E3A54E/62EBBDFE" Ref="#PWR?"  Part="1"
-F 0 "#PWR?" H 2750 2100 50  0001 C CNN
+AR Path="/62E3A54E/62EBBDFE" Ref="#PWR0171"  Part="1"
+F 0 "#PWR0171" H 2750 2100 50  0001 C CNN
 F 1 "+5V" H 2750 2390 50  0000 C CNN
 F 2 "" H 2750 2250 50  0001 C CNN
@@
 P 3800 2250
 AR Path="/62C842FF/62EC1DDC" Ref="#PWR?"  Part="1"
-AR Path="/62E3A54E/62EC1DDC" Ref="#PWR?"  Part="1"
-F 0 "#PWR?" H 3800 2000 50  0001 C CNN
+AR Path="/62E3A54E/62EC1DDC" Ref="#PWR0172"  Part="1"
+F 0 "#PWR0172" H 3800 2000 50  0001 C CNN
 F 1 "GND" H 3800 2100 50  0000 C CNN
 F 2 "" H 3800 2250 50  0001 C CNN
@@
 P 1400 4450
 AR Path="/62C842FF/62EC4233" Ref="#PWR?"  Part="1"
-AR Path="/62E3A54E/62EC4233" Ref="#PWR?"  Part="1"
-F 0 "#PWR?" H 1400 4200 50  0001 C CNN
+AR Path="/62E3A54E/62EC4233" Ref="#PWR0173"  Part="1"
+F 0 "#PWR0173" H 1400 4200 50  0001 C CNN
 F 1 "GND" H 1400 4300 50  0000 C CNN
 F 2 "" H 1400 4450 50  0001 C CNN
@@
 P 1000 2650
 AR Path="/62C842FF/62EC6521" Ref="#PWR?"  Part="1"
-AR Path="/62E3A54E/62EC6521" Ref="#PWR?"  Part="1"
-F 0 "#PWR?" H 1000 2400 50  0001 C CNN
+AR Path="/62E3A54E/62EC6521" Ref="#PWR0174"  Part="1"
+F 0 "#PWR0174" H 1000 2400 50  0001 C CNN
 F 1 "GND" H 1000 2500 50  0000 C CNN
 F 2 "" H 1000 2650 50  0001 C CNN
@@
 P 3950 3750
 AR Path="/62C842FF/62EDD1A8" Ref="#PWR?"  Part="1"
-AR Path="/62E3A54E/62EDD1A8" Ref="#PWR?"  Part="1"
-F 0 "#PWR?" H 3950 3600 50  0001 C CNN
+AR Path="/62E3A54E/62EDD1A8" Ref="#PWR0175"  Part="1"
+F 0 "#PWR0175" H 3950 3600 50  0001 C CNN
 F 1 "+5V" H 3950 3890 50  0000 C CNN
 F 2 "" H 3950 3750 50  0001 C CNN
@@
 P 3950 4050
 AR Path="/62C842FF/62EDE2D0" Ref="#PWR?"  Part="1"
-AR Path="/62E3A54E/62EDE2D0" Ref="#PWR?"  Part="1"
-F 0 "#PWR?" H 3950 3900 50  0001 C CNN
+AR Path="/62E3A54E/62EDE2D0" Ref="#PWR0176"  Part="1"
+F 0 "#PWR0176" H 3950 3900 50  0001 C CNN
 F 1 "+5V" H 3950 4190 50  0000 C CNN
 F 2 "" H 3950 4050 50  0001 C CNN
@@
 P 3950 4350
 AR Path="/62C842FF/62EE008D" Ref="#PWR?"  Part="1"
-AR Path="/62E3A54E/62EE008D" Ref="#PWR?"  Part="1"
-F 0 "#PWR?" H 3950 4200 50  0001 C CNN
+AR Path="/62E3A54E/62EE008D" Ref="#PWR0177"  Part="1"
+F 0 "#PWR0177" H 3950 4200 50  0001 C CNN
 F 1 "+5V" H 3950 4490 50  0000 C CNN
 F 2 "" H 3950 4350 50  0001 C CNN
@@
 P 6200 1750
 AR Path="/62C842FF/62F036E8" Ref="#PWR?"  Part="1"
-AR Path="/62E3A54E/62F036E8" Ref="#PWR?"  Part="1"
-F 0 "#PWR?" H 6200 1600 50  0001 C CNN
+AR Path="/62E3A54E/62F036E8" Ref="#PWR0178"  Part="1"
+F 0 "#PWR0178" H 6200 1600 50  0001 C CNN
 F 1 "+5V" H 6200 1890 50  0000 C CNN
 F 2 "" H 6200 1750 50  0001 C CNN
@@
 P 6500 1750
 AR Path="/62C842FF/62F036EE" Ref="L?"  Part="1"
-AR Path="/62E3A54E/62F036EE" Ref="L?"  Part="1"
-F 0 "L?" V 6450 1500 50  0000 L CNN
+AR Path="/62E3A54E/62F036EE" Ref="L17"  Part="1"
+F 0 "L17" V 6450 1550 50  0000 L CNN
 F 1 "Ferrite bead" V 6600 1500 50  0000 L CNN
 F 2 "commons-passives_THT:Passive_THT_ferrite_bead_W3.81mm_L15.24mm" V 6430 1750 50  0001 C CNN
@@
 P 7300 1750
 AR Path="/62C842FF/62F0B173" Ref="#PWR?"  Part="1"
-AR Path="/62E3A54E/62F0B173" Ref="#PWR?"  Part="1"
-F 0 "#PWR?" H 7300 1500 50  0001 C CNN
+AR Path="/62E3A54E/62F0B173" Ref="#PWR0179"  Part="1"
+F 0 "#PWR0179" H 7300 1500 50  0001 C CNN
 F 1 "GND" H 7300 1600 50  0000 C CNN
 F 2 "" H 7300 1750 50  0001 C CNN
@@
 P 5950 2350
 AR Path="/62C842FF/62F0F094" Ref="#PWR?"  Part="1"
-AR Path="/62E3A54E/62F0F094" Ref="#PWR?"  Part="1"
-F 0 "#PWR?" H 5950 2100 50  0001 C CNN
+AR Path="/62E3A54E/62F0F094" Ref="#PWR0180"  Part="1"
+F 0 "#PWR0180" H 5950 2100 50  0001 C CNN
 F 1 "GND" H 5950 2200 50  0000 C CNN
 F 2 "" H 5950 2350 50  0001 C CNN
@@
 P 4100 1000
 AR Path="/62C842FF/62F56006" Ref="#PWR?"  Part="1"
-AR Path="/62E3A54E/62F56006" Ref="#PWR?"  Part="1"
-F 0 "#PWR?" H 4100 850 50  0001 C CNN
+AR Path="/62E3A54E/62F56006" Ref="#PWR0181"  Part="1"
+F 0 "#PWR0181" H 4100 850 50  0001 C CNN
 F 1 "+5V" H 4100 1140 50  0000 C CNN
 F 2 "" H 4100 1000 50  0001 C CNN
@@
 P 5500 1000
 AR Path="/62C842FF/62F56026" Ref="#PWR?"  Part="1"
-AR Path="/62E3A54E/62F56026" Ref="#PWR?"  Part="1"
-F 0 "#PWR?" H 5500 750 50  0001 C CNN
+AR Path="/62E3A54E/62F56026" Ref="#PWR0182"  Part="1"
+F 0 "#PWR0182" H 5500 750 50  0001 C CNN
 F 1 "GND" H 5500 850 50  0000 C CNN
 F 2 "" H 5500 1000 50  0001 C CNN
@@
 P 5950 3300
 AR Path="/62C842FF/62F5603E" Ref="#PWR?"  Part="1"
-AR Path="/62E3A54E/62F5603E" Ref="#PWR?"  Part="1"
-F 0 "#PWR?" H 5950 3050 50  0001 C CNN
+AR Path="/62E3A54E/62F5603E" Ref="#PWR0183"  Part="1"
+F 0 "#PWR0183" H 5950 3050 50  0001 C CNN
 F 1 "GND" H 5950 3150 50  0000 C CNN
 F 2 "" H 5950 3300 50  0001 C CNN
@@
 	6300 2750 6300 3000
 $Comp
-L Device:D_Small CR?
+L Device:D_Small CR6
 U 1 1 62E453C3
 P 5900 3000
-F 0 "CR?" H 5950 2950 50  0000 L CNN
+F 0 "CR6" H 5950 2950 50  0000 L CNN
 F 1 "1N914" H 5600 2950 50  0000 L CNN
 F 2 "" V 5900 3000 50  0001 C CNN
@@
 P 5950 4250
 AR Path="/62C842FF/62E5A93B" Ref="#PWR?"  Part="1"
-AR Path="/62E3A54E/62E5A93B" Ref="#PWR?"  Part="1"
-F 0 "#PWR?" H 5950 4000 50  0001 C CNN
+AR Path="/62E3A54E/62E5A93B" Ref="#PWR0184"  Part="1"
+F 0 "#PWR0184" H 5950 4000 50  0001 C CNN
 F 1 "GND" H 5950 4100 50  0000 C CNN
 F 2 "" H 5950 4250 50  0001 C CNN
@@
 	6300 3700 6300 3950
 $Comp
-L Device:D_Small CR?
+L Device:D_Small CR5
 U 1 1 62E5A954
 P 5900 3950
-F 0 "CR?" H 5950 3900 50  0000 L CNN
+F 0 "CR5" H 5950 3900 50  0000 L CNN
 F 1 "1N914" H 5600 3900 50  0000 L CNN
 F 2 "" V 5900 3950 50  0001 C CNN
@@
 P 5950 5250
 AR Path="/62C842FF/62E634F9" Ref="#PWR?"  Part="1"
-AR Path="/62E3A54E/62E634F9" Ref="#PWR?"  Part="1"
-F 0 "#PWR?" H 5950 5000 50  0001 C CNN
+AR Path="/62E3A54E/62E634F9" Ref="#PWR0185"  Part="1"
+F 0 "#PWR0185" H 5950 5000 50  0001 C CNN
 F 1 "GND" H 5950 5100 50  0000 C CNN
 F 2 "" H 5950 5250 50  0001 C CNN
@@
 	6300 4700 6300 4950
 $Comp
-L Device:D_Small CR?
+L Device:D_Small CR4
 U 1 1 62E63512
 P 5900 4950
-F 0 "CR?" H 5950 4900 50  0000 L CNN
+F 0 "CR4" H 5950 4900 50  0000 L CNN
 F 1 "1N914" H 5600 4900 50  0000 L CNN
 F 2 "" V 5900 4950 50  0001 C CNN
@@
 P 7250 9700
 AR Path="/62C842FF/62EA7FD9" Ref="#PWR?"  Part="1"
-AR Path="/62E3A54E/62EA7FD9" Ref="#PWR?"  Part="1"
-F 0 "#PWR?" H 7250 9450 50  0001 C CNN
+AR Path="/62E3A54E/62EA7FD9" Ref="#PWR0186"  Part="1"
+F 0 "#PWR0186" H 7250 9450 50  0001 C CNN
 F 1 "GND" H 7250 9550 50  0000 C CNN
 F 2 "" H 7250 9700 50  0001 C CNN
@@
 	7250 9700 7250 9600
 $Comp
-L Connector_Generic_Shielded:Conn_01x10_Shielded JMOD
+L Connector_Generic_Shielded:Conn_01x10_Shielded JMOD1
 U 1 1 62EB0C08
 P 5250 6800
-F 0 "JMOD" H 5260 7290 50  0000 C CNN
+F 0 "JMOD1" H 5260 7290 50  0000 C CNN
 F 1 "Modulator" H 5290 6210 50  0000 L CNN
 F 2 "" H 5250 6800 50  0001 C CNN
@@
 P 5250 7600
 AR Path="/62C842FF/62EB1ADA" Ref="#PWR?"  Part="1"
-AR Path="/62E3A54E/62EB1ADA" Ref="#PWR?"  Part="1"
-F 0 "#PWR?" H 5250 7350 50  0001 C CNN
+AR Path="/62E3A54E/62EB1ADA" Ref="#PWR0187"  Part="1"
+F 0 "#PWR0187" H 5250 7350 50  0001 C CNN
 F 1 "GND" H 5250 7450 50  0000 C CNN
 F 2 "" H 5250 7600 50  0001 C CNN
@@
 HSYNC
 $Comp
-L power:+12V #PWR?
+L power:+12V #PWR0188
 U 1 1 62EBBFA5
 P 4250 6900
-F 0 "#PWR?" H 4250 6750 50  0001 C CNN
+F 0 "#PWR0188" H 4250 6750 50  0001 C CNN
 F 1 "+12V" H 4250 7040 50  0000 C CNN
 F 2 "" H 4250 6900 50  0001 C CNN
@@
 $EndComp
 $Comp
-L power:+5V #PWR?
+L power:+5V #PWR0189
 U 1 1 62EBC72E
 P 4000 6900
-F 0 "#PWR?" H 4000 6750 50  0001 C CNN
+F 0 "#PWR0189" H 4000 6750 50  0001 C CNN
 F 1 "+5V" H 4000 7040 50  0000 C CNN
 F 2 "" H 4000 6900 50  0001 C CNN
@@
 P 6350 9400
 AR Path="/62C842FF/62F38F2E" Ref="#PWR?"  Part="1"
-AR Path="/62E3A54E/62F38F2E" Ref="#PWR?"  Part="1"
-F 0 "#PWR?" H 6350 9150 50  0001 C CNN
+AR Path="/62E3A54E/62F38F2E" Ref="#PWR0190"  Part="1"
+F 0 "#PWR0190" H 6350 9150 50  0001 C CNN
 F 1 "GND" H 6350 9250 50  0000 C CNN
 F 2 "" H 6350 9400 50  0001 C CNN
@@
 HSYNC
 $Comp
-L power:+12V #PWR?
+L power:+12V #PWR0191
 U 1 1 62F39FC6
 P 6350 8900
-F 0 "#PWR?" H 6350 8750 50  0001 C CNN
+F 0 "#PWR0191" H 6350 8750 50  0001 C CNN
 F 1 "+12V" H 6350 9040 50  0000 C CNN
 F 2 "" H 6350 8900 50  0001 C CNN
@@
 $EndComp
 $Comp
-L Device:Q_NPN_CBE Q?
+L Device:Q_NPN_CBE Q10
 U 1 1 62E6E7AC
 P 2650 7950
-F 0 "Q?" H 2850 8000 50  0000 L CNN
+F 0 "Q10" H 2850 8000 50  0000 L CNN
 F 1 "2N3904" H 2850 7900 50  0000 L CNN
 F 2 "" H 2850 8050 50  0001 C CNN
@@
 P 2050 8300
 AR Path="/62C842FF/62EA08A6" Ref="#PWR?"  Part="1"
-AR Path="/62E3A54E/62EA08A6" Ref="#PWR?"  Part="1"
-F 0 "#PWR?" H 2050 8050 50  0001 C CNN
+AR Path="/62E3A54E/62EA08A6" Ref="#PWR0192"  Part="1"
+F 0 "#PWR0192" H 2050 8050 50  0001 C CNN
 F 1 "GND" H 2050 8150 50  0000 C CNN
 F 2 "" H 2050 8300 50  0001 C CNN
@@
 P 2750 7600
 AR Path="/62C842FF/6300D0A1" Ref="#PWR?"  Part="1"
-AR Path="/62E3A54E/6300D0A1" Ref="#PWR?"  Part="1"
-F 0 "#PWR?" H 2750 7450 50  0001 C CNN
+AR Path="/62E3A54E/6300D0A1" Ref="#PWR0193"  Part="1"
+F 0 "#PWR0193" H 2750 7450 50  0001 C CNN
 F 1 "+5V" H 2750 7740 50  0000 C CNN
 F 2 "" H 2750 7600 50  0001 C CNN

Commit message: Wired 'Vqq' together to remove label, add missing annotations, assigned footprints
Parts:
- CR1, CR10, CR2, CR3, CR4, CR5, CR6, CR9: footprint (none) -> commons-passives_THT:Passive_THT_diode_W2.54mm_L15.24mm
- J6: footprint (none) -> atari-interconnect:socket-din-13
- JMOD1: footprint (none) -> Connector_PinSocket_2.54mm:PinSocket_1x10_P2.54mm_Vertical
- Q10, Q2, Q4, Q5: footprint (none) -> Package_TO_SOT_THT:TO-92L_Inline_Wide
- Q3: value Q_NPN_CBE -> 2N3904; footprint (none) -> Package_TO_SOT_THT:TO-92L_Inline_Wide
- R115, R116, R117, R127, R129, R130, R131, R42, R43, R44, R45, R46, R47, R48, R49, R50, R51, R52, R53, R54, R55, R56, R57, R58, R59, R60, R61, R62, R63, R64, R66, R87: footprint (none) -> commons-passives_THT:Passive_THT_resistor_W2.54mm_L15.24mm
Connections:
- net Vqq: no longer names the net of C51.1, L18.2, Q3.1 (C), Q4.1 (C), Q5.1 (C), R48.2, R51.2, R66.2
Other:
- moved on the sheet: C40, C51, CR4, CR5, CR6, L17, L18, Q2, Q3, Q4, Q5, R115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
