File: subsheet_102.sch (KiCad schematic (older format))
At the start: 54 parts, among them J6 DIN13S, Q10 2N3904, Q2 2N3904, Q3 2N3904, Q4 2N3904, Q5 2N3904, U31 ST_SHIFTER_PHY

Commit message: changed footprints, symbol for transistor, modulator port without shield
Parts:
- JMOD1: footprint Connector_PinSocket_2.54mm:PinSocket_1x10_P2.54mm_Vertical -> Connector_PinHeader_2.54mm:PinHeader_1x10_P2.54mm_Vertical; symbol Connector_Generic_Shielded:Conn_01x10_Shielded -> Connector_Generic:Conn_01x10
- Q10, Q2, Q3, Q4, Q5: symbol Device:Q_NPN_CBE -> Device:Q_NPN_EBC
- R115, R116, R117, R127, R129, R130, R131, R42, R43, R44, R45, R46, R47, R48, R49, R50, R51, R52, R53, R54, R55, R56, R57, R58, R59, R60, R61, R62, R63, R64, R66, R87: footprint commons-passives_THT:Passive_THT_resistor_W2.54mm_L15.24mm -> commons-passives_THT:Passive_THT_resistor_W2.54mm_L12.70mm
Connections:
- net +5V: now also Q10.3 (C); no longer Q10.1 (C)
- net GND: no longer JMOD1.SH (Shield)
- net blue_mod: now also Q3.1 (E); no longer Q3.3 (E)
- net green_mod: now also Q4.1 (E); no longer Q4.3 (E)
- net red_mod: now also Q5.1 (E); no longer Q5.3 (E)
- net at C51.1, L18.2, R48.2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: now also Q3.3 (C), Q4.3 (C), Q5.3 (C); no longer Q3.1 (C), Q4.1 (C), Q5.1 (C)
- net at R130.2, R131.1: now also Q10.1 (E); no longer Q10.3 (E)
- net at C40.1, L17.1: now also Q2.3 (C); no longer Q2.1 (C)
- net at R42.1, R43.2: now also Q2.1 (E); no longer Q2.3 (E)

Commit message: pcb session -- 2022-09-09T05:25:13+02:00
Parts:
- CR1, CR10, CR2, CR3, CR4, CR5, CR6, CR9: footprint commons-passives_THT:Passive_THT_diode_W2.54mm_L15.24mm -> commons-passives_THT:Passive_THT_diode_W2.54mm_L12.70mm
- L18: footprint commons-passives_THT:Passive_THT_inductor_W5.08mm_L17.78mm -> commons-passives_THT:Passive_THT_inductor_W5.08mm_L15.24mm
Changed lines of the file:
@@
 F 0 "CR1" H 4950 3800 50  0000 L CNN
 F 1 "1N914" H 4600 3800 50  0000 L CNN
-F 2 "commons-passives_THT:Passive_THT_diode_W2.54mm_L15.24mm" V 4900 3750 50  0001 C CNN
+F 2 "commons-passives_THT:Passive_THT_diode_W2.54mm_L12.70mm" V 4900 3750 50  0001 C CNN
 F 3 "~" V 4900 3750 50  0001 C CNN
 	1    4900 3750
@@
 F 0 "CR2" H 4950 4100 50  0000 L CNN
 F 1 "1N914" H 4600 4100 50  0000 L CNN
-F 2 "commons-passives_THT:Passive_THT_diode_W2.54mm_L15.24mm" V 4900 4050 50  0001 C CNN
+F 2 "commons-passives_THT:Passive_THT_diode_W2.54mm_L12.70mm" V 4900 4050 50  0001 C CNN
 F 3 "~" V 4900 4050 50  0001 C CNN
 	1    4900 4050
@@
 F 0 "CR3" H 4950 4400 50  0000 L CNN
 F 1 "1N914" H 4600 4400 50  0000 L CNN
-F 2 "commons-passives_THT:Passive_THT_diode_W2.54mm_L15.24mm" V 4900 4350 50  0001 C CNN
+F 2 "commons-passives_THT:Passive_THT_diode_W2.54mm_L12.70mm" V 4900 4350 50  0001 C CNN
 F 3 "~" V 4900 4350 50  0001 C CNN
 	1    4900 4350
@@
 F 0 "CR6" H 5700 2950 50  0000 L CNN
 F 1 "1N914" H 5350 2950 50  0000 L CNN
-F 2 "commons-passives_THT:Passive_THT_diode_W2.54mm_L15.24mm" V 5650 3000 50  0001 C CNN
+F 2 "commons-passives_THT:Passive_THT_diode_W2.54mm_L12.70mm" V 5650 3000 50  0001 C CNN
 F 3 "~" V 5650 3000 50  0001 C CNN
 	1    5650 3000
@@
 F 0 "CR5" H 5700 3900 50  0000 L CNN
 F 1 "1N914" H 5350 3900 50  0000 L CNN
-F 2 "commons-passives_THT:Passive_THT_diode_W2.54mm_L15.24mm" V 5650 3950 50  0001 C CNN
+F 2 "commons-passives_THT:Passive_THT_diode_W2.54mm_L12.70mm" V 5650 3950 50  0001 C CNN
 F 3 "~" V 5650 3950 50  0001 C CNN
 	1    5650 3950
@@
 F 0 "CR4" H 5700 4900 50  0000 L CNN
 F 1 "1N914" H 5350 4900 50  0000 L CNN
-F 2 "commons-passives_THT:Passive_THT_diode_W2.54mm_L15.24mm" V 5650 4950 50  0001 C CNN
+F 2 "commons-passives_THT:Passive_THT_diode_W2.54mm_L12.70mm" V 5650 4950 50  0001 C CNN
 F 3 "~" V 5650 4950 50  0001 C CNN
 	1    5650 4950
@@
 F 0 "CR9" H 1450 7850 50  0000 L CNN
 F 1 "1N914" H 1750 7850 50  0000 L CNN
-F 2 "commons-passives_THT:Passive_THT_diode_W2.54mm_L15.24mm" V 1700 7800 50  0001 C CNN
+F 2 "commons-passives_THT:Passive_THT_diode_W2.54mm_L12.70mm" V 1700 7800 50  0001 C CNN
 F 3 "~" V 1700 7800 50  0001 C CNN
 	1    1700 7800
@@
 F 0 "CR10" H 1450 8000 50  0000 L CNN
 F 1 "1N914" H 1750 8000 50  0000 L CNN
-F 2 "commons-passives_THT:Passive_THT_diode_W2.54mm_L15.24mm" V 1700 7950 50  0001 C CNN
+F 2 "commons-passives_THT:Passive_THT_diode_W2.54mm_L12.70mm" V 1700 7950 50  0001 C CNN
 F 3 "~" V 1700 7950 50  0001 C CNN
 	1    1700 7950
@@
 F 0 "L18" H 7200 1300 50  0000 R CNN
 F 1 "0.27uH" H 7200 1200 50  0000 R CNN
-F 2 "commons-passives_THT:Passive_THT_inductor_W5.08mm_L17.78mm" H 7250 1250 50  0001 C CNN
+F 2 "commons-passives_THT:Passive_THT_inductor_W5.08mm_L15.24mm" H 7250 1250 50  0001 C CNN
 F 3 "~" H 7250 1250 50  0001 C CNN
 	1    7250 1250
