File: subsheet_103.sch (KiCad schematic (older format))
At the start: 15 parts, among them J1 Cartridge port, U2 27C512_PHY, U3 27C512_PHY, U4 27C512_PHY, U5 27C512_PHY, U6 27C512_PHY, U7 27C512_PHY

Commit message: eproms, cartridge port : footprints, update pcb, start placing
Parts:
- J1: footprint (none) -> atari-interconnect:socket-edge-pcb_40p_P2.01mm_no_post
Changed lines of the file:
@@
 P 3400 2000
 AR Path="/62C842FF/63555EE3" Ref="#PWR?"  Part="1"
-AR Path="/6351BFF4/63555EE3" Ref="#PWR?"  Part="1"
-F 0 "#PWR?" H 3400 1750 50  0001 C CNN
+AR Path="/6351BFF4/63555EE3" Ref="#PWR0187"  Part="1"
+F 0 "#PWR0187" H 3400 1750 50  0001 C CNN
 F 1 "GND" H 3400 1850 50  0000 C CNN
 F 2 "" H 3400 2000 50  0001 C CNN
@@
 P 2750 2000
 AR Path="/62C842FF/63557F06" Ref="#PWR?"  Part="1"
-AR Path="/6351BFF4/63557F06" Ref="#PWR?"  Part="1"
-F 0 "#PWR?" H 2750 1850 50  0001 C CNN
+AR Path="/6351BFF4/63557F06" Ref="#PWR0194"  Part="1"
+F 0 "#PWR0194" H 2750 1850 50  0001 C CNN
 F 1 "+5V" H 2750 2140 50  0000 C CNN
 F 2 "" H 2750 2000 50  0001 C CNN
@@
 P 750 3300
 AR Path="/62C842FF/6355972C" Ref="#PWR?"  Part="1"
-AR Path="/6351BFF4/6355972C" Ref="#PWR?"  Part="1"
-F 0 "#PWR?" H 750 3050 50  0001 C CNN
+AR Path="/6351BFF4/6355972C" Ref="#PWR0195"  Part="1"
+F 0 "#PWR0195" H 750 3050 50  0001 C CNN
 F 1 "GND" H 750 3150 50  0000 C CNN
 F 2 "" H 750 3300 50  0001 C CNN
@@
 P 750 2000
 AR Path="/62C842FF/63559BE9" Ref="#PWR?"  Part="1"
-AR Path="/6351BFF4/63559BE9" Ref="#PWR?"  Part="1"
-F 0 "#PWR?" H 750 1850 50  0001 C CNN
+AR Path="/6351BFF4/63559BE9" Ref="#PWR0196"  Part="1"
+F 0 "#PWR0196" H 750 1850 50  0001 C CNN
 F 1 "+5V" H 750 2140 50  0000 C CNN
 F 2 "" H 750 2000 50  0001 C CNN
@@
 P 3400 4000
 AR Path="/62C842FF/63563CFB" Ref="#PWR?"  Part="1"
-AR Path="/6351BFF4/63563CFB" Ref="#PWR?"  Part="1"
-F 0 "#PWR?" H 3400 3750 50  0001 C CNN
+AR Path="/6351BFF4/63563CFB" Ref="#PWR0197"  Part="1"
+F 0 "#PWR0197" H 3400 3750 50  0001 C CNN
 F 1 "GND" H 3400 3850 50  0000 C CNN
 F 2 "" H 3400 4000 50  0001 C CNN
@@
 P 2750 4000
 AR Path="/62C842FF/63563D01" Ref="#PWR?"  Part="1"
-AR Path="/6351BFF4/63563D01" Ref="#PWR?"  Part="1"
-F 0 "#PWR?" H 2750 3850 50  0001 C CNN
+AR Path="/6351BFF4/63563D01" Ref="#PWR0198"  Part="1"
+F 0 "#PWR0198" H 2750 3850 50  0001 C CNN
 F 1 "+5V" H 2750 4140 50  0000 C CNN
 F 2 "" H 2750 4000 50  0001 C CNN
@@
 P 750 5300
 AR Path="/62C842FF/63563D07" Ref="#PWR?"  Part="1"
-AR Path="/6351BFF4/63563D07" Ref="#PWR?"  Part="1"
-F 0 "#PWR?" H 750 5050 50  0001 C CNN
+AR Path="/6351BFF4/63563D07" Ref="#PWR0199"  Part="1"
+F 0 "#PWR0199" H 750 5050 50  0001 C CNN
 F 1 "GND" H 750 5150 50  0000 C CNN
 F 2 "" H 750 5300 50  0001 C CNN
@@
 P 750 4000
 AR Path="/62C842FF/63563D0D" Ref="#PWR?"  Part="1"
-AR Path="/6351BFF4/63563D0D" Ref="#PWR?"  Part="1"
-F 0 "#PWR?" H 750 3850 50  0001 C CNN
+AR Path="/6351BFF4/63563D0D" Ref="#PWR0200"  Part="1"
+F 0 "#PWR0200" H 750 3850 50  0001 C CNN
 F 1 "+5V" H 750 4140 50  0000 C CNN
 F 2 "" H 750 4000 50  0001 C CNN
@@
 P 3400 6000
 AR Path="/62C842FF/6356E8C4" Ref="#PWR?"  Part="1"
-AR Path="/6351BFF4/6356E8C4" Ref="#PWR?"  Part="1"
-F 0 "#PWR?" H 3400 5750 50  0001 C CNN
+AR Path="/6351BFF4/6356E8C4" Ref="#PWR0201"  Part="1"
+F 0 "#PWR0201" H 3400 5750 50  0001 C CNN
 F 1 "GND" H 3400 5850 50  0000 C CNN
 F 2 "" H 3400 6000 50  0001 C CNN
@@
 P 2750 6000
 AR Path="/62C842FF/6356E8CA" Ref="#PWR?"  Part="1"
-AR Path="/6351BFF4/6356E8CA" Ref="#PWR?"  Part="1"
-F 0 "#PWR?" H 2750 5850 50  0001 C CNN
+AR Path="/6351BFF4/6356E8CA" Ref="#PWR0202"  Part="1"
+F 0 "#PWR0202" H 2750 5850 50  0001 C CNN
 F 1 "+5V" H 2750 6140 50  0000 C CNN
 F 2 "" H 2750 6000 50  0001 C CNN
@@
 P 750 7300
 AR Path="/62C842FF/6356E8D0" Ref="#PWR?"  Part="1"
-AR Path="/6351BFF4/6356E8D0" Ref="#PWR?"  Part="1"
-F 0 "#PWR?" H 750 7050 50  0001 C CNN
+AR Path="/6351BFF4/6356E8D0" Ref="#PWR0203"  Part="1"
+F 0 "#PWR0203" H 750 7050 50  0001 C CNN
 F 1 "GND" H 750 7150 50  0000 C CNN
 F 2 "" H 750 7300 50  0001 C CNN
@@
 P 750 6000
 AR Path="/62C842FF/6356E8D6" Ref="#PWR?"  Part="1"
-AR Path="/6351BFF4/6356E8D6" Ref="#PWR?"  Part="1"
-F 0 "#PWR?" H 750 5850 50  0001 C CNN
+AR Path="/6351BFF4/6356E8D6" Ref="#PWR0204"  Part="1"
+F 0 "#PWR0204" H 750 5850 50  0001 C CNN
 F 1 "+5V" H 750 6140 50  0000 C CNN
 F 2 "" H 750 6000 50  0001 C CNN
@@
 P 6400 2000
 AR Path="/62C842FF/6358419D" Ref="#PWR?"  Part="1"
-AR Path="/6351BFF4/6358419D" Ref="#PWR?"  Part="1"
-F 0 "#PWR?" H 6400 1750 50  0001 C CNN
+AR Path="/6351BFF4/6358419D" Ref="#PWR0205"  Part="1"
+F 0 "#PWR0205" H 6400 1750 50  0001 C CNN
 F 1 "GND" H 6400 1850 50  0000 C CNN
 F 2 "" H 6400 2000 50  0001 C CNN
@@
 P 5750 2000
 AR Path="/62C842FF/635841A3" Ref="#PWR?"  Part="1"
-AR Path="/6351BFF4/635841A3" Ref="#PWR?"  Part="1"
-F 0 "#PWR?" H 5750 1850 50  0001 C CNN
+AR Path="/6351BFF4/635841A3" Ref="#PWR0206"  Part="1"
+F 0 "#PWR0206" H 5750 1850 50  0001 C CNN
 F 1 "+5V" H 5750 2140 50  0000 C CNN
 F 2 "" H 5750 2000 50  0001 C CNN
@@
 P 3750 3300
 AR Path="/62C842FF/635841A9" Ref="#PWR?"  Part="1"
-AR Path="/6351BFF4/635841A9" Ref="#PWR?"  Part="1"
-F 0 "#PWR?" H 3750 3050 50  0001 C CNN
+AR Path="/6351BFF4/635841A9" Ref="#PWR0207"  Part="1"
+F 0 "#PWR0207" H 3750 3050 50  0001 C CNN
 F 1 "GND" H 3750 3150 50  0000 C CNN
 F 2 "" H 3750 3300 50  0001 C CNN
@@
 P 3750 2000
 AR Path="/62C842FF/635841AF" Ref="#PWR?"  Part="1"
-AR Path="/6351BFF4/635841AF" Ref="#PWR?"  Part="1"
-F 0 "#PWR?" H 3750 1850 50  0001 C CNN
+AR Path="/6351BFF4/635841AF" Ref="#PWR0208"  Part="1"
+F 0 "#PWR0208" H 3750 1850 50  0001 C CNN
 F 1 "+5V" H 3750 2140 50  0000 C CNN
 F 2 "" H 3750 2000 50  0001 C CNN
@@
 P 6400 4000
 AR Path="/62C842FF/635841F9" Ref="#PWR?"  Part="1"
-AR Path="/6351BFF4/635841F9" Ref="#PWR?"  Part="1"
-F 0 "#PWR?" H 6400 3750 50  0001 C CNN
+AR Path="/6351BFF4/635841F9" Ref="#PWR0209"  Part="1"
+F 0 "#PWR0209" H 6400 3750 50  0001 C CNN
 F 1 "GND" H 6400 3850 50  0000 C CNN
 F 2 "" H 6400 4000 50  0001 C CNN
@@
 P 5750 4000
 AR Path="/62C842FF/635841FF" Ref="#PWR?"  Part="1"
-AR Path="/6351BFF4/635841FF" Ref="#PWR?"  Part="1"
-F 0 "#PWR?" H 5750 3850 50  0001 C CNN
+AR Path="/6351BFF4/635841FF" Ref="#PWR0210"  Part="1"
+F 0 "#PWR0210" H 5750 3850 50  0001 C CNN
 F 1 "+5V" H 5750 4140 50  0000 C CNN
 F 2 "" H 5750 4000 50  0001 C CNN
@@
 P 3750 5300
 AR Path="/62C842FF/63584205" Ref="#PWR?"  Part="1"
-AR Path="/6351BFF4/63584205" Ref="#PWR?"  Part="1"
-F 0 "#PWR?" H 3750 5050 50  0001 C CNN
+AR Path="/6351BFF4/63584205" Ref="#PWR0211"  Part="1"
+F 0 "#PWR0211" H 3750 5050 50  0001 C CNN
 F 1 "GND" H 3750 5150 50  0000 C CNN
 F 2 "" H 3750 5300 50  0001 C CNN
@@
 P 3750 4000
 AR Path="/62C842FF/6358420B" Ref="#PWR?"  Part="1"
-AR Path="/6351BFF4/6358420B" Ref="#PWR?"  Part="1"
-F 0 "#PWR?" H 3750 3850 50  0001 C CNN
+AR Path="/6351BFF4/6358420B" Ref="#PWR0212"  Part="1"
+F 0 "#PWR0212" H 3750 3850 50  0001 C CNN
 F 1 "+5V" H 3750 4140 50  0000 C CNN
 F 2 "" H 3750 4000 50  0001 C CNN
@@
 P 6400 6000
 AR Path="/62C842FF/63584255" Ref="#PWR?"  Part="1"
-AR Path="/6351BFF4/63584255" Ref="#PWR?"  Part="1"
-F 0 "#PWR?" H 6400 5750 50  0001 C CNN
+AR Path="/6351BFF4/63584255" Ref="#PWR0213"  Part="1"
+F 0 "#PWR0213" H 6400 5750 50  0001 C CNN
 F 1 "GND" H 6400 5850 50  0000 C CNN
 F 2 "" H 6400 6000 50  0001 C CNN
@@
 P 5750 6000
 AR Path="/62C842FF/6358425B" Ref="#PWR?"  Part="1"
-AR Path="/6351BFF4/6358425B" Ref="#PWR?"  Part="1"
-F 0 "#PWR?" H 5750 5850 50  0001 C CNN
+AR Path="/6351BFF4/6358425B" Ref="#PWR0214"  Part="1"
+F 0 "#PWR0214" H 5750 5850 50  0001 C CNN
 F 1 "+5V" H 5750 6140 50  0000 C CNN
 F 2 "" H 5750 6000 50  0001 C CNN
@@
 P 3750 7300
 AR Path="/62C842FF/63584261" Ref="#PWR?"  Part="1"
-AR Path="/6351BFF4/63584261" Ref="#PWR?"  Part="1"
-F 0 "#PWR?" H 3750 7050 50  0001 C CNN
+AR Path="/6351BFF4/63584261" Ref="#PWR0215"  Part="1"
+F 0 "#PWR0215" H 3750 7050 50  0001 C CNN
 F 1 "GND" H 3750 7150 50  0000 C CNN
 F 2 "" H 3750 7300 50  0001 C CNN
@@
 P 3750 6000
 AR Path="/62C842FF/63584267" Ref="#PWR?"  Part="1"
-AR Path="/6351BFF4/63584267" Ref="#PWR?"  Part="1"
-F 0 "#PWR?" H 3750 5850 50  0001 C CNN
+AR Path="/6351BFF4/63584267" Ref="#PWR0216"  Part="1"
+F 0 "#PWR0216" H 3750 5850 50  0001 C CNN
 F 1 "+5V" H 3750 6140 50  0000 C CNN
 F 2 "" H 3750 6000 50  0001 C CNN
@@
 F 0 "J1" H 7400 9500 50  0000 C CNN
 F 1 "Cartridge port" H 7400 5400 50  0000 C CNN
-F 2 "" H 7400 7500 50  0001 C CNN
+F 2 "atari-interconnect:socket-edge-pcb_40p_P2.01mm_no_post" H 7400 7500 50  0001 C CNN
 F 3 "~" H 7400 7500 50  0001 C CNN
 	1    7400 7500
@@
 P 6350 5200
 AR Path="/62C842FF/636D797A" Ref="#PWR?"  Part="1"
-AR Path="/6351BFF4/636D797A" Ref="#PWR?"  Part="1"
-F 0 "#PWR?" H 6350 5050 50  0001 C CNN
+AR Path="/6351BFF4/636D797A" Ref="#PWR0217"  Part="1"
+F 0 "#PWR0217" H 6350 5050 50  0001 C CNN
 F 1 "+5V" H 6350 5340 50  0000 C CNN
 F 2 "" H 6350 5200 50  0001 C CNN
@@
 P 7550 5200
 AR Path="/62C842FF/636E6B80" Ref="#PWR?"  Part="1"
-AR Path="/6351BFF4/636E6B80" Ref="#PWR?"  Part="1"
-F 0 "#PWR?" H 7550 4950 50  0001 C CNN
+AR Path="/6351BFF4/636E6B80" Ref="#PWR0218"  Part="1"
+F 0 "#PWR0218" H 7550 4950 50  0001 C CNN
 F 1 "GND" H 7550 5050 50  0000 C CNN
 F 2 "" H 7550 5200 50  0001 C CNN
@@
 P 6800 9500
 AR Path="/62C842FF/63C14E0D" Ref="#PWR?"  Part="1"
-AR Path="/6351BFF4/63C14E0D" Ref="#PWR?"  Part="1"
-F 0 "#PWR?" H 6800 9250 50  0001 C CNN
+AR Path="/6351BFF4/63C14E0D" Ref="#PWR0219"  Part="1"
+F 0 "#PWR0219" H 6800 9250 50  0001 C CNN
 F 1 "GND" H 6800 9350 50  0000 C CNN
 F 2 "" H 6800 9500 50  0001 C CNN
