File: subsheet_104.kicad_sch (KiCad schematic)
At the start: 1 part

Commit message: schematics : done U12-GLUE
Parts:
- added C13: 0.1uF, commons-passives_THT:Passive_THT_capacitor_mlcc_W2.54mm_L12.70mm, symbol Device:C_Small
- added R5: 1K, symbol Device:R_Small_US
Connections:
- net A1: now also U?.56 (A1); no longer U?.60 (A5)
- net A2: now also U?.57 (A2); no longer U?.59 (A4)
- net A4: now also U?.59 (A4); no longer U?.57 (A2)
- net A5: now also U?.60 (A5); no longer U?.56 (A1)
- net +5V: now reaches U?.1 (VCC)
- net +5V: now also C13.1, R5.2
- net XAS: now reaches U?.12 (~{AS})
- net FC2: now reaches U?.13 (FC2)
- net FC1: now reaches U?.14 (FC1)
- net FC0: now reaches U?.15 (FC0)
- net XVMA: now reaches U?.16 (~{VMA})
- net ROM4: now reaches U?.17 (~{ROM4})
- net ROM3: now reaches U?.18 (~{ROM3})
- net ROM2: now reaches U?.19 (~{ROM2})
- net ROM1: now reaches U?.20 (~{ROM1})
- net ROM0: now reaches U?.21 (~{ROM0})
- net XRESET: now reaches U?.22 (~{RESET})
- net XRAM: now reaches U?.23 (~{RAM})
- net XDMA: now reaches U?.24 (~{DMA})
- net XDEV: now reaches U?.25 (~{DEV})
- net XFCS: now reaches U?.26 (~{FCS})
- net XBG: now reaches U?.27 (~{BGI})
- net XRDY: now reaches U?.28 (RDY)
- net XRDY: now also R5.1
- net XVPA: now reaches U?.29 (~{VPA})
- net XBERR: now reaches U?.30 (~{BERR})
- net XDTACK: now reaches U?.31 (~{DTACK})
- net IPL1: now reaches U?.32 (~{IPL1})
- net IPL2: now reaches U?.33 (~{IPL2})
- net 8MHZ: now reaches U?.34 (8MHZ)
- net GND: now reaches U?.35 (GND)
- net GND: now also U?.52 (GND), C13.2
- net BLANK: now reaches U?.36 (~{BLANK})
- net HSYNC: now reaches U?.37 (HSYNC)
- net VSYNC: now reaches U?.38 (VSYNC)
- net DE: now reaches U?.39 (DE)
- net XBR: now reaches U?.40 (~{BR})
- net XBGACK: now reaches U?.41 (~{BGACK})
- net N6850: now reaches U?.42 (6850CS)
- net KHZ500: now reaches U?.43 (500KHZ)
- net XMFPINT: now reaches U?.44 (~{MFPINT})
- net XLDS: now reaches U?.46 (~{LDS})
- net XUDS: now reaches U?.47 (~{UDS})
- net XIACK: now reaches U?.50 (~{IACK})
- net XMFPCS: now reaches U?.51 (~{MFPCS})
- net SNDCS: now reaches U?.53 (~{SNDCS})
- net 2MHZ: now reaches U?.54 (2MHZ)
- net XRXW: now reaches U?.55 (R/~{W})

Commit message: pcb session 2023-01-17T19:16:31+01:00
Parts:
- R5: footprint (none) -> commons-passives_THT:Passive_THT_resistor_W2.54mm_L12.70mm
- gave numbers to parts that had none: 1
Changed lines of the file:
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@@
   (symbol (lib_id "st_glue:ST_GLUE_PHY") (at 101.6 114.3 0) (unit 1)
     (in_bom yes) (on_board yes)
-    (property "Reference" "U?" (id 0) (at 124.46 77.47 0)
+    (property "Reference" "U12" (id 0) (at 124.46 77.47 0)
       (effects (font (size 1.27 1.27)) (justify left top))
     )
@@
   (symbol (lib_id "power:+5V") (at 101.6 50.8 0) (unit 1)
     (in_bom yes) (on_board yes)
-    (property "Reference" "#PWR?" (id 0) (at 101.6 54.61 0)
+    (property "Reference" "#PWR0221" (id 0) (at 101.6 54.61 0)
       (effects (font (size 1.27 1.27)) hide)
     )
@@
   (symbol (lib_id "power:+5V") (at 68.58 176.53 0) (unit 1)
     (in_bom yes) (on_board yes)
-    (property "Reference" "#PWR?" (id 0) (at 68.58 180.34 0)
+    (property "Reference" "#PWR0224" (id 0) (at 68.58 180.34 0)
       (effects (font (size 1.27 1.27)) hide)
     )
@@
     (property "Reference" "R5" (id 0) (at 76.2 173.99 90))
     (property "Value" "1K" (id 1) (at 76.2 179.07 90))
-    (property "Footprint" "" (id 2) (at 76.2 176.53 0)
+    (property "Footprint" "commons-passives_THT:Passive_THT_resistor_W2.54mm_L12.70mm" (id 2) (at 76.2 176.53 0)
       (effects (font (size 1.27 1.27)) hide)
     )
@@
   (symbol (lib_id "power:GND") (at 173.99 113.03 0) (unit 1)
     (in_bom yes) (on_board yes)
-    (property "Reference" "#PWR?" (id 0) (at 173.99 119.38 0)
+    (property "Reference" "#PWR0220" (id 0) (at 173.99 119.38 0)
       (effects (font (size 1.27 1.27)) hide)
     )
@@
   (symbol (lib_id "power:GND") (at 116.84 55.88 0) (unit 1)
     (in_bom yes) (on_board yes)
-    (property "Reference" "#PWR?" (id 0) (at 116.84 62.23 0)
+    (property "Reference" "#PWR0222" (id 0) (at 116.84 62.23 0)
       (effects (font (size 1.27 1.27)) hide)
     )
@@
   (symbol (lib_id "power:GND") (at 101.6 156.21 0) (unit 1)
     (in_bom yes) (on_board yes)
-    (property "Reference" "#PWR?" (id 0) (at 101.6 162.56 0)
+    (property "Reference" "#PWR0223" (id 0) (at 101.6 162.56 0)
       (effects (font (size 1.27 1.27)) hide)
     )
