File: subsheet_104.kicad_sch (KiCad schematic)
At the start: 29 parts, among them J2 DB19S ACSI, J3 Floppy disk, U1 ST_DMA_DIP40_PHY, U8 7406 HEX INVERTER, U9 WD1772_FLOPPY_DISK_CONTROLLER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

Commit message: assigning footprints
Parts:
- J2: footprint (none) -> atari-interconnect:DSUB-19_Female_Horizontal_P2.77x2.84mm_EdgePinOffset7.70mm_Housed_MountingHolesOffset9.12mm
- J3: footprint (none) -> atari-interconnect:socket-din-14
Changed lines of the file:
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@@
       (effects (font (size 1.27 1.27)) (justify left))
     )
-    (property "Footprint" "" (id 2) (at 177.8 185.42 0)
+    (property "Footprint" "atari-interconnect:socket-din-14" (id 2) (at 177.8 185.42 0)
       (effects (font (size 1.27 1.27)) hide)
     )
@@
       (effects (font (size 1.27 1.27)) (justify left))
     )
-    (property "Footprint" "" (id 2) (at 172.72 73.66 0)
-      (effects (font (size 1.27 1.27)) hide)
-    )
+    (property "Footprint" "atari-interconnect:DSUB-19_Female_Horizontal_P2.77x2.84mm_EdgePinOffset7.70mm_Housed_MountingHolesOffset9.12mm" (id 2) (at 172.72 73.66 0)
+      (effects (font (size 1.27 1.27)) hide)
+    )
