File: subsheet_104.kicad_sch (KiCad schematic)
At the start: 29 parts, among them J2 DB19S ACSI, J3 Floppy disk, U1 ST_DMA_DIP40_PHY, U8 7406 HEX INVERTER, U9 WD1772_FLOPPY_DISK_CONTROLLER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

Commit message: assign footprints of remaining Resistors
Parts:
- R100, R101, R102, R103, R13, R14, R15, R16: footprint (none) -> commons-passives_THT:Passive_THT_resistor_W2.54mm_L12.70mm
Changed lines of the file:
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@@
       (effects (font (size 1.27 1.27)) (justify left))
     )
-    (property "Footprint" "" (id 2) (at 96.52 149.86 0)
+    (property "Footprint" "commons-passives_THT:Passive_THT_resistor_W2.54mm_L12.70mm" (id 2) (at 96.52 149.86 0)
       (effects (font (size 1.27 1.27)) hide)
     )
@@
       (effects (font (size 1.27 1.27)) (justify left))
     )
-    (property "Footprint" "" (id 2) (at 111.76 200.66 0)
+    (property "Footprint" "commons-passives_THT:Passive_THT_resistor_W2.54mm_L12.70mm" (id 2) (at 111.76 200.66 0)
       (effects (font (size 1.27 1.27)) hide)
     )
@@
       (effects (font (size 1.27 1.27)) (justify left))
     )
-    (property "Footprint" "" (id 2) (at 99.06 241.3 0)
+    (property "Footprint" "commons-passives_THT:Passive_THT_resistor_W2.54mm_L12.70mm" (id 2) (at 99.06 241.3 0)
       (effects (font (size 1.27 1.27)) hide)
     )
@@
       (effects (font (size 1.27 1.27)) (justify left))
     )
-    (property "Footprint" "" (id 2) (at 95.25 85.09 0)
+    (property "Footprint" "commons-passives_THT:Passive_THT_resistor_W2.54mm_L12.70mm" (id 2) (at 95.25 85.09 0)
       (effects (font (size 1.27 1.27)) hide)
     )
@@
       (effects (font (size 1.27 1.27)) (justify left))
     )
-    (property "Footprint" "" (id 2) (at 99.06 231.14 0)
+    (property "Footprint" "commons-passives_THT:Passive_THT_resistor_W2.54mm_L12.70mm" (id 2) (at 99.06 231.14 0)
       (effects (font (size 1.27 1.27)) hide)
     )
@@
       (effects (font (size 1.27 1.27)) (justify left))
     )
-    (property "Footprint" "" (id 2) (at 111.76 210.82 0)
+    (property "Footprint" "commons-passives_THT:Passive_THT_resistor_W2.54mm_L12.70mm" (id 2) (at 111.76 210.82 0)
       (effects (font (size 1.27 1.27)) hide)
     )
@@
       (effects (font (size 1.27 1.27)) (justify left))
     )
-    (property "Footprint" "" (id 2) (at 134.62 96.52 0)
+    (property "Footprint" "commons-passives_THT:Passive_THT_resistor_W2.54mm_L12.70mm" (id 2) (at 134.62 96.52 0)
       (effects (font (size 1.27 1.27)) hide)
     )
@@
       (effects (font (size 1.27 1.27)) (justify left))
     )
-    (property "Footprint" "" (id 2) (at 111.76 127 0)
-      (effects (font (size 1.27 1.27)) hide)
-    )
+    (property "Footprint" "commons-passives_THT:Passive_THT_resistor_W2.54mm_L12.70mm" (id 2) (at 111.76 127 0)
+      (effects (font (size 1.27 1.27)) hide)
+    )

Commit message: assigned footprint for all remaining standard passives
Parts:
- L55, L56, L57, L58, L59, L60, L61, L62, L63, L64, L65, L66: footprint (none) -> commons-passives_THT:Passive_THT_EMI_filter_W5.08mm_L7.62mm
Changed lines of the file:
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@@
       (effects (font (size 1.27 1.27)) (justify left))
     )
-    (property "Footprint" "" (id 2) (at 127 193.04 90)
+    (property "Footprint" "commons-passives_THT:Passive_THT_EMI_filter_W5.08mm_L7.62mm" (id 2) (at 127 193.04 90)
       (effects (font (size 1.27 1.27)) hide)
     )
@@
       (effects (font (size 1.27 1.27)) (justify left))
     )
-    (property "Footprint" "" (id 2) (at 142.24 182.88 90)
+    (property "Footprint" "commons-passives_THT:Passive_THT_EMI_filter_W5.08mm_L7.62mm" (id 2) (at 142.24 182.88 90)
       (effects (font (size 1.27 1.27)) hide)
     )
@@
       (effects (font (size 1.27 1.27)) (justify left))
     )
-    (property "Footprint" "" (id 2) (at 127 233.68 90)
+    (property "Footprint" "commons-passives_THT:Passive_THT_EMI_filter_W5.08mm_L7.62mm" (id 2) (at 127 233.68 90)
       (effects (font (size 1.27 1.27)) hide)
     )
@@
       (effects (font (size 1.27 1.27)) (justify left))
     )
-    (property "Footprint" "" (id 2) (at 142.24 243.84 90)
+    (property "Footprint" "commons-passives_THT:Passive_THT_EMI_filter_W5.08mm_L7.62mm" (id 2) (at 142.24 243.84 90)
       (effects (font (size 1.27 1.27)) hide)
     )
@@
       (effects (font (size 1.27 1.27)) (justify left))
     )
-    (property "Footprint" "" (id 2) (at 127 152.4 90)
+    (property "Footprint" "commons-passives_THT:Passive_THT_EMI_filter_W5.08mm_L7.62mm" (id 2) (at 127 152.4 90)
       (effects (font (size 1.27 1.27)) hide)
     )
@@
       (effects (font (size 1.27 1.27)) (justify left))
     )
-    (property "Footprint" "" (id 2) (at 142.24 223.52 90)
+    (property "Footprint" "commons-passives_THT:Passive_THT_EMI_filter_W5.08mm_L7.62mm" (id 2) (at 142.24 223.52 90)
       (effects (font (size 1.27 1.27)) hide)
     )
@@
       (effects (font (size 1.27 1.27)) (justify left))
     )
-    (property "Footprint" "" (id 2) (at 127 213.36 90)
+    (property "Footprint" "commons-passives_THT:Passive_THT_EMI_filter_W5.08mm_L7.62mm" (id 2) (at 127 213.36 90)
       (effects (font (size 1.27 1.27)) hide)
     )
@@
       (effects (font (size 1.27 1.27)) (justify left))
     )
-    (property "Footprint" "" (id 2) (at 127 172.72 90)
+    (property "Footprint" "commons-passives_THT:Passive_THT_EMI_filter_W5.08mm_L7.62mm" (id 2) (at 127 172.72 90)
       (effects (font (size 1.27 1.27)) hide)
     )
@@
       (effects (font (size 1.27 1.27)) (justify left))
     )
-    (property "Footprint" "" (id 2) (at 142.24 142.24 90)
+    (property "Footprint" "commons-passives_THT:Passive_THT_EMI_filter_W5.08mm_L7.62mm" (id 2) (at 142.24 142.24 90)
       (effects (font (size 1.27 1.27)) hide)
     )
@@
       (effects (font (size 1.27 1.27)) (justify left))
     )
-    (property "Footprint" "" (id 2) (at 127 132.08 90)
+    (property "Footprint" "commons-passives_THT:Passive_THT_EMI_filter_W5.08mm_L7.62mm" (id 2) (at 127 132.08 90)
       (effects (font (size 1.27 1.27)) hide)
     )
@@
       (effects (font (size 1.27 1.27)) (justify left))
     )
-    (property "Footprint" "" (id 2) (at 142.24 162.56 90)
+    (property "Footprint" "commons-passives_THT:Passive_THT_EMI_filter_W5.08mm_L7.62mm" (id 2) (at 142.24 162.56 90)
       (effects (font (size 1.27 1.27)) hide)
     )
@@
       (effects (font (size 1.27 1.27)) (justify left))
     )
-    (property "Footprint" "" (id 2) (at 142.24 203.2 90)
-      (effects (font (size 1.27 1.27)) hide)
-    )
+    (property "Footprint" "commons-passives_THT:Passive_THT_EMI_filter_W5.08mm_L7.62mm" (id 2) (at 142.24 203.2 90)
+      (effects (font (size 1.27 1.27)) hide)
+    )
