File: motherboard.kicad_sch (KiCad schematic)
At the start: 0 parts

Commit message: starting CPU -- u10, rp for addresses
Other:
- added sheet U10-68000 (subsheet_105.kicad_sch)
- note added: "Page 7"
Changed lines of the file:
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@@
   (title_block
     (title "Converted schematics of Atari 260/520 ST")
-    (date "2023-01-13")
+    (date "2023-02-23")
     (rev "0")
     (comment 1 "…sporniket/kicad-conversions--atari-260-520-st-motherboard--c070231")
@@
   (text "Sheet 1" (at 25.4 50.8 0)
     (effects (font (size 3.9878 3.9878)) (justify left bottom))
+  )
+  (text "Page 7" (at 176.53 110.49 0)
+    (effects (font (size 1.27 1.27)) (justify left bottom))
   )
   (text "Page 6" (at 176.53 100.33 0)
@@
     )
     (property "Sheet file" "subsheet_104.kicad_sch" (id 1) (at 25.4 102.1846 0)
+      (effects (font (size 1.27 1.27)) (justify left top))
+    )
+  )
+  (sheet (at 25.4 107.95) (size 160.02 3.81) (fields_autoplaced)
+    (stroke (width 0.1524) (type solid) (color 0 0 0 0))
+    (fill (color 0 0 0 0.0000))
+    (property "Sheet name" "U10-68000" (id 0) (at 25.4 106.9734 0)
+      (effects (font (size 1.8 1.8)) (justify left bottom))
+    )
+    (property "Sheet file" "subsheet_105.kicad_sch" (id 1) (at 25.4 112.3446 0)
       (effects (font (size 1.27 1.27)) (justify left top))
     )
@@
     (path "/00000000-0000-0000-0000-00006351bff4" (page "5"))
     (path "/00000000-0000-0000-0000-000063c0e747" (page "6"))
+    (path "/5b318927-956e-4f28-80bb-c09676827d9a" (page "7"))
   )
   (symbol_instances
@@
       (reference "R134") (unit 1) (value "68R") (footprint "commons-passives_THT:Passive_THT_resistor_W2.54mm_L12.70mm")
     )
+    (path "/5b318927-956e-4f28-80bb-c09676827d9a/fa2ed178-d71a-47cb-b52e-1065d46615ab"
+      (reference "RP1") (unit 1) (value "10K×8") (footprint "Resistor_THT:R_Array_SIP9")
+    )
+    (path "/5b318927-956e-4f28-80bb-c09676827d9a/2cb22489-ce82-448d-905e-01465d95bc47"
+      (reference "RP2") (unit 1) (value "10K×8") (footprint "Resistor_THT:R_Array_SIP9")
+    )
+    (path "/5b318927-956e-4f28-80bb-c09676827d9a/d0564698-ba14-4bda-b9e9-0b388f21bac2"
+      (reference "RP3") (unit 1) (value "10K×8") (footprint "Resistor_THT:R_Array_SIP9")
+    )
+    (path "/5b318927-956e-4f28-80bb-c09676827d9a/3e670fa4-4e6c-44b6-8bdb-ef4ae836a4bf"
+      (reference "RP4") (unit 1) (value "4K7×8") (footprint "Resistor_THT:R_Array_SIP9")
+    )
+    (path "/5b318927-956e-4f28-80bb-c09676827d9a/7bba4360-0b90-4aaf-9fed-4f7961efe14b"
+      (reference "RP5") (unit 1) (value "10K×8") (footprint "Resistor_THT:R_Array_SIP9")
+    )
+    (path "/5b318927-956e-4f28-80bb-c09676827d9a/4a695da9-73c5-4eda-80d5-d4bc04662a45"
+      (reference "RP6") (unit 1) (value "10K×8") (footprint "Resistor_THT:R_Array_SIP9")
+    )
     (path "/00000000-0000-0000-0000-00006351bff4/00000000-0000-0000-0000-00006356e89e"
       (reference "U2") (unit 1) (value "27C512_PHY") (footprint "Package_DIP:DIP-28_W15.24mm_LongPads")
@@
       (reference "U7") (unit 1) (value "27C512_PHY") (footprint "Package_DIP:DIP-28_W15.24mm_LongPads")
     )
+    (path "/5b318927-956e-4f28-80bb-c09676827d9a/0ad984e5-573c-4a8b-8dee-9cd70d550511"
+      (reference "U10") (unit 1) (value "MC68000_DIP_64_PHY") (footprint "Package_DIP:DIP-64_W22.86mm_LongPads")
+    )
     (path "/00000000-0000-0000-0000-000063c0e747/00000000-0000-0000-0000-000063c0f30d"

Commit message: reset circuit around u37
Other:
- sheet U10-68000 renamed U10-68000 ; U36–37–Reset circuit
Changed lines of the file:
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@@
     (stroke (width 0.1524) (type solid) (color 0 0 0 0))
     (fill (color 0 0 0 0.0000))
-    (property "Sheet name" "U10-68000" (id 0) (at 25.4 106.9734 0)
+    (property "Sheet name" "U10-68000 ; U36–37–Reset circuit" (id 0) (at 25.4 106.9734 0)
       (effects (font (size 1.8 1.8)) (justify left bottom))
     )
@@
       (reference "#PWR?") (unit 1) (value "+5V") (footprint "")
     )
+    (path "/5b318927-956e-4f28-80bb-c09676827d9a/3fe0de95-c3a8-4b89-9907-9c53930b061e"
+      (reference "#PWR?") (unit 1) (value "GND") (footprint "")
+    )
     (path "/5b318927-956e-4f28-80bb-c09676827d9a/486d4e53-7158-47b2-963f-d35c444782b0"
       (reference "#PWR?") (unit 1) (value "GND") (footprint "")
     )
+    (path "/5b318927-956e-4f28-80bb-c09676827d9a/49334b3d-6990-4a84-8088-0cfea786f6c8"
+      (reference "#PWR?") (unit 1) (value "+5V") (footprint "")
+    )
+    (path "/5b318927-956e-4f28-80bb-c09676827d9a/4ef0a41d-d5eb-47ab-a511-a19bc0fb1afe"
+      (reference "#PWR?") (unit 1) (value "+5V") (footprint "")
+    )
     (path "/5b318927-956e-4f28-80bb-c09676827d9a/53316c2c-d36c-4f57-95c5-96ca6301eb48"
       (reference "#PWR?") (unit 1) (value "+5V") (footprint "")
     )
+    (path "/5b318927-956e-4f28-80bb-c09676827d9a/74d79676-f388-40c1-a5f7-e3c191b7f7eb"
+      (reference "#PWR?") (unit 1) (value "+5V") (footprint "")
+    )
     (path "/5b318927-956e-4f28-80bb-c09676827d9a/7a17ded4-f901-4cfa-ad3d-21bdd5494e11"
       (reference "#PWR?") (unit 1) (value "+5V") (footprint "")
     )
+    (path "/5b318927-956e-4f28-80bb-c09676827d9a/808017d9-e8b6-4e48-a94f-b816372f20e5"
+      (reference "#PWR?") (unit 1) (value "GND") (footprint "")
+    )
+    (path "/5b318927-956e-4f28-80bb-c09676827d9a/80e4d482-dadd-45ef-9576-d2f3729f872a"
+      (reference "#PWR?") (unit 1) (value "GND") (footprint "")
+    )
+    (path "/5b318927-956e-4f28-80bb-c09676827d9a/964a8741-acf0-49ed-8b00-d462e9b78d85"
+      (reference "#PWR?") (unit 1) (value "GND") (footprint "")
+    )
     (path "/5b318927-956e-4f28-80bb-c09676827d9a/9f329afb-6e7e-4e5a-bed3-7a1c47d267dc"
       (reference "#PWR?") (unit 1) (value "+5V") (footprint "")
     )
+    (path "/5b318927-956e-4f28-80bb-c09676827d9a/d8f6467f-cc89-4d4e-8ca2-c195ac9733c5"
+      (reference "#PWR?") (unit 1) (value "+5V") (footprint "")
+    )
     (path "/5b318927-956e-4f28-80bb-c09676827d9a/f9b98555-db21-40ca-b3e6-907bd3e24c82"
       (reference "#PWR?") (unit 1) (value "GND") (footprint "")
@@
       (reference "C45") (unit 1) (value "22uF") (footprint "commons-passives_THT:Passive_THT_capacitor_mlcc_W2.54mm_L12.70mm")
     )
+    (path "/5b318927-956e-4f28-80bb-c09676827d9a/c1d51f25-0ff6-4322-90d8-14ad1e9a5228"
+      (reference "C48") (unit 1) (value "0.01uF") (footprint "commons-passives_THT:Passive_THT_capacitor_mlcc_W2.54mm_L12.70mm")
+    )
+    (path "/5b318927-956e-4f28-80bb-c09676827d9a/fb3bbfdd-4e79-4218-8e82-0b9eff351407"
+      (reference "C49") (unit 1) (value "0.01uF") (footprint "commons-passives_THT:Passive_THT_capacitor_mlcc_W2.54mm_L12.70mm")
+    )
+    (path "/5b318927-956e-4f28-80bb-c09676827d9a/fb7218d4-df32-41e1-9dce-2b9f4dc870ef"
+      (reference "C50") (unit 1) (value "22uF") (footprint "")
+    )
     (path "/00000000-0000-0000-0000-000062e3a54e/00000000-0000-0000-0000-000062f5601f"
       (reference "C51") (unit 1) (value "0.1uF") (footprint "commons-passives_THT:Passive_THT_capacitor_mlcc_W2.54mm_L12.70mm")
@@
       (reference "C54") (unit 1) (value "0.1uF") (footprint "commons-passives_THT:Passive_THT_capacitor_mlcc_W2.54mm_L12.70mm")
     )
+    (path "/5b318927-956e-4f28-80bb-c09676827d9a/336d836f-5cc4-4f9d-9e69-3213e129d423"
+      (reference "C55") (unit 1) (value "22uF") (footprint "")
+    )
     (path "/00000000-0000-0000-0000-000062db00cc/00000000-0000-0000-0000-000062ee0e8c"
       (reference "C57") (unit 1) (value "22uF") (footprint "commons-passives_THT:Passive_THT_capacitor_mlcc_W2.54mm_L12.70mm")
     )
+    (path "/5b318927-956e-4f28-80bb-c09676827d9a/0df7b336-06c3-4cad-9a2e-f58d4fc33819"
+      (reference "C70") (unit 1) (value "0.1uF") (footprint "commons-passives_THT:Passive_THT_capacitor_mlcc_W2.54mm_L12.70mm")
+    )
     (path "/00000000-0000-0000-0000-000062db00cc/00000000-0000-0000-0000-000062ee5cdb"
       (reference "C78") (unit 1) (value "22uF") (footprint "commons-passives_THT:Passive_THT_capacitor_mlcc_W2.54mm_L12.70mm")
@@
       (reference "R75") (unit 1) (value "4K7") (footprint "")
     )
+    (path "/5b318927-956e-4f28-80bb-c09676827d9a/19652f52-4ebe-4276-b1bc-827e10b12f00"
+      (reference "R82") (unit 1) (value "12K") (footprint "")
+    )
+    (path "/5b318927-956e-4f28-80bb-c09676827d9a/23c49af6-87df-4cbd-bb61-89161e55849f"
+      (reference "R83") (unit 1) (value "12K") (footprint "")
+    )
     (path "/00000000-0000-0000-0000-000062e3a54e/00000000-0000-0000-0000-000062f56032"
       (reference "R87") (unit 1) (value "3K6") (footprint "commons-passives_THT:Passive_THT_resistor_W2.54mm_L12.70mm")
     )
+    (path "/5b318927-956e-4f28-80bb-c09676827d9a/9cbd6214-ee5a-47bb-877d-bfbda1e12028"
+      (reference "R93") (unit 1) (value "12K") (footprint "")
+    )
     (path "/00000000-0000-0000-0000-000062e3a54e/00000000-0000-0000-0000-000062e634e7"
       (reference "R115") (unit 1) (value "27") (footprint "commons-passives_THT:Passive_THT_resistor_W2.54mm_L12.70mm")
@@
       (reference "RP6") (unit 1) (value "10K×8") (footprint "Resistor_THT:R_Array_SIP9")
     )
+    (path "/5b318927-956e-4f28-80bb-c09676827d9a/c40b4c5e-0054-472b-92ef-7d5a32a3dd16"
+      (reference "SW2") (unit 1) (value "RESET") (footprint "")
+    )
     (path "/00000000-0000-0000-0000-00006351bff4/00000000-0000-0000-0000-00006356e89e"
       (reference "U2") (unit 1) (value "27C512_PHY") (footprint "Package_DIP:DIP-28_W15.24mm_LongPads")
@@
       (reference "U34") (unit 1) (value "DRAM_256K×1_PHY") (footprint "Package_DIP:DIP-16_W7.62mm_LongPads")
     )
+    (path "/5b318927-956e-4f28-80bb-c09676827d9a/1c32df98-362b-45fc-ae4f-14f9aff703a2"
+      (reference "U37") (unit 1) (value "LM556_DUAL_TIMER_PHY") (footprint "Package_DIP:DIP-14_W7.62mm_LongPads")
+    )
     (path "/00000000-0000-0000-0000-000062db00cc/00000000-0000-0000-0000-000062edd17c"
