File: subsheet_105.kicad_sch (KiCad schematic)
At the start: 7 parts, among them U10 MC68000_DIP_64_PHY

Commit message: continue CPU : some resistor networks, power supply, buses
Parts:
- added C105: 22uF, symbol Device:C_Polarized_Small_US
- added C9: 0.1uF, commons-passives_THT:Passive_THT_capacitor_mlcc_W2.54mm_L12.70mm, symbol Device:C_Small
- added L25: Ferrite bead, commons-passives_THT:Passive_THT_ferrite_bead_W3.81mm_L15.24mm, symbol Device:Ferrite_Bead_Small
Connections:
- net A16: now also RP5.9 (R8); no longer RP5.2 (R1)
- net A17: now also RP5.8 (R7); no longer RP5.3 (R2)
- net A18: now also RP5.7 (R6); no longer RP5.4 (R3)
- net A19: now also RP5.6 (R5); no longer RP5.5 (R4)
- net A20: now also RP5.5 (R4); no longer RP5.6 (R5)
- net A21: now also RP5.4 (R3), U10.50 (A21); no longer RP5.7 (R6), U10.49 (VCC)
- net A22: now also RP5.3 (R2), U10.51 (A22); no longer RP5.8 (R7), U10.50 (A21)
- net A23: now also RP5.2 (R1), U10.52 (A23); no longer RP5.9 (R8), U10.51 (A22)
- net D4: now reaches U10.1 (D4)
- net D4: now also RP3.6 (R5)
- net VCC: now reaches U10.14 (VCC)
- net VCC: now also U10.49 (VCC), C105.1, C9.1, L25.1
- net D3: now reaches U10.2 (D3)
- net D3: now also RP3.5 (R4)
- net D2: now reaches U10.3 (D2)
- net D2: now also RP3.4 (R3)
- net D1: now reaches U10.4 (D1)
- net D1: now also RP3.3 (R2)
- net D0: now reaches U10.5 (D0)
- net D0: now also RP3.2 (R1)
- net GND: now reaches U10.53 (GND)
- net GND: now also C105.2, C9.2
- net D15: now reaches U10.54 (D15)
- net D15: now also RP6.9 (R8)
- net D14: now reaches U10.55 (D14)
- net D14: now also RP6.8 (R7)
- net D13: now reaches U10.56 (D13)
- net D13: now also RP6.7 (R6)
- net D12: now reaches U10.57 (D12)
- net D12: now also RP6.6 (R5)
- net D11: now reaches U10.58 (D11)
- net D11: now also RP6.5 (R4)
- net D10: now reaches U10.59 (D10)
- net D10: now also RP6.4 (R3)
- net D9: now reaches U10.60 (D09)
- net D9: now also RP6.3 (R2)
- net D8: now reaches U10.61 (D08)
- net D8: now also RP6.2 (R1)
- net D7: now reaches U10.62 (D07)
- net D7: now also RP3.9 (R8)
- net D6: now reaches U10.63 (D06)
- net D6: now also RP3.8 (R7)
- net D5: now reaches U10.64 (D05)
- net D5: now also RP3.7 (R6)
- new net +5V: L25.2
Other:
- moved on the sheet: RP1, RP2, RP3, RP5, RP6, U10

Commit message: wiring of data and address bus to RP
Connections:
- net A10: now also RP2.6 (R5); no longer RP2.7 (R6)
- net A11: now also RP2.8 (R7); no longer RP2.6 (R5)
- net A12: now also RP2.7 (R6); no longer RP2.5 (R4)
- net A13: now also RP2.3 (R2); no longer RP2.4 (R3)
- net A14: now also RP2.4 (R3); no longer RP2.3 (R2)
- net A16: now also RP5.2 (R1); no longer RP5.9 (R8)
- net A17: now also RP5.3 (R2); no longer RP5.8 (R7)
- net A18: now also RP5.4 (R3); no longer RP5.7 (R6)
- net A19: now also RP5.8 (R7); no longer RP5.6 (R5)
- net A20: now also RP5.7 (R6); no longer RP5.5 (R4)
- net A21: now also RP5.9 (R8); no longer RP5.4 (R3)
- net A22: now also RP5.5 (R4); no longer RP5.3 (R2)
- net A23: now also RP5.6 (R5); no longer RP5.2 (R1)
- net A8: now also RP2.5 (R4); no longer RP2.9 (R8)
- net A9: now also RP2.9 (R8); no longer RP2.8 (R7)
Other:
- moved on the sheet: RP3, RP6

Commit message: Rearrange pull-up resistor networks, general layout
Connections:
- net +5V: now also RP1.1 (common), RP2.1 (common), RP3.1 (common), RP5.1 (common), RP6.1 (common)
Other:
- note added: "Pull-ups"
- moved on the sheet: C105, C9, L25, RP1, RP2, RP3, RP4, RP5, RP6

Commit message: continue pull-ups
Parts:
- added R1, R11, R2, R29, R32, R6, R75: 4K7, symbol Device:R_Small_US
- added R10, R12, R9: 10K, symbol Device:R_Small_US
- added R30, R31: 1K, symbol Device:R_Small_US
Connections:
- net +5V: now also RP4.1 (common), R1.1, R10.1, R11.1, R12.1, R2.1, R29.1, R30.1, R31.1, R32.1, R6.1, R75.1, R9.1
- net XDTACK: now reaches U10.10 (~{DTACK})
- net XDTACK: now also R30.2
- net IPL2: now reaches U10.23 (IPL2)
- net IPL2: now also RP4.4 (R3)
- net IPL1: now reaches U10.24 (IPL1)
- net IPL1: now also RP4.9 (R8)
- net IPL0: now reaches U10.25 (IPL0)
- net IPL0: now also R1.2
- net FC2: now reaches U10.26 (FC2)
- net FC2: now also R12.2
- net FC1: now reaches U10.27 (FC1)
- net FC1: now also R10.2
- net FC0: now reaches U10.28 (FC0)
- net FC0: now also R9.2
Other:
- moved on the sheet: RP1, RP2, RP3, RP4, RP5, RP6

Commit message: almost done CPU, ready to do reset circuit
Connections:
- net GND: now also U10.16 (GND)
- net XBG: now reaches U10.11 (~{BG})
- net XBG: now also RP4.2 (R1)
- net XBGACK: now reaches U10.12 (~{BGACK})
- net XBGACK: now also R2.2
- net XBR: now reaches U10.13 (~{BR})
- net XBR: now also RP4.8 (R7)
- net 8MHZ: now reaches U10.15 (CLK)
- net HALT: now reaches U10.17 (~{HALT})
- net XRESET: now reaches U10.18 (~{RESET})
- net XRESET: now also R31.2
- net XVMA: now reaches U10.19 (~{VMA})
- net XVMA: now also RP4.6 (R5)
- net E: now reaches U10.20 (E)
- net XVPA: now reaches U10.21 (~{VPA})
- net XVPA: now also RP4.3 (R2)
- net XBERR: now reaches U10.22 (~{BERR})
- net XBERR: now also RP4.7 (R6)
- net XAS: now reaches U10.6 (~{AS})
- net XAS: now also R29.2
- net XUDS: now reaches U10.7 (~{UDS})
- net XUDS: now also R32.2
- net XLDS: now reaches U10.8 (~{LDS})
- net XLDS: now also R11.2
- net XRXW: now reaches U10.9 (R/~{W})
- net XRXW: now also R6.2
Changed lines of the file:
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@@
     (stroke (width 0) (type default) (color 0 0 0 0))
   )
-  (wire (pts (xy 138.43 129.54) (xy 147.32 129.54))
+  (wire (pts (xy 125.73 129.54) (xy 147.32 129.54))
     (stroke (width 0) (type default) (color 0 0 0 0))
   )
@@
     (effects (font (size 1.27 1.27)) (justify left bottom))
   )
+  (label "HALT" (at 138.43 132.08 0)
+    (effects (font (size 1.27 1.27)) (justify left bottom))
+  )
   (label "A23" (at 191.77 121.92 180)
     (effects (font (size 1.27 1.27)) (justify right bottom))
@@
     (effects (font (size 1.27 1.27)) (justify right bottom))
   )
-  (label "VCC" (at 138.43 124.46 180)
-    (effects (font (size 1.27 1.27)) (justify right bottom))
+  (label "VCC" (at 138.43 124.46 0)
+    (effects (font (size 1.27 1.27)) (justify left bottom))
   )
   (label "FC2" (at 180.34 237.49 180)
@@
     (property "Intersheet References" "${INTERSHEET_REFS}" (id 0) (at -6.35 0 0)
       (effects (font (size 1.27 1.27)) hide)
+    )
+  )
+  (global_label "XBR" (shape input) (at 138.43 121.92 180) (fields_autoplaced)
+    (effects (font (size 1.27 1.27)) (justify right))
+    (property "Intersheet References" "${INTERSHEET_REFS}" (id 0) (at 132.3563 121.8406 0)
+      (effects (font (size 1.27 1.27)) (justify right) hide)
+    )
+  )
+  (global_label "XBG" (shape output) (at 138.43 116.84 180) (fields_autoplaced)
+    (effects (font (size 1.27 1.27)) (justify right))
+    (property "Intersheet References" "${INTERSHEET_REFS}" (id 0) (at 132.3563 116.7606 0)
+      (effects (font (size 1.27 1.27)) (justify right) hide)
+    )
+  )
+  (global_label "XBG" (shape output) (at 144.78 248.92 0) (fields_autoplaced)
+    (effects (font (size 1.27 1.27)) (justify left))
+    (property "Intersheet References" "${INTERSHEET_REFS}" (id 0) (at 150.8537 248.9994 0)
+      (effects (font (size 1.27 1.27)) (justify left) hide)
+    )
+  )
+  (global_label "XBGACK" (shape input) (at 138.43 119.38 180) (fields_autoplaced)
+    (effects (font (size 1.27 1.27)) (justify right))
+    (property "Intersheet References" "${INTERSHEET_REFS}" (id 0) (at 128.7277 119.3006 0)
+      (effects (font (size 1.27 1.27)) (justify right) hide)
     )
   )
@@
     )
   )
+  (global_label "XRXW" (shape output) (at 180.34 214.63 0) (fields_autoplaced)
+    (effects (font (size 1.27 1.27)) (justify left))
+    (property "Intersheet References" "${INTERSHEET_REFS}" (id 0) (at 187.8047 214.7094 0)
+      (effects (font (size 1.27 1.27)) (justify left) hide)
+    )
+  )
+  (global_label "XBGACK" (shape input) (at 180.34 212.09 0) (fields_autoplaced)
+    (effects (font (size 1.27 1.27)) (justify left))
+    (property "Intersheet References" "${INTERSHEET_REFS}" (id 0) (at 190.0423 212.1694 0)
+      (effects (font (size 1.27 1.27)) (justify left) hide)
+    )
+  )
   (global_label "XDTACK" (shape input) (at 180.34 199.39 0) (fields_autoplaced)
     (effects (font (size 1.27 1.27)) (justify left))
@@
     )
   )
+  (global_label "XVPA" (shape input) (at 144.78 246.38 0) (fields_autoplaced)
+    (effects (font (size 1.27 1.27)) (justify left))
+    (property "Intersheet References" "${INTERSHEET_REFS}" (id 0) (at 151.7609 246.4594 0)
+      (effects (font (size 1.27 1.27)) (justify left) hide)
+    )
+  )
+  (global_label "XBERR" (shape input) (at 144.78 236.22 0) (fields_autoplaced)
+    (effects (font (size 1.27 1.27)) (justify left))
+    (property "Intersheet References" "${INTERSHEET_REFS}" (id 0) (at 153.2728 236.2994 0)
+      (effects (font (size 1.27 1.27)) (justify left) hide)
+    )
+  )
   (global_label "FC[0..2]" (shape bidirectional) (at 107.95 25.4 0) (fields_autoplaced)
     (effects (font (size 1.27 1.27)) (justify left))
@@
     )
   )
+  (global_label "XVMA" (shape output) (at 144.78 238.76 0) (fields_autoplaced)
+    (effects (font (size 1.27 1.27)) (justify left))
+    (property "Intersheet References" "${INTERSHEET_REFS}" (id 0) (at 151.9423 238.8394 0)
+      (effects (font (size 1.27 1.27)) (justify left) hide)
+    )
+  )
+  (global_label "8MHZ" (shape input) (at 138.43 127 180) (fields_autoplaced)
+    (effects (font (size 1.27 1.27)) (justify right))
+    (property "Intersheet References" "${INTERSHEET_REFS}" (id 0) (at 130.9048 126.9206 0)
+      (effects (font (size 1.27 1.27)) (justify right) hide)
+    )
+  )
+  (global_label "XLDS" (shape output) (at 180.34 217.17 0) (fields_autoplaced)
+    (effects (font (size 1.27 1.27)) (justify left))
+    (property "Intersheet References" "${INTERSHEET_REFS}" (id 0) (at 187.3813 217.2494 0)
+      (effects (font (size 1.27 1.27)) (justify left) hide)
+    )
+  )
+  (global_label "XAS" (shape output) (at 180.34 219.71 0) (fields_autoplaced)
+    (effects (font (size 1.27 1.27)) (justify left))
+    (property "Intersheet References" "${INTERSHEET_REFS}" (id 0) (at 186.1718 219.7894 0)
+      (effects (font (size 1.27 1.27)) (justify left) hide)
+    )
+  )
+  (global_label "XLDS" (shape output) (at 138.43 109.22 180) (fields_autoplaced)
+    (effects (font (size 1.27 1.27)) (justify right))
+    (property "Intersheet References" "${INTERSHEET_REFS}" (id 0) (at 131.3887 109.1406 0)
+      (effects (font (size 1.27 1.27)) (justify right) hide)
+    )
+  )
+  (global_label "XVMA" (shape output) (at 138.43 137.16 180) (fields_autoplaced)
+    (effects (font (size 1.27 1.27)) (justify right))
+    (property "Intersheet References" "${INTERSHEET_REFS}" (id 0) (at 131.2677 137.0806 0)
+      (effects (font (size 1.27 1.27)) (justify right) hide)
+    )
+  )
+  (global_label "XVPA" (shape input) (at 138.43 142.24 180) (fields_autoplaced)
+    (effects (font (size 1.27 1.27)) (justify right))
+    (property "Intersheet References" "${INTERSHEET_REFS}" (id 0) (at 131.4491 142.1606 0)
+      (effects (font (size 1.27 1.27)) (justify right) hide)
+    )
+  )
   (global_label "ADDR[1..23]" (shape output) (at 31.75 25.4 0) (fields_autoplaced)
     (effects (font (size 1.27 1.27)) (justify left))
@@
     )
   )
+  (global_label "XRESET" (shape bidirectional) (at 138.43 134.62 180) (fields_autoplaced)
+    (effects (font (size 1.27 1.27)) (justify right))
+    (property "Intersheet References" "${INTERSHEET_REFS}" (id 0) (at 129.151 134.5406 0)
+      (effects (font (size 1.27 1.27)) (justify right) hide)
+    )
+  )
+  (global_label "E" (shape output) (at 138.43 139.7 180) (fields_autoplaced)
+    (effects (font (size 1.27 1.27)) (justify right))
+    (property "Intersheet References" "${INTERSHEET_REFS}" (id 0) (at 134.9568 139.6206 0)
+      (effects (font (size 1.27 1.27)) (justify right) hide)
+    )
+  )
+  (global_label "XRXW" (shape output) (at 138.43 111.76 180) (fields_autoplaced)
+    (effects (font (size 1.27 1.27)) (justify right))
+    (property "Intersheet References" "${INTERSHEET_REFS}" (id 0) (at 130.9653 111.6806 0)
+      (effects (font (size 1.27 1.27)) (justify right) hide)
+    )
+  )
+  (global_label "XBERR" (shape input) (at 138.43 144.78 180) (fields_autoplaced)
+    (effects (font (size 1.27 1.27)) (justify right))
+    (property "Intersheet References" "${INTERSHEET_REFS}" (id 0) (at 129.9372 144.7006 0)
+      (effects (font (size 1.27 1.27)) (justify right) hide)
+    )
+  )
   (global_label "XIPL[1..2]" (shape input) (at 146.05 25.4 0) (fields_autoplaced)
     (effects (font (size 1.27 1.27)) (justify left))
     (property "Intersheet References" "${INTERSHEET_REFS}" (id 0) (at 157.8085 25.3206 0)
       (effects (font (size 1.27 1.27)) (justify left) hide)
+    )
+  )
+  (global_label "XAS" (shape output) (at 138.43 104.14 180) (fields_autoplaced)
+    (effects (font (size 1.27 1.27)) (justify right))
+    (property "Intersheet References" "${INTERSHEET_REFS}" (id 0) (at 132.5982 104.0606 0)
+      (effects (font (size 1.27 1.27)) (justify right) hide)
+    )
+  )
+  (global_label "XBR" (shape input) (at 144.78 233.68 0) (fields_autoplaced)
+    (effects (font (size 1.27 1.27)) (justify left))
+    (property "Intersheet References" "${INTERSHEET_REFS}" (id 0) (at 150.8537 233.7594 0)
+      (effects (font (size 1.27 1.27)) (justify left) hide)
+    )
+  )
+  (global_label "XUDS" (shape output) (at 180.34 222.25 0) (fields_autoplaced)
+    (effects (font (size 1.27 1.27)) (justify left))
+    (property "Intersheet References" "${INTERSHEET_REFS}" (id 0) (at 187.6837 222.3294 0)
+      (effects (font (size 1.27 1.27)) (justify left) hide)
+    )
+  )
+  (global_label "XRESET" (shape bidirectional) (at 180.34 201.93 0) (fields_autoplaced)
+    (effects (font (size 1.27 1.27)) (justify left))
+    (property "Intersheet References" "${INTERSHEET_REFS}" (id 0) (at 189.619 202.0094 0)
+      (effects (font (size 1.27 1.27)) (justify left) hide)
+    )
+  )
+  (global_label "XUDS" (shape output) (at 138.43 106.68 180) (fields_autoplaced)
+    (effects (font (size 1.27 1.27)) (justify right))
+    (property "Intersheet References" "${INTERSHEET_REFS}" (id 0) (at 131.0863 106.6006 0)
+      (effects (font (size 1.27 1.27)) (justify right) hide)
     )
   )
@@
     (pin "2")
   )
+  (symbol (lib_id "power:GND") (at 125.73 129.54 0) (unit 1)
+    (in_bom yes) (on_board yes)
+    (property "Reference" "#PWR?" (id 0) (at 125.73 135.89 0)
+      (effects (font (size 1.27 1.27)) hide)
+    )
+    (property "Value" "GND" (id 1) (at 124.46 130.81 0)
+      (effects (font (size 1.27 1.27)) (justify right))
+    )
+    (property "Footprint" "" (id 2) (at 125.73 129.54 0)
+      (effects (font (size 1.27 1.27)) hide)
+    )
+    (property "Datasheet" "" (id 3) (at 125.73 129.54 0)
+      (effects (font (size 1.27 1.27)) hide)
+    )
+    (pin "1")
+  )
   (symbol (lib_id "Device:R_Network08_US") (at 96.52 195.58 90) (unit 1)

Commit message: little touch on pull ups
Connections:
- net HALT: now also R75.2
- no-connect marks 1 -> 2

Commit message: reset circuit around u37
Parts:
- added C48, C49: 0.01uF, commons-passives_THT:Passive_THT_capacitor_mlcc_W2.54mm_L12.70mm, symbol Device:C_Small
- added C50, C55: 22uF, symbol Device:C_Polarized_Small_US
- added C70: 0.1uF, commons-passives_THT:Passive_THT_capacitor_mlcc_W2.54mm_L12.70mm, symbol Device:C_Small
- added R82, R83, R93: 12K, symbol Device:R_Small_US
- added SW2: RESET, symbol Switch:SW_Push
- added U37: LM556_DUAL_TIMER_PHY, Package_DIP:DIP-14_W7.62mm_LongPads, symbol lm556:LM556_DUAL_TIMER_PHY
Connections:
- net +5V: now also R82.2, R83.2, R93.2, U37.10 (~{2RESET}), U37.14 (VCC), U37.4 (~{1RESET})
- net GND: now also C48.2, C49.2, C50.2, C55.2, C70.2, SW2.1, U37.7 (GND)
- new net: C70.1, R93.1, SW2.2, U37.6 (1TRIGGER)
- new net: C55.1, R82.1, U37.1 (1DISCHARGE), U37.2 (1THRESHOLD)
- new net: C48.1, U37.11 (2CTLVLT)
- new net: C50.1, R83.1, U37.12 (2THRESHOLD), U37.8 (2TRIGGER)
- new net: C49.1, U37.3 (1CTLVLT)
- new net out1: U37.5 (1OUTPUT)
- new net out2: U37.9 (2OUTPUT)
- no-connect marks 2 -> 3

Commit message: finished reset circuit
Parts:
- added C?: 0.1uF, commons-passives_THT:Passive_THT_capacitor_mlcc_W2.54mm_L12.70mm, symbol Device:C_Small
- added U36: 74LS05_PHY, Package_DIP:DIP-14_W7.62mm_LongPads, symbol 74x05:74LS05_PHY
Connections:
- net +5V: now also C?.1, U36.14 (VCC)
- net GND: now also C?.2, U36.7 (GND)
- net HALT: now also U36.2 (1Y), U36.4 (2Y)
- net XRESET: now also U36.10 (5Y), U36.12 (6Y)
- net out1: now also U36.1 (1A), U36.13 (6A)
- net out2: now also U36.11 (5A), U36.3 (2A)
- new net ACIA_MIDI_RX: U36.9 (4A)
- new net ACIA_MIDI_TX: U36.5 (3A)
- new net MIDI_OUT: U36.6 (3Y)
- new net MIDI_THROUGH: U36.8 (4Y)
Other:
- note added: "From/To : ACIA to MIDI Ports"
