File: subsheet_105.kicad_sch (KiCad schematic)
At the start: 0 parts

Commit message: done power socket
Parts:
- added C100, C102, C71: 0.1uF, commons-passives_THT:Passive_THT_capacitor_mlcc_W2.54mm_L12.70mm, symbol Device:C_Small
- added C101, C103, C72: 680pF, commons-passives_THT:Passive_THT_capacitor_mlcc_W2.54mm_L12.70mm, symbol Device:C_Small
- added J9: DIN-7 POWER, symbol Connector:DIN-7
- added L3: SNH19L-0601-4, symbol common-mode-filters_custom_Atari-ST:SNH19L-0601-4
- added SW?: SW_SPST, symbol Switch:SW_SPST
Connections:
- new net: J9.1, J9.6, L3.1
- new net: J9.3, J9.7, L3.7
- new net: J9.4, L3.3
- new net: J9.5, L3.5
- new net: L3.14, SW?.1 (A)
- new net +12V: C100.1, C101.1, L3.12
- new net +5V: C71.1, C72.1, SW?.2 (B)
- new net -12V: C102.1, C103.1, L3.10
- new net GND: C100.2, C101.2, C102.2, C103.2, C71.2, C72.2, L3.8
- no-connect marks 0 -> 1
Other:
- note added: "+12V"
- note added: "+5V"
- note added: "-12V"
- note added: "GND"

Commit message: power socket subsheet : added missing polarized capacitor
Parts:
- added C106: 470uF, symbol Device:C_Polarized_Small_US
Connections:
- net +5V: now also C106.1
- net GND: now also C106.2
Other:
- moved on the sheet: C101, C103, C72

Commit message: fixed some DRC errors
Changed lines of the file:
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@@
   (junction (at 157.48 33.02) (diameter 0) (color 0 0 0 0)
+  )
+  (junction (at 88.9 76.2) (diameter 0) (color 0 0 0 0)
   )
   (junction (at 45.72 63.5) (diameter 0) (color 0 0 0 0)
@@
     (stroke (width 0) (type default) (color 0 0 0 0))
   )
-  (wire (pts (xy 88.9 55.88) (xy 88.9 77.47))
+  (wire (pts (xy 88.9 55.88) (xy 88.9 76.2))
     (stroke (width 0) (type default) (color 0 0 0 0))
   )
@@
   )
   (wire (pts (xy 110.49 50.8) (xy 110.49 52.07))
+    (stroke (width 0) (type default) (color 0 0 0 0))
+  )
+  (wire (pts (xy 88.9 76.2) (xy 88.9 77.47))
     (stroke (width 0) (type default) (color 0 0 0 0))
   )
@@
   (symbol (lib_id "power:PWR_FLAG") (at 157.48 33.02 270) (unit 1)
     (in_bom yes) (on_board yes)
-    (property "Reference" "#FLG?" (id 0) (at 159.385 33.02 0)
+    (property "Reference" "#FLG0106" (id 0) (at 159.385 33.02 0)
       (effects (font (size 1.27 1.27)) hide)
     )
@@
   (symbol (lib_id "power:PWR_FLAG") (at 157.48 50.8 270) (unit 1)
     (in_bom yes) (on_board yes)
-    (property "Reference" "#FLG?" (id 0) (at 159.385 50.8 0)
+    (property "Reference" "#FLG0105" (id 0) (at 159.385 50.8 0)
       (effects (font (size 1.27 1.27)) hide)
     )
@@
   (symbol (lib_id "power:GND") (at 110.49 41.91 0) (unit 1)
     (in_bom yes) (on_board yes)
-    (property "Reference" "#PWR?" (id 0) (at 110.49 48.26 0)
+    (property "Reference" "#PWR0352" (id 0) (at 110.49 48.26 0)
       (effects (font (size 1.27 1.27)) hide)
     )
@@
   (symbol (lib_id "power:PWR_FLAG") (at 157.48 68.58 270) (unit 1)
     (in_bom yes) (on_board yes)
-    (property "Reference" "#FLG?" (id 0) (at 159.385 68.58 0)
+    (property "Reference" "#FLG0107" (id 0) (at 159.385 68.58 0)
       (effects (font (size 1.27 1.27)) hide)
     )
@@
   (symbol (lib_id "power:GND") (at 110.49 77.47 0) (unit 1)
     (in_bom yes) (on_board yes)
-    (property "Reference" "#PWR?" (id 0) (at 110.49 83.82 0)
+    (property "Reference" "#PWR0355" (id 0) (at 110.49 83.82 0)
       (effects (font (size 1.27 1.27)) hide)
     )
@@
   (symbol (lib_id "power:GND") (at 123.19 41.91 0) (unit 1)
     (in_bom yes) (on_board yes)
-    (property "Reference" "#PWR?" (id 0) (at 123.19 48.26 0)
+    (property "Reference" "#PWR0357" (id 0) (at 123.19 48.26 0)
       (effects (font (size 1.27 1.27)) hide)
     )
@@
   (symbol (lib_id "power:GND") (at 123.19 59.69 0) (unit 1)
     (in_bom yes) (on_board yes)
-    (property "Reference" "#PWR?" (id 0) (at 123.19 66.04 0)
+    (property "Reference" "#PWR0359" (id 0) (at 123.19 66.04 0)
       (effects (font (size 1.27 1.27)) hide)
     )
@@
   (symbol (lib_id "power:+5V") (at 157.48 33.02 0) (unit 1)
     (in_bom yes) (on_board yes)
-    (property "Reference" "#PWR?" (id 0) (at 157.48 36.83 0)
+    (property "Reference" "#PWR0360" (id 0) (at 157.48 36.83 0)
       (effects (font (size 1.27 1.27)) hide)
     )
@@
   (symbol (lib_id "power:+12V") (at 157.48 50.8 0) (unit 1)
     (in_bom yes) (on_board yes)
-    (property "Reference" "#PWR?" (id 0) (at 157.48 54.61 0)
+    (property "Reference" "#PWR0362" (id 0) (at 157.48 54.61 0)
       (effects (font (size 1.27 1.27)) hide)
     )
@@
   (symbol (lib_id "power:GND") (at 110.49 59.69 0) (unit 1)
     (in_bom yes) (on_board yes)
-    (property "Reference" "#PWR?" (id 0) (at 110.49 66.04 0)
+    (property "Reference" "#PWR0354" (id 0) (at 110.49 66.04 0)
       (effects (font (size 1.27 1.27)) hide)
     )
@@
   (symbol (lib_id "power:-12V") (at 157.48 68.58 0) (unit 1)
     (in_bom yes) (on_board yes)
-    (property "Reference" "#PWR?" (id 0) (at 157.48 66.04 0)
+    (property "Reference" "#PWR0361" (id 0) (at 157.48 66.04 0)
       (effects (font (size 1.27 1.27)) hide)
     )
@@
     (pin "1")
   )
+  (symbol (lib_id "power:PWR_FLAG") (at 88.9 76.2 90) (unit 1)
+    (in_bom yes) (on_board yes)
+    (property "Reference" "#FLG0110" (id 0) (at 86.995 76.2 0)
+      (effects (font (size 1.27 1.27)) hide)
+    )
+    (property "Value" "PWR_FLAG" (id 1) (at 81.28 76.2 90))
+    (property "Footprint" "" (id 2) (at 88.9 76.2 0)
+      (effects (font (size 1.27 1.27)) hide)
+    )
+    (property "Datasheet" "~" (id 3) (at 88.9 76.2 0)
+      (effects (font (size 1.27 1.27)) hide)
+    )
+    (pin "1")
+  )
   (symbol (lib_id "power:GND") (at 88.9 77.47 0) (unit 1)
     (in_bom yes) (on_board yes)
-    (property "Reference" "#PWR?" (id 0) (at 88.9 83.82 0)
+    (property "Reference" "#PWR0353" (id 0) (at 88.9 83.82 0)
       (effects (font (size 1.27 1.27)) hide)
     )
@@
   (symbol (lib_id "power:GND") (at 123.19 77.47 0) (unit 1)
     (in_bom yes) (on_board yes)
-    (property "Reference" "#PWR?" (id 0) (at 123.19 83.82 0)
+    (property "Reference" "#PWR0356" (id 0) (at 123.19 83.82 0)
       (effects (font (size 1.27 1.27)) hide)
     )
@@
   (symbol (lib_id "power:GND") (at 135.89 41.91 0) (unit 1)
     (in_bom yes) (on_board yes)
-    (property "Reference" "#PWR?" (id 0) (at 135.89 48.26 0)
-      (effects (font (size 1.27 1.27)) hide)
-    )
+    (property "Reference" "#PWR0358" (id 0) (at 135.89 48.26 0)
+      (effects (font (size 1.27 1.27)) hide)
+    )

Commit message: fixed some DRC errors
Parts:
- gave numbers to parts that had none: 1
Changed lines of the file:
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@@
   (symbol (lib_id "Switch:SW_SPST") (at 100.33 33.02 0) (unit 1)
     (in_bom yes) (on_board yes)
-    (property "Reference" "SW?" (id 0) (at 100.33 29.845 0))
+    (property "Reference" "SW1" (id 0) (at 100.33 29.845 0))
     (property "Value" "SW_SPST" (id 1) (at 100.33 35.56 0))
     (property "Footprint" "" (id 2) (at 100.33 33.02 0)

Commit message: added some mounting holes : the 3 plated holes on the south border
Parts:
- added H? (x3): 6-32, symbol Mechanical:MountingHole_Pad
Connections:
- net GND: now also H?.1, H?.1, H?.1
Other:
- note added: "Mounting holes"
Changed lines of the file:
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@@
   (junction (at 157.48 68.58) (diameter 0) (color 0 0 0 0)
   )
+  (junction (at 38.1 149.86) (diameter 0) (color 0 0 0 0)
+  )
   (junction (at 110.49 50.8) (diameter 0) (color 0 0 0 0)
   )
@@
   )
   (junction (at 157.48 50.8) (diameter 0) (color 0 0 0 0)
+  )
+  (junction (at 50.8 149.86) (diameter 0) (color 0 0 0 0)
   )
   (no_connect (at 53.34 52.07))
@@
     (stroke (width 0) (type default) (color 0 0 0 0))
   )
+  (wire (pts (xy 50.8 149.86) (xy 63.5 149.86))
+    (stroke (width 0) (type default) (color 0 0 0 0))
+  )
   (wire (pts (xy 135.89 33.02) (xy 135.89 34.29))
     (stroke (width 0) (type default) (color 0 0 0 0))
@@
     (stroke (width 0) (type default) (color 0 0 0 0))
   )
+  (wire (pts (xy 38.1 152.4) (xy 38.1 149.86))
+    (stroke (width 0) (type default) (color 0 0 0 0))
+  )
   (wire (pts (xy 92.71 33.02) (xy 95.25 33.02))
     (stroke (width 0) (type default) (color 0 0 0 0))
@@
     (stroke (width 0) (type default) (color 0 0 0 0))
   )
+  (wire (pts (xy 63.5 149.86) (xy 63.5 143.51))
+    (stroke (width 0) (type default) (color 0 0 0 0))
+  )
   (wire (pts (xy 110.49 68.58) (xy 123.19 68.58))
     (stroke (width 0) (type default) (color 0 0 0 0))
@@
     (stroke (width 0) (type default) (color 0 0 0 0))
   )
+  (wire (pts (xy 38.1 149.86) (xy 50.8 149.86))
+    (stroke (width 0) (type default) (color 0 0 0 0))
+  )
   (wire (pts (xy 123.19 68.58) (xy 157.48 68.58))
     (stroke (width 0) (type default) (color 0 0 0 0))
@@
     (stroke (width 0) (type default) (color 0 0 0 0))
   )
+  (wire (pts (xy 50.8 143.51) (xy 50.8 149.86))
+    (stroke (width 0) (type default) (color 0 0 0 0))
+  )
   (wire (pts (xy 87.63 53.34) (xy 92.71 53.34))
     (stroke (width 0) (type default) (color 0 0 0 0))
@@
   )
   (wire (pts (xy 45.72 40.64) (xy 45.72 44.45))
+    (stroke (width 0) (type default) (color 0 0 0 0))
+  )
+  (wire (pts (xy 38.1 143.51) (xy 38.1 149.86))
     (stroke (width 0) (type default) (color 0 0 0 0))
   )
@@
   (text "GND" (at 64.77 55.88 0)
     (effects (font (size 1.27 1.27)) (justify left bottom))
+  )
+  (text "Mounting holes" (at 85.09 114.3 0)
+    (effects (font (size 2 2)) (justify left bottom))
   )
   (text "-12V" (at 64.77 53.34 0)
@@
     (pin "1")
   )
+  (symbol (lib_id "Mechanical:MountingHole_Pad") (at 50.8 140.97 0) (unit 1)
+    (in_bom yes) (on_board yes)
+    (property "Reference" "H?" (id 0) (at 50.8 134.62 0))
+    (property "Value" "6-32" (id 1) (at 50.8 136.525 0))
+    (property "Footprint" "" (id 2) (at 50.8 140.97 0)
+      (effects (font (size 1.27 1.27)) hide)
+    )
+    (property "Datasheet" "~" (id 3) (at 50.8 140.97 0)
+      (effects (font (size 1.27 1.27)) hide)
+    )
+    (pin "1")
+  )
+  (symbol (lib_id "Mechanical:MountingHole_Pad") (at 38.1 140.97 0) (unit 1)
+    (in_bom yes) (on_board yes)
+    (property "Reference" "H?" (id 0) (at 38.1 134.62 0))
+    (property "Value" "6-32" (id 1) (at 38.1 136.525 0))
+    (property "Footprint" "" (id 2) (at 38.1 140.97 0)
+      (effects (font (size 1.27 1.27)) hide)
+    )
+    (property "Datasheet" "~" (id 3) (at 38.1 140.97 0)
+      (effects (font (size 1.27 1.27)) hide)
+    )
+    (pin "1")
+  )
   (symbol (lib_id "Device:C_Small") (at 123.19 54.61 0) (unit 1)
     (in_bom yes) (on_board yes)
@@
     (pin "1")
   )
+  (symbol (lib_id "power:GND") (at 38.1 152.4 0) (unit 1)
+    (in_bom yes) (on_board yes)
+    (property "Reference" "#PWR?" (id 0) (at 38.1 158.75 0)
+      (effects (font (size 1.27 1.27)) hide)
+    )
+    (property "Value" "GND" (id 1) (at 38.1 156.21 0))
+    (property "Footprint" "" (id 2) (at 38.1 152.4 0)
+      (effects (font (size 1.27 1.27)) hide)
+    )
+    (property "Datasheet" "" (id 3) (at 38.1 152.4 0)
+      (effects (font (size 1.27 1.27)) hide)
+    )
+    (pin "1")
+  )
   (symbol (lib_id "power:-12V") (at 157.48 68.58 0) (unit 1)
     (in_bom yes) (on_board yes)
@@
       (effects (font (size 1.27 1.27)) hide)
     )
+    (pin "1")
+  )
+  (symbol (lib_id "Mechanical:MountingHole_Pad") (at 63.5 140.97 0) (unit 1)
+    (in_bom yes) (on_board yes)
+    (property "Reference" "H?" (id 0) (at 63.5 134.62 0))
+    (property "Value" "6-32" (id 1) (at 63.5 136.525 0))
+    (property "Footprint" "" (id 2) (at 63.5 140.97 0)
+      (effects (font (size 1.27 1.27)) hide)
+    )
+    (property "Datasheet" "~" (id 3) (at 63.5 140.97 0)
+      (effects (font (size 1.27 1.27)) hide)
+    )

Commit message: name the declared mounting holes
Parts:
- gave numbers to parts that had none: 3
Other:
- note added: "South border, screws go through"
Changed lines of the file:
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@@
+    (effects (font (size 1.27 1.27)) (justify left bottom))
+  )
+  (text "South border, screws go through" (at 44.45 130.81 0)
     (effects (font (size 1.27 1.27)) (justify left bottom))
   )
@@
   (symbol (lib_id "Mechanical:MountingHole_Pad") (at 50.8 140.97 0) (unit 1)
     (in_bom yes) (on_board yes)
-    (property "Reference" "H?" (id 0) (at 50.8 134.62 0))
+    (property "Reference" "H2" (id 0) (at 50.8 134.62 0))
     (property "Value" "6-32" (id 1) (at 50.8 136.525 0))
     (property "Footprint" "" (id 2) (at 50.8 140.97 0)
@@
   (symbol (lib_id "Mechanical:MountingHole_Pad") (at 38.1 140.97 0) (unit 1)
     (in_bom yes) (on_board yes)
-    (property "Reference" "H?" (id 0) (at 38.1 134.62 0))
+    (property "Reference" "H1" (id 0) (at 38.1 134.62 0))
     (property "Value" "6-32" (id 1) (at 38.1 136.525 0))
     (property "Footprint" "" (id 2) (at 38.1 140.97 0)
@@
   (symbol (lib_id "power:GND") (at 38.1 152.4 0) (unit 1)
     (in_bom yes) (on_board yes)
-    (property "Reference" "#PWR?" (id 0) (at 38.1 158.75 0)
+    (property "Reference" "#PWR0397" (id 0) (at 38.1 158.75 0)
       (effects (font (size 1.27 1.27)) hide)
     )
@@
   (symbol (lib_id "Mechanical:MountingHole_Pad") (at 63.5 140.97 0) (unit 1)
     (in_bom yes) (on_board yes)
-    (property "Reference" "H?" (id 0) (at 63.5 134.62 0))
+    (property "Reference" "H3" (id 0) (at 63.5 134.62 0))
     (property "Value" "6-32" (id 1) (at 63.5 136.525 0))
     (property "Footprint" "" (id 2) (at 63.5 140.97 0)

Commit message: assigning footprints
Parts:
- H1, H2, H3: footprint (none) -> MountingHole:MountingHole_3.7mm_Pad_Via
Changed lines of the file:
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@@
     (property "Reference" "H2" (id 0) (at 50.8 134.62 0))
     (property "Value" "6-32" (id 1) (at 50.8 136.525 0))
-    (property "Footprint" "" (id 2) (at 50.8 140.97 0)
+    (property "Footprint" "MountingHole:MountingHole_3.7mm_Pad_Via" (id 2) (at 50.8 140.97 0)
       (effects (font (size 1.27 1.27)) hide)
     )
@@
     (property "Reference" "H1" (id 0) (at 38.1 134.62 0))
     (property "Value" "6-32" (id 1) (at 38.1 136.525 0))
-    (property "Footprint" "" (id 2) (at 38.1 140.97 0)
+    (property "Footprint" "MountingHole:MountingHole_3.7mm_Pad_Via" (id 2) (at 38.1 140.97 0)
       (effects (font (size 1.27 1.27)) hide)
     )
@@
     (property "Reference" "H3" (id 0) (at 63.5 134.62 0))
     (property "Value" "6-32" (id 1) (at 63.5 136.525 0))
-    (property "Footprint" "" (id 2) (at 63.5 140.97 0)
+    (property "Footprint" "MountingHole:MountingHole_3.7mm_Pad_Via" (id 2) (at 63.5 140.97 0)
       (effects (font (size 1.27 1.27)) hide)
     )
