File: subsheet_105.kicad_sch (KiCad schematic)
At the start: 13 parts, among them J9 DIN-7 POWER, SW1 SW_SPST

Commit message: assigned footprint for all remaining standard passives
Parts:
- C106: footprint (none) -> Capacitor_THT:CP_Radial_D10.0mm_P5.00mm
Changed lines of the file:
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@@
       (effects (font (size 1.27 1.27)) (justify left))
     )
-    (property "Footprint" "" (id 2) (at 135.89 36.83 0)
+    (property "Footprint" "Capacitor_THT:CP_Radial_D10.0mm_P5.00mm" (id 2) (at 135.89 36.83 0)
       (effects (font (size 1.27 1.27)) hide)
     )

Commit message: footprint for L3
Parts:
- L3: footprint (none) -> atari-passives_THT:4-CHANNELS-COMMON-MODE-DIP-14
Changed lines of the file:
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@@
     (property "Reference" "L3" (id 0) (at 78.74 44.45 0))
     (property "Value" "SNH19L-0601-4" (id 1) (at 78.74 59.69 0))
-    (property "Footprint" "" (id 2) (at 78.74 49.53 0)
+    (property "Footprint" "atari-passives_THT:4-CHANNELS-COMMON-MODE-DIP-14" (id 2) (at 78.74 49.53 0)
       (effects (font (size 1.27 1.27)) hide)
     )

Commit message: done assigning footprints
Parts:
- J9: footprint (none) -> atari-interconnect:receptacle-din-7-male-power
- SW1: footprint (none) -> atari-interconnect:switch-spdt-vertical-right-angle-c-k-E101J1AV2BE2
Changed lines of the file:
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@@
       (effects (font (size 1.27 1.27)) (justify right))
     )
-    (property "Footprint" "" (id 2) (at 45.72 52.07 0)
+    (property "Footprint" "atari-interconnect:receptacle-din-7-male-power" (id 2) (at 45.72 52.07 0)
       (effects (font (size 1.27 1.27)) hide)
     )
@@
     (property "Reference" "SW1" (id 0) (at 100.33 29.845 0))
     (property "Value" "SW_SPST" (id 1) (at 100.33 35.56 0))
-    (property "Footprint" "" (id 2) (at 100.33 33.02 0)
+    (property "Footprint" "atari-interconnect:switch-spdt-vertical-right-angle-c-k-E101J1AV2BE2" (id 2) (at 100.33 33.02 0)
       (effects (font (size 1.27 1.27)) hide)
     )
