File: subsheet_101.kicad_sch (KiCad schematic)
At the start: 21 parts, among them J11 Mouse / Joy 0, J12 Joy 1, J12 Keyboard, U21 MC6850_PHY

Commit message: fixed : acia connexion to address bus and to data bus
Connections:
- net D0 renamed D8
- net D1 renamed D9
- net D2 renamed D10
- net D3 renamed D11
- net D4 renamed D12
- net D5 renamed D13
- net D6 renamed D14
- net D7 renamed D15
Changed lines of the file:
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@@
   (title_block
     (title "Converted schematics of Atari 260/520 ST")
-    (date "2023-04-19")
+    (date "2023-04-20")
     (rev "0")
     (comment 1 "…sporniket/kicad-conversions--atari-260-520-st-motherboard--c070231")
@@
     (effects (font (size 1.27 1.27)) (justify left bottom))
   )
-  (label "D3" (at 144.78 50.8 180)
-    (effects (font (size 1.27 1.27)) (justify right bottom))
-  )
-  (label "D0" (at 144.78 43.18 180)
+  (label "D9" (at 144.78 45.72 180)
+    (effects (font (size 1.27 1.27)) (justify right bottom))
+  )
+  (label "D14" (at 144.78 58.42 180)
     (effects (font (size 1.27 1.27)) (justify right bottom))
   )
@@
     (effects (font (size 1.27 1.27)) (justify left bottom))
   )
-  (label "D1" (at 144.78 45.72 180)
+  (label "D12" (at 144.78 53.34 180)
     (effects (font (size 1.27 1.27)) (justify right bottom))
   )
@@
     (effects (font (size 1.27 1.27)) (justify left bottom))
   )
-  (label "D6" (at 144.78 58.42 180)
-    (effects (font (size 1.27 1.27)) (justify right bottom))
-  )
-  (label "D2" (at 144.78 48.26 180)
-    (effects (font (size 1.27 1.27)) (justify right bottom))
-  )
   (label "A2" (at 92.71 58.42 0)
     (effects (font (size 1.27 1.27)) (justify left bottom))
   )
-  (label "D7" (at 144.78 60.96 180)
+  (label "D11" (at 144.78 50.8 180)
     (effects (font (size 1.27 1.27)) (justify right bottom))
   )
@@
     (effects (font (size 1.27 1.27)) (justify right bottom))
   )
-  (label "D4" (at 144.78 53.34 180)
+  (label "D15" (at 144.78 60.96 180)
     (effects (font (size 1.27 1.27)) (justify right bottom))
   )
@@
     (effects (font (size 1.27 1.27)) (justify right bottom))
   )
-  (label "D5" (at 144.78 55.88 180)
+  (label "D8" (at 144.78 43.18 180)
     (effects (font (size 1.27 1.27)) (justify right bottom))
   )
@@
     (effects (font (size 1.27 1.27)) (justify left bottom))
   )
+  (label "D10" (at 144.78 48.26 180)
+    (effects (font (size 1.27 1.27)) (justify right bottom))
+  )
+  (label "D13" (at 144.78 55.88 180)
+    (effects (font (size 1.27 1.27)) (justify right bottom))
+  )
   (global_label "N6850" (shape input) (at 92.71 55.88 180) (fields_autoplaced)
