File: subsheet_101.kicad_sch (KiCad schematic)
At the start: 21 parts, among them J11 Mouse / Joy 0, J12 Joy 1, J12 Keyboard, U21 MC6850_PHY

Commit message: fixed some DRC errors
Parts:
- renumbered J12 to J10
Changed lines of the file:
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@@
     (comment 4 "Reference : C070231")
   )
-  (junction (at 85.09 60.96) (diameter 0) (color 0 0 0 0)
-  )
   (junction (at 99.06 43.18) (diameter 0) (color 0 0 0 0)
   )
   (junction (at 97.79 72.39) (diameter 0) (color 0 0 0 0)
+  )
+  (junction (at 97.79 66.04) (diameter 0) (color 0 0 0 0)
+  )
+  (junction (at 82.55 60.96) (diameter 0) (color 0 0 0 0)
   )
   (junction (at 55.88 106.68) (diameter 0) (color 0 0 0 0)
@@
     (stroke (width 0) (type default) (color 0 0 0 0))
   )
-  (wire (pts (xy 85.09 60.96) (xy 101.6 60.96))
+  (wire (pts (xy 82.55 60.96) (xy 101.6 60.96))
     (stroke (width 0) (type default) (color 0 0 0 0))
   )
@@
     (stroke (width 0) (type default) (color 0 0 0 0))
   )
-  (wire (pts (xy 85.09 60.96) (xy 85.09 72.39))
+  (wire (pts (xy 82.55 60.96) (xy 82.55 72.39))
     (stroke (width 0) (type default) (color 0 0 0 0))
   )
@@
     (stroke (width 0) (type default) (color 0 0 0 0))
   )
-  (wire (pts (xy 76.2 60.96) (xy 85.09 60.96))
+  (wire (pts (xy 76.2 60.96) (xy 82.55 60.96))
     (stroke (width 0) (type default) (color 0 0 0 0))
   )
@@
     (stroke (width 0) (type default) (color 0 0 0 0))
   )
-  (wire (pts (xy 85.09 72.39) (xy 90.17 72.39))
+  (wire (pts (xy 82.55 72.39) (xy 90.17 72.39))
     (stroke (width 0) (type default) (color 0 0 0 0))
   )
@@
   (symbol (lib_id "power:GND") (at 109.22 97.79 0) (unit 1)
     (in_bom yes) (on_board yes)
-    (property "Reference" "#PWR?" (id 0) (at 109.22 104.14 0)
+    (property "Reference" "#PWR0252" (id 0) (at 109.22 104.14 0)
       (effects (font (size 1.27 1.27)) hide)
     )
@@
   (symbol (lib_id "power:GND") (at 124.46 87.63 0) (unit 1)
     (in_bom yes) (on_board yes)
-    (property "Reference" "#PWR?" (id 0) (at 124.46 93.98 0)
+    (property "Reference" "#PWR0270" (id 0) (at 124.46 93.98 0)
       (effects (font (size 1.27 1.27)) hide)
     )
@@
   (symbol (lib_id "power:GND") (at 152.4 38.1 0) (unit 1)
     (in_bom yes) (on_board yes)
-    (property "Reference" "#PWR?" (id 0) (at 152.4 44.45 0)
+    (property "Reference" "#PWR0269" (id 0) (at 152.4 44.45 0)
       (effects (font (size 1.27 1.27)) hide)
     )
@@
   (symbol (lib_id "power:GND") (at 71.12 172.72 0) (unit 1)
     (in_bom yes) (on_board yes)
-    (property "Reference" "#PWR?" (id 0) (at 71.12 179.07 0)
+    (property "Reference" "#PWR0261" (id 0) (at 71.12 179.07 0)
       (effects (font (size 1.27 1.27)) hide)
     )
@@
   (symbol (lib_id "power:GND") (at 71.12 215.9 0) (unit 1)
     (in_bom yes) (on_board yes)
-    (property "Reference" "#PWR?" (id 0) (at 71.12 222.25 0)
+    (property "Reference" "#PWR0265" (id 0) (at 71.12 222.25 0)
       (effects (font (size 1.27 1.27)) hide)
     )
@@
   (symbol (lib_id "power:+5V") (at 76.2 60.96 0) (unit 1)
     (in_bom yes) (on_board yes)
-    (property "Reference" "#PWR?" (id 0) (at 76.2 64.77 0)
+    (property "Reference" "#PWR0259" (id 0) (at 76.2 64.77 0)
       (effects (font (size 1.27 1.27)) hide)
     )
@@
   (symbol (lib_id "power:GND") (at 86.36 246.38 0) (unit 1)
     (in_bom yes) (on_board yes)
-    (property "Reference" "#PWR?" (id 0) (at 86.36 252.73 0)
+    (property "Reference" "#PWR0266" (id 0) (at 86.36 252.73 0)
       (effects (font (size 1.27 1.27)) hide)
     )
@@
   (symbol (lib_id "power:GND") (at 71.12 152.4 0) (unit 1)
     (in_bom yes) (on_board yes)
-    (property "Reference" "#PWR?" (id 0) (at 71.12 158.75 0)
+    (property "Reference" "#PWR0255" (id 0) (at 71.12 158.75 0)
       (effects (font (size 1.27 1.27)) hide)
     )
@@
     (pin "1")
   )
+  (symbol (lib_id "power:PWR_FLAG") (at 97.79 66.04 90) (unit 1)
+    (in_bom yes) (on_board yes)
+    (property "Reference" "#FLG0111" (id 0) (at 95.885 66.04 0)
+      (effects (font (size 1.27 1.27)) hide)
+    )
+    (property "Value" "PWR_FLAG" (id 1) (at 90.17 66.04 90))
+    (property "Footprint" "" (id 2) (at 97.79 66.04 0)
+      (effects (font (size 1.27 1.27)) hide)
+    )
+    (property "Datasheet" "~" (id 3) (at 97.79 66.04 0)
+      (effects (font (size 1.27 1.27)) hide)
+    )
+    (pin "1")
+  )
   (symbol (lib_id "power:GND") (at 88.9 35.56 0) (unit 1)
     (in_bom yes) (on_board yes)
-    (property "Reference" "#PWR?" (id 0) (at 88.9 41.91 0)
+    (property "Reference" "#PWR0258" (id 0) (at 88.9 41.91 0)
       (effects (font (size 1.27 1.27)) hide)
     )
@@
   (symbol (lib_id "power:+5V") (at 55.88 96.52 0) (unit 1)
     (in_bom yes) (on_board yes)
-    (property "Reference" "#PWR?" (id 0) (at 55.88 100.33 0)
+    (property "Reference" "#PWR0251" (id 0) (at 55.88 100.33 0)
       (effects (font (size 1.27 1.27)) hide)
     )
@@
   (symbol (lib_id "power:GND") (at 71.12 132.08 0) (unit 1)
     (in_bom yes) (on_board yes)
-    (property "Reference" "#PWR?" (id 0) (at 71.12 138.43 0)
+    (property "Reference" "#PWR0257" (id 0) (at 71.12 138.43 0)
       (effects (font (size 1.27 1.27)) hide)
     )
@@
   (symbol (lib_id "power:GND") (at 86.36 142.24 0) (unit 1)
     (in_bom yes) (on_board yes)
-    (property "Reference" "#PWR?" (id 0) (at 86.36 148.59 0)
+    (property "Reference" "#PWR0249" (id 0) (at 86.36 148.59 0)
       (effects (font (size 1.27 1.27)) hide)
     )
@@
   (symbol (lib_id "power:GND") (at 59.69 223.52 0) (unit 1)
     (in_bom yes) (on_board yes)
-    (property "Reference" "#PWR?" (id 0) (at 59.69 229.87 0)
+    (property "Reference" "#PWR0260" (id 0) (at 59.69 229.87 0)
       (effects (font (size 1.27 1.27)) hide)
     )
@@
   (symbol (lib_id "power:GND") (at 86.36 205.74 0) (unit 1)
     (in_bom yes) (on_board yes)
-    (property "Reference" "#PWR?" (id 0) (at 86.36 212.09 0)
+    (property "Reference" "#PWR0264" (id 0) (at 86.36 212.09 0)
       (effects (font (size 1.27 1.27)) hide)
     )
@@
   (symbol (lib_id "power:GND") (at 168.91 139.7 0) (unit 1)
     (in_bom yes) (on_board yes)
-    (property "Reference" "#PWR?" (id 0) (at 168.91 146.05 0)
+    (property "Reference" "#PWR0250" (id 0) (at 168.91 146.05 0)
       (effects (font (size 1.27 1.27)) hide)
     )
@@
   (symbol (lib_id "power:GND") (at 55.88 116.84 0) (unit 1)
     (in_bom yes) (on_board yes)
-    (property "Reference" "#PWR?" (id 0) (at 55.88 123.19 0)
+    (property "Reference" "#PWR0254" (id 0) (at 55.88 123.19 0)
       (effects (font (size 1.27 1.27)) hide)
     )
@@
   (symbol (lib_id "power:GND") (at 55.88 158.75 0) (unit 1)
     (in_bom yes) (on_board yes)
-    (property "Reference" "#PWR?" (id 0) (at 55.88 165.1 0)
+    (property "Reference" "#PWR0256" (id 0) (at 55.88 165.1 0)
       (effects (font (size 1.27 1.27)) hide)
     )
@@
   (symbol (lib_id "Connector:DB9_Male") (at 43.18 220.98 180) (unit 1)
     (in_bom yes) (on_board yes)
-    (property "Reference" "J12" (id 0) (at 43.18 234.95 0))
+    (property "Reference" "J10" (id 0) (at 43.18 234.95 0))
     (property "Value" "Joy 1" (id 1) (at 43.18 206.375 0))
     (property "Footprint" "" (id 2) (at 43.18 220.98 0)
@@
   (symbol (lib_id "power:GND") (at 71.12 236.22 0) (unit 1)
     (in_bom yes) (on_board yes)
-    (property "Reference" "#PWR?" (id 0) (at 71.12 242.57 0)
+    (property "Reference" "#PWR0267" (id 0) (at 71.12 242.57 0)
       (effects (font (size 1.27 1.27)) hide)
     )
@@
   (symbol (lib_id "power:GND") (at 86.36 162.56 0) (unit 1)
     (in_bom yes) (on_board yes)
-    (property "Reference" "#PWR?" (id 0) (at 86.36 168.91 0)
+    (property "Reference" "#PWR0262" (id 0) (at 86.36 168.91 0)
       (effects (font (size 1.27 1.27)) hide)
     )
@@
   (symbol (lib_id "power:GND") (at 111.76 72.39 0) (unit 1)
     (in_bom yes) (on_board yes)
-    (property "Reference" "#PWR?" (id 0) (at 111.76 78.74 0)
+    (property "Reference" "#PWR0253" (id 0) (at 111.76 78.74 0)
       (effects (font (size 1.27 1.27)) hide)
     )
@@
   (symbol (lib_id "power:GND") (at 71.12 195.58 0) (unit 1)
     (in_bom yes) (on_board yes)
-    (property "Reference" "#PWR?" (id 0) (at 71.12 201.93 0)
+    (property "Reference" "#PWR0263" (id 0) (at 71.12 201.93 0)
       (effects (font (size 1.27 1.27)) hide)
     )
@@
   (symbol (lib_id "power:GND") (at 86.36 226.06 0) (unit 1)
     (in_bom yes) (on_board yes)
-    (property "Reference" "#PWR?" (id 0) (at 86.36 232.41 0)
-      (effects (font (size 1.27 1.27)) hide)
-    )
+    (property "Reference" "#PWR0268" (id 0) (at 86.36 232.41 0)
+      (effects (font (size 1.27 1.27)) hide)
+    )

Commit message: fixed symbols causing DRC errors, fixed renamed symbol 'FerriteBead_small'
Parts:
- L27, L30: symbol Device:Ferrite_Bead_Small -> Device:FerriteBead_Small
Changed lines of the file:
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@@
     (pin "1")
   )
-  (symbol (lib_id "Device:Ferrite_Bead_Small") (at 92.71 72.39 270) (unit 1)
+  (symbol (lib_id "Device:FerriteBead_Small") (at 92.71 72.39 270) (unit 1)
     (in_bom yes) (on_board yes)
     (property "Reference" "L27" (id 0) (at 86.36 71.12 90)
@@
     (pin "2")
   )
-  (symbol (lib_id "Device:Ferrite_Bead_Small") (at 55.88 101.6 180) (unit 1)
+  (symbol (lib_id "Device:FerriteBead_Small") (at 55.88 101.6 180) (unit 1)
     (in_bom yes) (on_board yes)
     (property "Reference" "L30" (id 0) (at 58.42 100.33 0)

Commit message: assigned footprint for all remaining standard passives
Parts:
- L10, L12, L13, L14, L15, L16, L5, L6, L7, L8, L9, L91, L92: footprint (none) -> commons-passives_THT:Passive_THT_EMI_filter_W5.08mm_L7.62mm
Changed lines of the file:
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@@
       (effects (font (size 1.27 1.27)) (justify left))
     )
-    (property "Footprint" "" (id 2) (at 71.12 129.54 90)
+    (property "Footprint" "commons-passives_THT:Passive_THT_EMI_filter_W5.08mm_L7.62mm" (id 2) (at 71.12 129.54 90)
       (effects (font (size 1.27 1.27)) hide)
     )
@@
       (effects (font (size 1.27 1.27)) (justify left))
     )
-    (property "Footprint" "" (id 2) (at 86.36 139.7 90)
+    (property "Footprint" "commons-passives_THT:Passive_THT_EMI_filter_W5.08mm_L7.62mm" (id 2) (at 86.36 139.7 90)
       (effects (font (size 1.27 1.27)) hide)
     )
@@
       (effects (font (size 1.27 1.27)) (justify left))
     )
-    (property "Footprint" "" (id 2) (at 86.36 223.52 90)
+    (property "Footprint" "commons-passives_THT:Passive_THT_EMI_filter_W5.08mm_L7.62mm" (id 2) (at 86.36 223.52 90)
       (effects (font (size 1.27 1.27)) hide)
     )
@@
       (effects (font (size 1.27 1.27)) (justify left))
     )
-    (property "Footprint" "" (id 2) (at 86.36 160.02 90)
+    (property "Footprint" "commons-passives_THT:Passive_THT_EMI_filter_W5.08mm_L7.62mm" (id 2) (at 86.36 160.02 90)
       (effects (font (size 1.27 1.27)) hide)
     )
@@
       (effects (font (size 1.27 1.27)) (justify left))
     )
-    (property "Footprint" "" (id 2) (at 109.22 95.25 90)
+    (property "Footprint" "commons-passives_THT:Passive_THT_EMI_filter_W5.08mm_L7.62mm" (id 2) (at 109.22 95.25 90)
       (effects (font (size 1.27 1.27)) hide)
     )
@@
       (effects (font (size 1.27 1.27)) (justify left))
     )
-    (property "Footprint" "" (id 2) (at 71.12 149.86 90)
+    (property "Footprint" "commons-passives_THT:Passive_THT_EMI_filter_W5.08mm_L7.62mm" (id 2) (at 71.12 149.86 90)
       (effects (font (size 1.27 1.27)) hide)
     )
@@
       (effects (font (size 1.27 1.27)) (justify left))
     )
-    (property "Footprint" "" (id 2) (at 71.12 193.04 90)
+    (property "Footprint" "commons-passives_THT:Passive_THT_EMI_filter_W5.08mm_L7.62mm" (id 2) (at 71.12 193.04 90)
       (effects (font (size 1.27 1.27)) hide)
     )
@@
       (effects (font (size 1.27 1.27)) (justify left))
     )
-    (property "Footprint" "" (id 2) (at 71.12 170.18 90)
+    (property "Footprint" "commons-passives_THT:Passive_THT_EMI_filter_W5.08mm_L7.62mm" (id 2) (at 71.12 170.18 90)
       (effects (font (size 1.27 1.27)) hide)
     )
@@
       (effects (font (size 1.27 1.27)) (justify left))
     )
-    (property "Footprint" "" (id 2) (at 71.12 213.36 90)
+    (property "Footprint" "commons-passives_THT:Passive_THT_EMI_filter_W5.08mm_L7.62mm" (id 2) (at 71.12 213.36 90)
       (effects (font (size 1.27 1.27)) hide)
     )
@@
       (effects (font (size 1.27 1.27)) (justify left))
     )
-    (property "Footprint" "" (id 2) (at 71.12 233.68 90)
+    (property "Footprint" "commons-passives_THT:Passive_THT_EMI_filter_W5.08mm_L7.62mm" (id 2) (at 71.12 233.68 90)
       (effects (font (size 1.27 1.27)) hide)
     )
@@
       (effects (font (size 1.27 1.27)) (justify left))
     )
-    (property "Footprint" "" (id 2) (at 124.46 85.09 90)
+    (property "Footprint" "commons-passives_THT:Passive_THT_EMI_filter_W5.08mm_L7.62mm" (id 2) (at 124.46 85.09 90)
       (effects (font (size 1.27 1.27)) hide)
     )
@@
       (effects (font (size 1.27 1.27)) (justify left))
     )
-    (property "Footprint" "" (id 2) (at 86.36 243.84 90)
+    (property "Footprint" "commons-passives_THT:Passive_THT_EMI_filter_W5.08mm_L7.62mm" (id 2) (at 86.36 243.84 90)
       (effects (font (size 1.27 1.27)) hide)
     )
@@
       (effects (font (size 1.27 1.27)) (justify left))
     )
-    (property "Footprint" "" (id 2) (at 86.36 203.2 90)
-      (effects (font (size 1.27 1.27)) hide)
-    )
+    (property "Footprint" "commons-passives_THT:Passive_THT_EMI_filter_W5.08mm_L7.62mm" (id 2) (at 86.36 203.2 90)
+      (effects (font (size 1.27 1.27)) hide)
+    )

Commit message: assign dsub footprints and midi ports
Parts:
- J10, J11: footprint (none) -> atari-interconnect:Joystick_Port_DSUB-9_Male_Horizontal_P2.77x2.84mm_EdgePinOffset14.56mm_Housed_MountingHolesOffset8.2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
- J12: footprint (none) -> Connector_PinHeader_2.54mm:PinHeader_1x18_P2.54mm_Vertical
Changed lines of the file:
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@@
     (property "Reference" "J11" (id 0) (at 31.75 166.37 0))
     (property "Value" "Mouse / Joy 0" (id 1) (at 31.75 137.795 0))
-    (property "Footprint" "" (id 2) (at 31.75 152.4 0)
+    (property "Footprint" "atari-interconnect:Joystick_Port_DSUB-9_Male_Horizontal_P2.77x2.84mm_EdgePinOffset14.56mm_Housed_MountingHolesOffset8.20mm" (id 2) (at 31.75 152.4 0)
       (effects (font (size 1.27 1.27)) hide)
     )
@@
     (property "Reference" "J12" (id 0) (at 177.8 139.7 0))
     (property "Value" "Keyboard" (id 1) (at 177.8 91.44 0))
-    (property "Footprint" "" (id 2) (at 177.8 116.84 0)
+    (property "Footprint" "Connector_PinHeader_2.54mm:PinHeader_1x18_P2.54mm_Vertical" (id 2) (at 177.8 116.84 0)
       (effects (font (size 1.27 1.27)) hide)
     )
@@
     (property "Reference" "J10" (id 0) (at 43.18 234.95 0))
     (property "Value" "Joy 1" (id 1) (at 43.18 206.375 0))
-    (property "Footprint" "" (id 2) (at 43.18 220.98 0)
-      (effects (font (size 1.27 1.27)) hide)
-    )
+    (property "Footprint" "atari-interconnect:Joystick_Port_DSUB-9_Male_Horizontal_P2.77x2.84mm_EdgePinOffset14.56mm_Housed_MountingHolesOffset8.20mm" (id 2) (at 43.18 220.98 0)
+      (effects (font (size 1.27 1.27)) hide)
+    )
