File: subsheet_101.kicad_sch (KiCad schematic)
At the start: 21 parts, among them J10 Joy 1, J11 Mouse / Joy 0, J12 Keyboard, U21 MC6850_PHY

Commit message: fixed power supply of U20 and U21 (ACIAs)
Connections:
- net +5VD: now reaches C24.1, L27.1, U21.12 (VCC)
Other:
- note added: "For U20 and U21"
- moved on the sheet: C92, L27, L30

Commit message: fixed U21#10 (ACIA.CS1) -- use same network than U21#12 (ACIA.VCC)
Connections:
- net +5V: no longer U21.10 (CS1)
- net +5VD: now also U21.10 (CS1)
Other:
- moved on the sheet: L27

Commit message: pcb session 2024-05-04T07:32:37+02:00 -- done MIDI to ACIA, finished HSYNC, VSYNC
Connections:
- net +5VD renamed +5F
Changed lines of the file:
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@@
   (junction (at 96.52 72.39) (diameter 0) (color 0 0 0 0)
   )
+  (junction (at 171.45 25.4) (diameter 0) (color 0 0 0 0)
+  )
   (junction (at 88.9 72.39) (diameter 0) (color 0 0 0 0)
   )
   (junction (at 99.06 43.18) (diameter 0) (color 0 0 0 0)
-  )
-  (junction (at 168.91 25.4) (diameter 0) (color 0 0 0 0)
   )
   (junction (at 139.7 38.1) (diameter 0) (color 0 0 0 0)
@@
     (stroke (width 0) (type default))
   )
-  (wire (pts (xy 168.91 25.4) (xy 177.8 25.4))
+  (wire (pts (xy 165.1 25.4) (xy 171.45 25.4))
     (stroke (width 0) (type default))
   )
@@
     (stroke (width 0) (type default))
   )
+  (wire (pts (xy 171.45 25.4) (xy 177.8 25.4))
+    (stroke (width 0) (type default))
+  )
   (wire (pts (xy 25.4 96.52) (xy 25.4 99.06))
     (stroke (width 0) (type default))
@@
   )
   (wire (pts (xy 39.37 157.48) (xy 52.07 157.48))
-    (stroke (width 0) (type default))
-  )
-  (wire (pts (xy 165.1 25.4) (xy 168.91 25.4))
     (stroke (width 0) (type default))
   )
@@
         (path "/61fe4c73-be59-4519-98f1-a634322a841d/3f88e458-4d53-4de4-ada5-f2535e8a83f8"
           (reference "#PWR0251") (unit 1)
-        )
-      )
-    )
-  )
-  (symbol (lib_id "power:+5VD") (at 168.91 25.4 0) (unit 1)
-    (in_bom yes) (on_board yes) (dnp no)
-    (property "Reference" "#PWR02" (at 168.91 29.21 0)
-      (effects (font (size 1.27 1.27)) hide)
-    )
-    (property "Value" "+5VD" (at 168.91 21.844 0)
-      (effects (font (size 1.27 1.27)))
-    )
-    (property "Footprint" "" (at 168.91 25.4 0)
-      (effects (font (size 1.27 1.27)) hide)
-    )
-    (property "Datasheet" "" (at 168.91 25.4 0)
-      (effects (font (size 1.27 1.27)) hide)
-    )
-    (pin "1")
-    (instances
-      (project "motherboard"
-        (path "/61fe4c73-be59-4519-98f1-a634322a841d/3f88e458-4d53-4de4-ada5-f2535e8a83f8"
-          (reference "#PWR02") (unit 1)
         )
       )
@@
     )
   )
-  (symbol (lib_id "power:+5VD") (at 80.01 72.39 0) (unit 1)
-    (in_bom yes) (on_board yes) (dnp no)
-    (property "Reference" "#PWR04" (at 80.01 76.2 0)
-      (effects (font (size 1.27 1.27)) hide)
-    )
-    (property "Value" "+5VD" (at 80.01 68.834 0)
+  (symbol (lib_id "power:+5F") (at 80.01 72.39 0) (unit 1)
+    (in_bom yes) (on_board yes) (dnp no)
+    (property "Reference" "#PWR02" (at 80.01 76.2 0)
+      (effects (font (size 1.27 1.27)) hide)
+    )
+    (property "Value" "+5F" (at 80.01 68.834 0)
       (effects (font (size 1.27 1.27)))
     )
@@
       (project "motherboard"
         (path "/61fe4c73-be59-4519-98f1-a634322a841d/3f88e458-4d53-4de4-ada5-f2535e8a83f8"
-          (reference "#PWR04") (unit 1)
+          (reference "#PWR02") (unit 1)
         )
       )
@@
         )
       )
+    )
+  )
+  (symbol (lib_id "power:+5F") (at 171.45 25.4 0) (unit 1)
+    (in_bom yes) (on_board yes) (dnp no)
+    (property "Reference" "#PWR05" (at 171.45 29.21 0)
+      (effects (font (size 1.27 1.27)) hide)
+    )
+    (property "Value" "+5F" (at 171.45 21.844 0)
+      (effects (font (size 1.27 1.27)))
+    )
+    (property "Footprint" "" (at 171.45 25.4 0)
+      (effects (font (size 1.27 1.27)) hide)
+    )
+    (property "Datasheet" "" (at 171.45 25.4 0)
+      (effects (font (size 1.27 1.27)) hide)
+    )
+    (pin "1")
+    (instances
+      (project "motherboard"
+        (path "/61fe4c73-be59-4519-98f1-a634322a841d/3f88e458-4d53-4de4-ada5-f2535e8a83f8"
+          (reference "#PWR05") (unit 1)
+        )
+      )
