File: subsheet_102.kicad_sch (KiCad schematic)
At the start: 10 parts, among them J7 MIDI IN, J8 MIDI OUT

Commit message: done acia and midi ports, remaining dangling pins of u35
Parts:
- removed L?: Ferrite bead, commons-passives_THT:Passive_THT_ferrite_bead_W3.81mm_L15.24mm, symbol Device:Ferrite_Bead_Small
- added R77, R78, R79, R80: 220, symbol Device:R_Small_US
- added R81: 4K7, symbol Device:R_Small_US
- gave numbers to parts that had none: 5
Connections:
- net +5V: now also C23.1, U?.12 (VCC), R77.1, R78.1, R81.1
- net GND: now also J8.2
- net at U35.3 (2A), U39.4 (VO), U?.2 (RXDAT): now also R81.2
- net at J8.1: now also R77.2
- net at J8.3: now also R80.1
- net at J8.4: now also R78.2
- net at J8.5: now also R79.1
- new net MIDI_OUT: R79.2
- new net MIDI_THROUGH: R80.2
Other:
- note added: "From U36"
- moved on the sheet: C23, C46, C59, CR7, J7, J8, U35, U39, U?

Commit message: done remaining u36
Connections:
- net GND: now also U35.11 (5A), U35.13 (6A), U35.9 (4A)
- net ACSI_PORT_INT: now reaches U35.5 (3A)
- net ACSI_INT: now reaches U35.6 (3Y)
- no-connect marks 4 -> 7
Other:
- note added: "To U40"
- moved on the sheet: C46, U35

Commit message: missing annotation for U20
Parts:
- gave numbers to parts that had none: 1
Changed lines of the file:
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@@
   (symbol (lib_id "acia:MC6850_PHY") (at 73.66 90.17 0) (unit 1)
     (in_bom yes) (on_board yes)
-    (property "Reference" "U?" (id 0) (at 73.66 69.85 0))
+    (property "Reference" "U20" (id 0) (at 73.66 69.85 0))
     (property "Value" "MC6850_PHY" (id 1) (at 73.66 72.39 0)
       (effects (font (size 1.27 1.27) bold))

Commit message: fixed : acia connexion to address bus and to data bus
Connections:
- net +5V: no longer U20.10 (CS1)
- net A2: now also U20.10 (CS1); no longer U20.9 (~{CS2})
- net GND: now also U20.9 (~{CS2})
- net D0 renamed D8
- net D1 renamed D9
- net D2 renamed D10
- net D3 renamed D11
- net D4 renamed D12
- net D5 renamed D13
- net D6 renamed D14
- net D7 renamed D15
Changed lines of the file:
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@@
   (title_block
     (title "Converted schematics of Atari 260/520 ST")
-    (date "2023-04-19")
+    (date "2023-04-20")
     (rev "0")
     (comment 1 "…sporniket/kicad-conversions--atari-260-520-st-motherboard--c070231")
@@
   )
   (junction (at 25.4 173.99) (diameter 0) (color 0 0 0 0)
-  )
-  (junction (at 39.37 99.06) (diameter 0) (color 0 0 0 0)
   )
   (junction (at 184.15 139.7) (diameter 0) (color 0 0 0 0)
@@
   (no_connect (at 181.61 132.08))
   (no_connect (at 181.61 142.24))
-  (wire (pts (xy 39.37 110.49) (xy 52.07 110.49))
-    (stroke (width 0) (type default) (color 0 0 0 0))
-  )
   (wire (pts (xy 181.61 134.62) (xy 184.15 134.62))
     (stroke (width 0) (type default) (color 0 0 0 0))
@@
     (stroke (width 0) (type default) (color 0 0 0 0))
   )
-  (wire (pts (xy 39.37 99.06) (xy 39.37 110.49))
-    (stroke (width 0) (type default) (color 0 0 0 0))
-  )
   (wire (pts (xy 46.99 91.44) (xy 55.88 91.44))
     (stroke (width 0) (type default) (color 0 0 0 0))
@@
     (stroke (width 0) (type default) (color 0 0 0 0))
   )
-  (wire (pts (xy 39.37 99.06) (xy 55.88 99.06))
-    (stroke (width 0) (type default) (color 0 0 0 0))
-  )
   (wire (pts (xy 25.4 162.56) (xy 25.4 173.99))
     (stroke (width 0) (type default) (color 0 0 0 0))
@@
     (stroke (width 0) (type default) (color 0 0 0 0))
   )
-  (wire (pts (xy 30.48 99.06) (xy 39.37 99.06))
-    (stroke (width 0) (type default) (color 0 0 0 0))
-  )
   (wire (pts (xy 184.15 144.78) (xy 190.5 144.78))
     (stroke (width 0) (type default) (color 0 0 0 0))
@@
     (stroke (width 0) (type default) (color 0 0 0 0))
   )
-  (wire (pts (xy 46.99 96.52) (xy 55.88 96.52))
+  (wire (pts (xy 39.37 96.52) (xy 55.88 96.52))
     (stroke (width 0) (type default) (color 0 0 0 0))
   )
@@
     (stroke (width 0) (type default) (color 0 0 0 0))
   )
+  (wire (pts (xy 39.37 96.52) (xy 39.37 99.06))
+    (stroke (width 0) (type default) (color 0 0 0 0))
+  )
   (bus (pts (xy 38.1 25.4) (xy 44.45 25.4))
     (stroke (width 0) (type default) (color 0 0 0 0))
@@
     (stroke (width 0) (type default) (color 0 0 0 0))
   )
+  (wire (pts (xy 48.26 110.49) (xy 52.07 110.49))
+    (stroke (width 0) (type default) (color 0 0 0 0))
+  )
   (wire (pts (xy 100.33 162.56) (xy 100.33 165.1))
     (stroke (width 0) (type default) (color 0 0 0 0))
   )
   (wire (pts (xy 184.15 139.7) (xy 184.15 144.78))
+    (stroke (width 0) (type default) (color 0 0 0 0))
+  )
+  (wire (pts (xy 46.99 99.06) (xy 55.88 99.06))
     (stroke (width 0) (type default) (color 0 0 0 0))
   )
@@
     (effects (font (size 1.27 1.27)) (justify right bottom))
   )
-  (label "D6" (at 99.06 96.52 180)
-    (effects (font (size 1.27 1.27)) (justify right bottom))
-  )
-  (label "D5" (at 99.06 93.98 180)
-    (effects (font (size 1.27 1.27)) (justify right bottom))
-  )
-  (label "D3" (at 99.06 88.9 180)
-    (effects (font (size 1.27 1.27)) (justify right bottom))
-  )
-  (label "D4" (at 99.06 91.44 180)
-    (effects (font (size 1.27 1.27)) (justify right bottom))
-  )
-  (label "D2" (at 99.06 86.36 180)
+  (label "D12" (at 99.06 91.44 180)
+    (effects (font (size 1.27 1.27)) (justify right bottom))
+  )
+  (label "D10" (at 99.06 86.36 180)
+    (effects (font (size 1.27 1.27)) (justify right bottom))
+  )
+  (label "D8" (at 99.06 81.28 180)
+    (effects (font (size 1.27 1.27)) (justify right bottom))
+  )
+  (label "D15" (at 99.06 99.06 180)
+    (effects (font (size 1.27 1.27)) (justify right bottom))
+  )
+  (label "D13" (at 99.06 93.98 180)
     (effects (font (size 1.27 1.27)) (justify right bottom))
   )
@@
     (effects (font (size 1.27 1.27)) (justify left bottom))
   )
+  (label "D11" (at 99.06 88.9 180)
+    (effects (font (size 1.27 1.27)) (justify right bottom))
+  )
   (label "D[0..15]" (at 69.85 25.4 180)
     (effects (font (size 1.27 1.27)) (justify right bottom))
   )
-  (label "A2" (at 46.99 96.52 0)
+  (label "A2" (at 46.99 99.06 0)
     (effects (font (size 1.27 1.27)) (justify left bottom))
   )
-  (label "D7" (at 99.06 99.06 180)
-    (effects (font (size 1.27 1.27)) (justify right bottom))
-  )
-  (label "D1" (at 99.06 83.82 180)
-    (effects (font (size 1.27 1.27)) (justify right bottom))
-  )
-  (label "D0" (at 99.06 81.28 180)
+  (label "D14" (at 99.06 96.52 180)
     (effects (font (size 1.27 1.27)) (justify right bottom))
   )
   (label "A1" (at 46.99 101.6 0)
     (effects (font (size 1.27 1.27)) (justify left bottom))
+  )
+  (label "D9" (at 99.06 83.82 180)
+    (effects (font (size 1.27 1.27)) (justify right bottom))
   )
   (global_label "DATA[0..15]" (shape bidirectional) (at 76.2 25.4 0) (fields_autoplaced)
@@
     (pin "5")
   )
-  (symbol (lib_id "power:+5V") (at 30.48 99.06 0) (unit 1)
+  (symbol (lib_id "power:+5V") (at 48.26 110.49 0) (unit 1)
     (in_bom yes) (on_board yes)
-    (property "Reference" "#PWR?" (id 0) (at 30.48 102.87 0)
-      (effects (font (size 1.27 1.27)) hide)
-    )
-    (property "Value" "+5V" (id 1) (at 30.48 95.504 0))
-    (property "Footprint" "" (id 2) (at 30.48 99.06 0)
-      (effects (font (size 1.27 1.27)) hide)
-    )
-    (property "Datasheet" "" (id 3) (at 30.48 99.06 0)
-      (effects (font (size 1.27 1.27)) hide)
-    )
+    (property "Reference" "#PWR?" (id 0) (at 48.26 114.3 0)
+      (effects (font (size 1.27 1.27)) hide)
+    )
+    (property "Value" "+5V" (id 1) (at 48.26 106.934 0))
+    (property "Footprint" "" (id 2) (at 48.26 110.49 0)
+      (effects (font (size 1.27 1.27)) hide)
+    )
+    (property "Datasheet" "" (id 3) (at 48.26 110.49 0)
+      (effects (font (size 1.27 1.27)) hide)
+    )
+    (pin "1")
+  )
+  (symbol (lib_id "power:GND") (at 39.37 99.06 0) (unit 1)
+    (in_bom yes) (on_board yes)
+    (property "Reference" "#PWR?" (id 0) (at 39.37 105.41 0)
+      (effects (font (size 1.27 1.27)) hide)
+    )
+    (property "Value" "GND" (id 1) (at 39.37 102.87 0))
+    (property "Footprint" "" (id 2) (at 39.37 99.06 0)
+      (effects (font (size 1.27 1.27)) hide)
+    )
+    (property "Datasheet" "" (id 3) (at 39.37 99.06 0)
+      (effects (font (size 1.27 1.27)) hide)
+    )
