File: subsheet_102.kicad_sch (KiCad schematic)
At the start: 14 parts, among them J7 MIDI IN, J8 MIDI OUT, U20 MC6850_PHY, U35 74LS04_PHY, U39 PC900_PHY

Commit message: finition de la fiche, rajout de pwr_flag sur presque tous les points filtrés
Other:
- note added: "From J2"
Changed lines of the file:
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@@
+    (effects (font (size 1.27 1.27)) (justify right bottom))
+  )
+  (text "From J2" (at 125.73 138.43 180)
     (effects (font (size 1.27 1.27)) (justify right bottom))
   )

Commit message: complete hsync to line_phase for modulator
Connections:
- net GND: no longer U35.9 (4A)
- net LINE_PHASE: now reaches U35.8 (4Y)
- new net HSYNC: U35.9 (4A)
- no-connect marks 7 -> 6
Other:
- note added: "To U41"
- moved on the sheet: C46, U35

Commit message: use grounded midi connectors
Parts:
- J7, J8: symbol Connector:DIN-5_180degree -> connectors_with_ground:DIN-5_180degree_GND
Connections:
- net GND: now also J7.0, J8.0
Changed lines of the file:
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@@
+    (stroke (width 0) (type default) (color 0 0 0 0))
+  )
+  (wire (pts (xy 22.86 195.58) (xy 22.86 193.04))
     (stroke (width 0) (type default) (color 0 0 0 0))
   )
@@
     (stroke (width 0) (type default) (color 0 0 0 0))
   )
+  (wire (pts (xy 173.99 185.42) (xy 173.99 181.61))
+    (stroke (width 0) (type default) (color 0 0 0 0))
+  )
   (wire (pts (xy 165.1 134.62) (xy 165.1 135.89))
     (stroke (width 0) (type default) (color 0 0 0 0))
@@
     (stroke (width 0) (type default) (color 0 0 0 0))
   )
+  (wire (pts (xy 173.99 181.61) (xy 177.8 181.61))
+    (stroke (width 0) (type default) (color 0 0 0 0))
+  )
   (wire (pts (xy 142.24 187.96) (xy 148.59 187.96))
     (stroke (width 0) (type default) (color 0 0 0 0))
@@
     (stroke (width 0) (type default) (color 0 0 0 0))
   )
+  (wire (pts (xy 172.72 185.42) (xy 173.99 185.42))
+    (stroke (width 0) (type default) (color 0 0 0 0))
+  )
   (wire (pts (xy 43.18 165.1) (xy 40.64 165.1))
     (stroke (width 0) (type default) (color 0 0 0 0))
@@
   )
   (wire (pts (xy 153.67 187.96) (xy 157.48 187.96))
+    (stroke (width 0) (type default) (color 0 0 0 0))
+  )
+  (wire (pts (xy 22.86 193.04) (xy 25.4 193.04))
     (stroke (width 0) (type default) (color 0 0 0 0))
   )
@@
     (pin "2")
   )
-  (symbol (lib_id "Connector:DIN-5_180degree") (at 33.02 190.5 0) (unit 1)
+  (symbol (lib_id "connectors_with_ground:DIN-5_180degree_GND") (at 33.02 190.5 0) (unit 1)
     (in_bom yes) (on_board yes)
     (property "Reference" "J7" (id 0) (at 33.02 199.39 0))
@@
       (effects (font (size 1.27 1.27)) hide)
     )
+    (pin "0")
     (pin "1")
     (pin "2")
@@
     (pin "4")
     (pin "5")
+  )
+  (symbol (lib_id "power:GND") (at 177.8 181.61 0) (unit 1)
+    (in_bom yes) (on_board yes)
+    (property "Reference" "#PWR?" (id 0) (at 177.8 187.96 0)
+      (effects (font (size 1.27 1.27)) hide)
+    )
+    (property "Value" "GND" (id 1) (at 179.07 184.15 0)
+      (effects (font (size 1.27 1.27)) (justify left))
+    )
+    (property "Footprint" "" (id 2) (at 177.8 181.61 0)
+      (effects (font (size 1.27 1.27)) hide)
+    )
+    (property "Datasheet" "" (id 3) (at 177.8 181.61 0)
+      (effects (font (size 1.27 1.27)) hide)
+    )
+    (pin "1")
   )
   (symbol (lib_id "power:+5V") (at 48.26 110.49 0) (unit 1)
@@
     (pin "1")
   )
-  (symbol (lib_id "Connector:DIN-5_180degree") (at 165.1 187.96 180) (unit 1)
+  (symbol (lib_id "power:GND") (at 22.86 195.58 0) (unit 1)
+    (in_bom yes) (on_board yes)
+    (property "Reference" "#PWR?" (id 0) (at 22.86 201.93 0)
+      (effects (font (size 1.27 1.27)) hide)
+    )
+    (property "Value" "GND" (id 1) (at 22.86 199.39 0))
+    (property "Footprint" "" (id 2) (at 22.86 195.58 0)
+      (effects (font (size 1.27 1.27)) hide)
+    )
+    (property "Datasheet" "" (id 3) (at 22.86 195.58 0)
+      (effects (font (size 1.27 1.27)) hide)
+    )
+    (pin "1")
+  )
+  (symbol (lib_id "connectors_with_ground:DIN-5_180degree_GND") (at 165.1 187.96 180) (unit 1)
     (in_bom yes) (on_board yes)
     (property "Reference" "J8" (id 0) (at 165.1 179.07 0))
@@
       (effects (font (size 1.27 1.27)) hide)
     )
+    (pin "0")
     (pin "1")
     (pin "2")
