File: subsheet_102.kicad_sch (KiCad schematic)
At the start: 14 parts, among them J7 MIDI IN, J8 MIDI OUT, U20 MC6850_PHY, U35 74LS04_PHY, U39 PC900_PHY

Commit message: assigning footprints
Parts:
- CR7: footprint (none) -> commons-passives_THT:Passive_THT_diode_W2.54mm_L12.70mm
Changed lines of the file:
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@@
     (property "Reference" "CR7" (id 0) (at 33.02 171.45 0))
     (property "Value" "1N914" (id 1) (at 33.02 176.53 0))
-    (property "Footprint" "" (id 2) (at 33.02 173.99 0)
+    (property "Footprint" "commons-passives_THT:Passive_THT_diode_W2.54mm_L12.70mm" (id 2) (at 33.02 173.99 0)
       (effects (font (size 1.27 1.27)) hide)
     )

Commit message: assign footprints of remaining Resistors
Parts:
- R77, R78, R79, R80, R81: footprint (none) -> commons-passives_THT:Passive_THT_resistor_W2.54mm_L12.70mm
Changed lines of the file:
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@@
       (effects (font (size 1.27 1.27)) (justify left))
     )
-    (property "Footprint" "" (id 2) (at 120.65 167.64 0)
+    (property "Footprint" "commons-passives_THT:Passive_THT_resistor_W2.54mm_L12.70mm" (id 2) (at 120.65 167.64 0)
       (effects (font (size 1.27 1.27)) hide)
     )
@@
       (effects (font (size 1.27 1.27)) (justify left))
     )
-    (property "Footprint" "" (id 2) (at 151.13 187.96 0)
+    (property "Footprint" "commons-passives_THT:Passive_THT_resistor_W2.54mm_L12.70mm" (id 2) (at 151.13 187.96 0)
       (effects (font (size 1.27 1.27)) hide)
     )
@@
       (effects (font (size 1.27 1.27)) (justify left))
     )
-    (property "Footprint" "" (id 2) (at 180.34 190.5 0)
+    (property "Footprint" "commons-passives_THT:Passive_THT_resistor_W2.54mm_L12.70mm" (id 2) (at 180.34 190.5 0)
       (effects (font (size 1.27 1.27)) hide)
     )
@@
       (effects (font (size 1.27 1.27)) (justify left))
     )
-    (property "Footprint" "" (id 2) (at 151.13 190.5 0)
+    (property "Footprint" "commons-passives_THT:Passive_THT_resistor_W2.54mm_L12.70mm" (id 2) (at 151.13 190.5 0)
       (effects (font (size 1.27 1.27)) hide)
     )
@@
       (effects (font (size 1.27 1.27)) (justify left))
     )
-    (property "Footprint" "" (id 2) (at 180.34 187.96 0)
-      (effects (font (size 1.27 1.27)) hide)
-    )
+    (property "Footprint" "commons-passives_THT:Passive_THT_resistor_W2.54mm_L12.70mm" (id 2) (at 180.34 187.96 0)
+      (effects (font (size 1.27 1.27)) hide)
+    )

Commit message: assign dsub footprints and midi ports
Parts:
- J7, J8: footprint (none) -> commons-interconnect_THT:socket-din-5
Changed lines of the file:
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@@
     (property "Reference" "J7" (id 0) (at 33.02 199.39 0))
     (property "Value" "MIDI IN" (id 1) (at 33.02 196.85 0))
-    (property "Footprint" "" (id 2) (at 33.02 190.5 0)
+    (property "Footprint" "commons-interconnect_THT:socket-din-5" (id 2) (at 33.02 190.5 0)
       (effects (font (size 1.27 1.27)) hide)
     )
@@
     (property "Reference" "J8" (id 0) (at 165.1 179.07 0))
     (property "Value" "MIDI OUT" (id 1) (at 165.1 181.61 0))
-    (property "Footprint" "" (id 2) (at 165.1 187.96 0)
-      (effects (font (size 1.27 1.27)) hide)
-    )
+    (property "Footprint" "commons-interconnect_THT:socket-din-5" (id 2) (at 165.1 187.96 0)
+      (effects (font (size 1.27 1.27)) hide)
+    )
