File: subsheet_205.kicad_sch (KiCad schematic)
At the start: 34 parts, among them SW2 RESET, U10 MC68000_DIP_64_PHY, U36 74LS05_PHY, U37 LM556_DUAL_TIMER_PHY

Commit message: fixed missing annotation : C47
Parts:
- gave numbers to parts that had none: 1
Changed lines of the file:
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@@
   (symbol (lib_id "Device:C_Small") (at 91.44 146.05 0) (unit 1)
     (in_bom yes) (on_board yes)
-    (property "Reference" "C?" (id 0) (at 93.98 144.78 0)
+    (property "Reference" "C47" (id 0) (at 93.98 144.78 0)
       (effects (font (size 1.27 1.27)) (justify left))
     )
