File: subsheet_100.kicad_sch (KiCad schematic)
At the start: 0 parts

Commit message: MFP : direct connections
Parts:
- added C10, C11: 30pF, commons-passives_THT:Passive_THT_capacitor_mlcc_W2.54mm_L12.70mm, symbol Device:C_Small
- added C12: 0.1uF, commons-passives_THT:Passive_THT_capacitor_mlcc_W2.54mm_L12.70mm, symbol Device:C_Small
- added R4: 4K7, symbol Device:R_Small_US
- added U11: MC68901_DIP_48_PHY, Package_DIP:DIP-48_W15.24mm_LongPads, symbol mc68901d-dip48:MC68901_DIP_48_PHY
- added Y1: 2.4576 MHz, symbol Device:Crystal_Small
Connections:
- new net: C11.1, U11.17 (XTAL1), Y1.1
- new net: C10.1, U11.18 (XTAL2), Y1.2
- new net: R4.1, U11.25 (I3)
- new net: U11.10 (RC), U11.16 (TDO), U11.7 (TC)
- new net: U11.19 (TAI), U11.22 (I0)
- new net +5V: C12.1, R4.2, U11.11 (VCC)
- new net 4MHZ: U11.35 (CLK)
- new net A1: U11.2 (RS1)
- new net A2: U11.3 (RS2)
- new net A3: U11.4 (RS3)
- new net A4: U11.5 (RS4)
- new net A5: U11.6 (RS5)
- new net ACIA_IRQ: U11.26 (I4)
- new net D0: U11.37 (D0)
- new net D1: U11.38 (D1)
- new net D2: U11.39 (D2)
- new net D3: U11.40 (D3)
- new net D4: U11.41 (D4)
- new net D5: U11.42 (D5)
- new net D6: U11.43 (D6)
- new net D7: U11.44 (D7)
- new net DE: U11.20 (TBI)
- new net GND: C10.2, C11.2, C12.2, U11.34 (~{IEI}), U11.36 (GND)
- new net MONOMON: U11.29 (I7)
- new net XDTACK: U11.46 (~{DTACK})
- new net XIACK: U11.45 (~{IACK})
- new net XLDS: U11.47 (~{DS})
- new net XMFPCS: U11.48 (~{CS})
- new net XMFPINT: U11.32 (~{IRQ})
- new net XRESET: U11.21 (~{RESET})
- new net XRXW: U11.1 (R/~{W})
- new net media_int: U11.27 (I5)
- no-connect marks 0 -> 6

Commit message: rs 232 port
Parts:
- added J4: RS-232, symbol Connector:DB25_Male_MountingHoles
- added L67, L68, L69, L70, L71, L72, L73: Filter LCL, symbol Device:Filter_EMI_LCL
Connections:
- net GND: now also J4.0 (PAD), J4.1, J4.7, L67.2, L68.2, L69.2, L70.2, L71.2, L72.2, L73.2
- new net: J4.22 (P22), L73.3
- new net: J4.3, L71.3
- new net: J4.2, L72.3
- new net: J4.20 (P20), L68.3
- new net: J4.4, L70.3
- new net: J4.5, L69.3
- new net: J4.8, L67.3
- no-connect marks 6 -> 22

Commit message: rs 232 transcievers
Parts:
- added U13: 1489_SOCKET, Package_DIP:DIP-14_W7.62mm_LongPads, symbol mc1489:1489_SOCKET
- added U14: 1488_PHY, Package_DIP:DIP-14_W7.62mm_LongPads, symbol mc1488:1488_PHY
Connections:
- net at L73.1: now also U13.10 (IC)
- net at L71.1: now also U13.1 (IA)
- net at L70.1: now also U14.11 (OD)
- net at L69.1: now also U13.13 (ID)
- net at L68.1: now also U14.3 (OA)
- net at L67.1: now also U13.4 (IB)
- net at L72.1: now also U14.8 (OC)
- new net: U14.10 (IC1), U14.9 (IC2)
- new net: U14.12 (ID2), U14.13 (ID1)

Commit message: done RS-232 port to MFP68901
Parts:
- added C15, C17, C22: 0.1uF, commons-passives_THT:Passive_THT_capacitor_mlcc_W2.54mm_L12.70mm, symbol Device:C_Small
- added C18, C19, C20, C21: 100pF, commons-passives_THT:Passive_THT_capacitor_mlcc_W2.54mm_L12.70mm, symbol Device:C_Small
- U13: value 1489_SOCKET -> MC1489; symbol mc1489:1489_SOCKET -> mc1489:1489_PHY
- U14: value 1488_PHY -> MC1488
Connections:
- net +5V: now also U13.14 (VCC), C17.1
- net GND: now also U13.7 (GND), U14.4 (IB1), U14.5 (IB2), U14.7 (GND), C15.2, C17.2, C18.2, C19.2, C20.2, C21.2, C22.2
- net RI: now reaches L73.1, U13.10 (IC)
- net RxD: now reaches L71.1, U13.1 (IA)
- net RTS: now reaches L70.1, U14.11 (OD)
- net CTS: now reaches L69.1, U13.13 (ID)
- net DTR: now reaches L68.1, U14.3 (OA)
- net DCD: now reaches L67.1, U13.4 (IB)
- net TxD: now reaches L72.1, U14.8 (OC)
- net mfp_i1: now reaches U11.23 (I1)
- net mfp_i1: now also U13.6 (OB)
- net mfp_i2: now reaches U11.24 (I2)
- net mfp_i2: now also U13.11 (OD)
- net mfp_i6: now reaches U11.28 (I6)
- net mfp_i6: now also U13.8 (OC)
- net mfp_so: now reaches U11.8 (SO)
- net mfp_so: now also U14.10 (IC1), U14.9 (IC2)
- net mfp_si: now reaches U11.9 (SI)
- net mfp_si: now also U13.3 (OA)
- net at U13.12 (RCD): now also C18.1
- net at U13.2 (RCA): now also C20.1
- net at U13.5 (RCB): now also C21.1
- net at U13.9 (RCC): now also C19.1
- net -12V: now reaches U14.1 (VEE)
- net -12V: now also C15.1
- net SERIAL_RTS: now reaches U14.12 (ID2), U14.13 (ID1)
- net +12V: now reaches U14.14 (VCC)
- net +12V: now also C22.1
- net SERIAL_DTR: now reaches U14.2 (IA)
- net media_int renamed MEDIA_IRQ
- no-connect marks 22 -> 23
Other:
- note added: "CD"
- note added: "CI"
- note added: "CS"
- note added: "ER"
- note added: "FG"
- note added: "From U40"
- note added: "RD"
- note added: "RS"
- note added: "SD"
- note added: "SG"
- moved on the sheet: C10, C11, C12, J4, L67, L68, L69, L70, L71, L72, L73, R4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

Commit message: finishing touch MFP to serial port
Parts:
- U11: value MC68901_DIP_48_PHY -> MC68901 Multi Function Peripheral DIP 48
- U13: value MC1489 -> MC1489 Quad Line EIA-232D Receivers
- U14: value MC1488 -> MC1488 Quad Line EIA-232D Driver
Other:
- moved on the sheet: C10, C11, C12, R4, U11, Y1

Commit message: Start YM2149, sound mixer, parallel port ; update MFP
Connections:
- net PARALLEL_BUSY: now reaches U11.19 (TAI), U11.22 (I0)
Other:
- note added: "From U19"
Changed lines of the file:
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@@
   (junction (at 82.55 63.5) (diameter 0) (color 0 0 0 0)
+  )
+  (junction (at 74.93 101.6) (diameter 0) (color 0 0 0 0)
   )
   (junction (at 62.23 91.44) (diameter 0) (color 0 0 0 0)
@@
     (stroke (width 0) (type default) (color 0 0 0 0))
   )
+  (wire (pts (xy 71.12 114.3) (xy 74.93 114.3))
+    (stroke (width 0) (type default) (color 0 0 0 0))
+  )
   (wire (pts (xy 96.52 175.26) (xy 96.52 171.45))
     (stroke (width 0) (type default) (color 0 0 0 0))
@@
     (stroke (width 0) (type default) (color 0 0 0 0))
   )
+  (wire (pts (xy 74.93 114.3) (xy 74.93 101.6))
+    (stroke (width 0) (type default) (color 0 0 0 0))
+  )
   (wire (pts (xy 165.1 175.26) (xy 166.37 175.26))
     (stroke (width 0) (type default) (color 0 0 0 0))
@@
     (stroke (width 0) (type default) (color 0 0 0 0))
   )
+  (text "From U19" (at 36.83 146.05 0)
+    (effects (font (size 1.27 1.27)) (justify left bottom))
+  )
   (text "From U40" (at 156.21 102.87 0)
     (effects (font (size 1.27 1.27)) (justify left bottom))
   )
   (text "FG" (at 176.53 154.94 180)
+    (effects (font (size 1.27 1.27)) (justify right bottom))
+  )
+  (text "From U19" (at 109.22 143.51 180)
     (effects (font (size 1.27 1.27)) (justify right bottom))
   )
@@
       (effects (font (size 1.27 1.27)) (justify right) hide)
     )
+  )
+  (global_label "PARALLEL_BUSY" (shape input) (at 71.12 114.3 180) (fields_autoplaced)
+    (effects (font (size 1.27 1.27)) (justify right))
+    (property "Intersheet References" "${INTERSHEET_REFS}" (id 0) (at 53.9791 114.2206 0)
+      (effects (font (size 1.27 1.27)) (justify right) hide)
+    )
