File: subsheet_100.kicad_sch (KiCad schematic)
At the start: 23 parts, among them J4 RS-232, U11 MC68901 Multi Function Periph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, U13 MC1489 Quad Line EIA-232D Rec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, U14 MC1488 Quad Line EIA-232D Dri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, Y1 2.4576 MHz

Commit message: assign footprints of remaining Resistors
Parts:
- R4: footprint (none) -> commons-passives_THT:Passive_THT_resistor_W2.54mm_L12.70mm
Changed lines of the file:
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@@
       (effects (font (size 1.27 1.27)) (justify right))
     )
-    (property "Footprint" "" (id 2) (at 138.43 106.68 0)
+    (property "Footprint" "commons-passives_THT:Passive_THT_resistor_W2.54mm_L12.70mm" (id 2) (at 138.43 106.68 0)
       (effects (font (size 1.27 1.27)) hide)
     )

Commit message: assigned footprint for all remaining standard passives
Parts:
- L67, L68, L69, L70, L71, L72, L73: footprint (none) -> commons-passives_THT:Passive_THT_EMI_filter_W5.08mm_L7.62mm
- Y1: footprint (none) -> Crystal:Crystal_HC50_Vertical
Changed lines of the file:
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@@
       (effects (font (size 1.27 1.27)) (justify left))
     )
-    (property "Footprint" "" (id 2) (at 157.48 218.44 90)
+    (property "Footprint" "commons-passives_THT:Passive_THT_EMI_filter_W5.08mm_L7.62mm" (id 2) (at 157.48 218.44 90)
       (effects (font (size 1.27 1.27)) hide)
     )
@@
       (effects (font (size 1.27 1.27)) (justify left))
     )
-    (property "Footprint" "" (id 2) (at 57.15 91.44 0)
+    (property "Footprint" "Crystal:Crystal_HC50_Vertical" (id 2) (at 57.15 91.44 0)
       (effects (font (size 1.27 1.27)) hide)
     )
@@
       (effects (font (size 1.27 1.27)) (justify left))
     )
-    (property "Footprint" "" (id 2) (at 144.78 167.64 90)
+    (property "Footprint" "commons-passives_THT:Passive_THT_EMI_filter_W5.08mm_L7.62mm" (id 2) (at 144.78 167.64 90)
       (effects (font (size 1.27 1.27)) hide)
     )
@@
       (effects (font (size 1.27 1.27)) (justify left))
     )
-    (property "Footprint" "" (id 2) (at 157.48 177.8 90)
+    (property "Footprint" "commons-passives_THT:Passive_THT_EMI_filter_W5.08mm_L7.62mm" (id 2) (at 157.48 177.8 90)
       (effects (font (size 1.27 1.27)) hide)
     )
@@
       (effects (font (size 1.27 1.27)) (justify left))
     )
-    (property "Footprint" "" (id 2) (at 144.78 187.96 90)
+    (property "Footprint" "commons-passives_THT:Passive_THT_EMI_filter_W5.08mm_L7.62mm" (id 2) (at 144.78 187.96 90)
       (effects (font (size 1.27 1.27)) hide)
     )
@@
       (effects (font (size 1.27 1.27)) (justify left))
     )
-    (property "Footprint" "" (id 2) (at 157.48 198.12 90)
+    (property "Footprint" "commons-passives_THT:Passive_THT_EMI_filter_W5.08mm_L7.62mm" (id 2) (at 157.48 198.12 90)
       (effects (font (size 1.27 1.27)) hide)
     )
@@
       (effects (font (size 1.27 1.27)) (justify left))
     )
-    (property "Footprint" "" (id 2) (at 144.78 208.28 90)
+    (property "Footprint" "commons-passives_THT:Passive_THT_EMI_filter_W5.08mm_L7.62mm" (id 2) (at 144.78 208.28 90)
       (effects (font (size 1.27 1.27)) hide)
     )
@@
       (effects (font (size 1.27 1.27)) (justify left))
     )
-    (property "Footprint" "" (id 2) (at 157.48 157.48 90)
-      (effects (font (size 1.27 1.27)) hide)
-    )
+    (property "Footprint" "commons-passives_THT:Passive_THT_EMI_filter_W5.08mm_L7.62mm" (id 2) (at 157.48 157.48 90)
+      (effects (font (size 1.27 1.27)) hide)
+    )
