File: subsheet_100.kicad_sch (KiCad schematic)
At the start: 23 parts, among them J4 RS-232, U11 MC68901 Multi Function Periph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, U13 MC1489 Quad Line EIA-232D Rec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, U14 MC1488 Quad Line EIA-232D Dri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, Y1 2.4576 MHz

Commit message: Fixed footprint of C22 -- pitch of 500mils instead of 400
Parts:
- C22: footprint commons-passives_THT:Passive_THT_capacitor_mlcc_W2.54mm_L10.16mm -> commons-passives_THT:Passive_THT_capacitor_mlcc_W2.54mm_L12.70mm
Changed lines of the file:
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@@
       (effects (font (size 1.27 1.27)) (justify left))
     )
-    (property "Footprint" "commons-passives_THT:Passive_THT_capacitor_mlcc_W2.54mm_L10.16mm" (at 114.3 143.51 0)
+    (property "Footprint" "commons-passives_THT:Passive_THT_capacitor_mlcc_W2.54mm_L12.70mm" (at 114.3 143.51 0)
       (effects (font (size 1.27 1.27)) hide)
     )

Commit message: Fixed -- forgotten 1K pullup on XMFPINT
Parts:
- added R3: 1K, commons-passives_THT:Passive_THT_resistor_W2.54mm_L12.70mm, symbol Device:R_Small_US
Connections:
- net +5V: now also R3.2
- net XMFPINT: now also R3.1
Changed lines of the file:
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@@
   (junction (at 53.34 149.86) (diameter 0) (color 0 0 0 0)
+  )
+  (junction (at 139.7 88.9) (diameter 0) (color 0 0 0 0)
   )
   (junction (at 121.92 171.45) (diameter 0) (color 0 0 0 0)
@@
     (stroke (width 0) (type default))
   )
+  (wire (pts (xy 139.7 88.9) (xy 143.51 88.9))
+    (stroke (width 0) (type default))
+  )
   (wire (pts (xy 62.23 63.5) (xy 82.55 63.5))
     (stroke (width 0) (type default))
@@
     (stroke (width 0) (type default))
   )
+  (wire (pts (xy 162.56 88.9) (xy 157.48 88.9))
+    (stroke (width 0) (type default))
+  )
   (wire (pts (xy 92.71 144.78) (xy 96.52 144.78))
     (stroke (width 0) (type default))
@@
     (stroke (width 0) (type default))
   )
+  (wire (pts (xy 139.7 88.9) (xy 139.7 91.44))
+    (stroke (width 0) (type default))
+  )
   (wire (pts (xy 53.34 154.94) (xy 53.34 149.86))
     (stroke (width 0) (type default))
   )
-  (wire (pts (xy 133.35 88.9) (xy 143.51 88.9))
+  (wire (pts (xy 133.35 88.9) (xy 139.7 88.9))
     (stroke (width 0) (type default))
   )
@@
     (stroke (width 0) (type default))
   )
+  (wire (pts (xy 157.48 88.9) (xy 157.48 91.44))
+    (stroke (width 0) (type default))
+  )
   (wire (pts (xy 133.35 55.88) (xy 143.51 55.88))
     (stroke (width 0) (type default))
@@
     (stroke (width 0) (type default))
   )
+  (wire (pts (xy 167.64 88.9) (xy 177.8 88.9))
+    (stroke (width 0) (type default))
+  )
   (wire (pts (xy 177.8 148.59) (xy 187.96 148.59))
+    (stroke (width 0) (type default))
+  )
+  (wire (pts (xy 157.48 91.44) (xy 139.7 91.44))
     (stroke (width 0) (type default))
   )
@@
         (path "/61fe4c73-be59-4519-98f1-a634322a841d/3540a282-3d60-41a6-91eb-10c674ce4d4d"
           (reference "L71") (unit 1)
+        )
+      )
+    )
+  )
+  (symbol (lib_id "Device:R_Small_US") (at 165.1 88.9 90) (unit 1)
+    (in_bom yes) (on_board yes) (dnp no)
+    (property "Reference" "R3" (at 162.56 87.63 90)
+      (effects (font (size 1.27 1.27)) (justify left))
+    )
+    (property "Value" "1K" (at 166.37 87.63 90)
+      (effects (font (size 1.27 1.27)) (justify right))
+    )
+    (property "Footprint" "commons-passives_THT:Passive_THT_resistor_W2.54mm_L12.70mm" (at 165.1 88.9 0)
+      (effects (font (size 1.27 1.27)) hide)
+    )
+    (property "Datasheet" "~" (at 165.1 88.9 0)
+      (effects (font (size 1.27 1.27)) hide)
+    )
+    (pin "1")
+    (pin "2")
+    (instances
+      (project "motherboard"
+        (path "/61fe4c73-be59-4519-98f1-a634322a841d/3540a282-3d60-41a6-91eb-10c674ce4d4d"
+          (reference "R3") (unit 1)
         )
       )
@@
         )
       )
+    )
+  )
+  (symbol (lib_id "power:+5V") (at 177.8 88.9 0) (unit 1)
+    (in_bom yes) (on_board yes) (dnp no)
+    (property "Reference" "#PWR01" (at 177.8 92.71 0)
+      (effects (font (size 1.27 1.27)) hide)
+    )
+    (property "Value" "+5V" (at 179.07 87.63 0)
+      (effects (font (size 1.27 1.27)) (justify left))
+    )
+    (property "Footprint" "" (at 177.8 88.9 0)
+      (effects (font (size 1.27 1.27)) hide)
+    )
+    (property "Datasheet" "" (at 177.8 88.9 0)
+      (effects (font (size 1.27 1.27)) hide)
+    )
+    (pin "1")
+    (instances
+      (project "motherboard"
+        (path "/61fe4c73-be59-4519-98f1-a634322a841d/3540a282-3d60-41a6-91eb-10c674ce4d4d"
+          (reference "#PWR01") (unit 1)
+        )
+      )

Commit message: Fixed -- renamed 1K pullup on XMFPINT -- R105 instead of R3
Parts:
- renumbered R3 to R105
Changed lines of the file:
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@@
   (symbol (lib_id "Device:R_Small_US") (at 165.1 88.9 90) (unit 1)
     (in_bom yes) (on_board yes) (dnp no)
-    (property "Reference" "R3" (at 162.56 87.63 90)
+    (property "Reference" "R105" (at 162.56 87.63 90)
       (effects (font (size 1.27 1.27)) (justify left))
     )
@@
       (project "motherboard"
         (path "/61fe4c73-be59-4519-98f1-a634322a841d/3540a282-3d60-41a6-91eb-10c674ce4d4d"
-          (reference "R3") (unit 1)
+          (reference "R105") (unit 1)
         )
       )
