File: subsheet_200.kicad_sch (KiCad schematic)
At the start: 22 parts, among them U15 ST_MMU_PHY, U22 74LS373_PHY, U23 74LS373_PHY, U26 74LS244_PHY, U27 74LS244_PHY

Commit message: done power socket
Changed lines of the file:
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@@
   (junction (at 152.4 38.1) (diameter 0) (color 0 0 0 0)
-  )
-  (junction (at 147.32 38.1) (diameter 0) (color 0 0 0 0)
   )
   (junction (at 83.82 165.1) (diameter 0) (color 0 0 0 0)
@@
       (effects (font (size 1.27 1.27)) hide)
     )
-    (pin "1")
-  )
-  (symbol (lib_id "power:PWR_FLAG") (at 147.32 38.1 90) (unit 1)
-    (in_bom yes) (on_board yes)
-    (property "Reference" "#FLG0101" (id 0) (at 145.415 38.1 0)
-      (effects (font (size 1.27 1.27)) hide)
-    )
-    (property "Value" "PWR_FLAG" (id 1) (at 139.7 38.1 90))
-    (property "Footprint" "" (id 2) (at 147.32 38.1 0)
-      (effects (font (size 1.27 1.27)) hide)
-    )
-    (property "Datasheet" "~" (id 3) (at 147.32 38.1 0)
-      (effects (font (size 1.27 1.27)) hide)
-    )

Commit message: fixed symbols causing DRC errors, fixed renamed symbol 'FerriteBead_small'
Parts:
- L26, L28: symbol Device:Ferrite_Bead_Small -> Device:FerriteBead_Small
Changed lines of the file:
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@@
     (pin "1")
   )
-  (symbol (lib_id "Device:Ferrite_Bead_Small") (at 161.29 50.8 270) (unit 1)
+  (symbol (lib_id "Device:FerriteBead_Small") (at 161.29 50.8 270) (unit 1)
     (in_bom yes) (on_board yes)
     (property "Reference" "L28" (id 0) (at 154.94 49.53 90)
@@
     (pin "1")
   )
-  (symbol (lib_id "Device:Ferrite_Bead_Small") (at 161.29 38.1 270) (unit 1)
+  (symbol (lib_id "Device:FerriteBead_Small") (at 161.29 38.1 270) (unit 1)
     (in_bom yes) (on_board yes)
     (property "Reference" "L26" (id 0) (at 154.94 36.83 90)
