File: subsheet_200.kicad_sch (KiCad schematic)
At the start: 22 parts, among them U15 ST_MMU_PHY, U22 74LS373_PHY, U23 74LS373_PHY, U26 74LS244_PHY, U27 74LS244_PHY

Commit message: pcb session 2024-05-01T23:19:53+02:00 -- fixed MMU VCC net, almost done U20 -- need to shield E signal
Connections:
- net +5VD: no longer C16.1, C25.2, U15.10 (VCC), U15.44 (VCC)
- new net +5Vmmu: C16.1, C25.2, U15.10 (VCC), U15.44 (VCC)
Changed lines of the file:
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@@
   (junction (at 172.72 165.1) (diameter 0) (color 0 0 0 0)
   )
-  (junction (at 38.1 73.66) (diameter 0) (color 0 0 0 0)
-  )
   (junction (at 152.4 38.1) (diameter 0) (color 0 0 0 0)
   )
   (junction (at 83.82 165.1) (diameter 0) (color 0 0 0 0)
-  )
-  (junction (at 133.35 114.3) (diameter 0) (color 0 0 0 0)
   )
   (junction (at 171.45 38.1) (diameter 0) (color 0 0 0 0)
@@
     (stroke (width 0) (type default))
   )
-  (wire (pts (xy 121.92 114.3) (xy 133.35 114.3))
+  (wire (pts (xy 121.92 114.3) (xy 140.97 114.3))
     (stroke (width 0) (type default))
   )
@@
     (stroke (width 0) (type default))
   )
-  (wire (pts (xy 27.94 73.66) (xy 38.1 73.66))
+  (wire (pts (xy 27.94 73.66) (xy 43.18 73.66))
     (stroke (width 0) (type default))
   )
@@
     (stroke (width 0) (type default))
   )
-  (wire (pts (xy 38.1 73.66) (xy 43.18 73.66))
-    (stroke (width 0) (type default))
-  )
   (wire (pts (xy 78.74 167.64) (xy 83.82 167.64))
     (stroke (width 0) (type default))
@@
     (stroke (width 0) (type default))
   )
-  (wire (pts (xy 133.35 114.3) (xy 140.97 114.3))
-    (stroke (width 0) (type default))
-  )
   (wire (pts (xy 121.92 104.14) (xy 127 104.14))
     (stroke (width 0) (type default))
@@
     (effects (font (size 1.27 1.27)) (justify left bottom))
   )
+  (label "+5Vmmu" (at 127 114.3 0) (fields_autoplaced)
+    (effects (font (size 1.27 1.27)) (justify left bottom))
+  )
   (label "D7" (at 132.08 228.6 180) (fields_autoplaced)
     (effects (font (size 1.27 1.27)) (justify right bottom))
@@
   (label "MD5" (at 38.1 226.06 180) (fields_autoplaced)
     (effects (font (size 1.27 1.27)) (justify right bottom))
+  )
+  (label "+5Vmmu" (at 34.29 73.66 0) (fields_autoplaced)
+    (effects (font (size 1.27 1.27)) (justify left bottom))
   )
   (label "D0" (at 172.72 233.68 0) (fields_autoplaced)
@@
     )
   )
-  (symbol (lib_id "power:+5VD") (at 38.1 73.66 0) (unit 1)
-    (in_bom yes) (on_board yes) (dnp no)
-    (property "Reference" "#PWR0118" (at 38.1 77.47 0)
-      (effects (font (size 1.27 1.27)) hide)
-    )
-    (property "Value" "+5VD" (at 38.1 70.104 0)
-      (effects (font (size 1.27 1.27)))
-    )
-    (property "Footprint" "" (at 38.1 73.66 0)
-      (effects (font (size 1.27 1.27)) hide)
-    )
-    (property "Datasheet" "" (at 38.1 73.66 0)
-      (effects (font (size 1.27 1.27)) hide)
-    )
-    (pin "1")
-    (instances
-      (project "motherboard"
-        (path "/61fe4c73-be59-4519-98f1-a634322a841d/00000000-0000-0000-0000-000062c842ff"
-          (reference "#PWR0118") (unit 1)
-        )
-      )
-    )
-  )
   (symbol (lib_id "Device:C_Small") (at 143.51 114.3 90) (unit 1)
     (in_bom yes) (on_board yes) (dnp no)
@@
         )
       )
-    )
-  )
-  (symbol (lib_id "power:+5VD") (at 133.35 114.3 0) (unit 1)
-    (in_bom yes) (on_board yes) (dnp no)
-    (property "Reference" "#PWR0119" (at 133.35 118.11 0)
-      (effects (font (size 1.27 1.27)) hide)
-    )
-    (property "Value" "+5VD" (at 133.35 110.49 0)
-      (effects (font (size 1.27 1.27)))
-    )
-    (property "Footprint" "" (at 133.35 114.3 0)
-      (effects (font (size 1.27 1.27)) hide)
-    )
-    (property "Datasheet" "" (at 133.35 114.3 0)
-      (effects (font (size 1.27 1.27)) hide)
-    )
-    (pin "1")
-    (instances
-      (project "motherboard"
-        (path "/61fe4c73-be59-4519-98f1-a634322a841d/00000000-0000-0000-0000-000062c842ff"
-          (reference "#PWR0119") (unit 1)
-        )
-      )

Commit message: pcb session 2024-05-08T18:28:50+02:00 -- working on power rails, fixed +5VD vs +5Vmmu
Connections:
- net +5VD is gone; now on net +5Vmmu: L26.1
Changed lines of the file:
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@@
   (junction (at 83.82 165.1) (diameter 0) (color 0 0 0 0)
-  )
-  (junction (at 171.45 38.1) (diameter 0) (color 0 0 0 0)
   )
   (junction (at 171.45 50.8) (diameter 0) (color 0 0 0 0)
@@
   )
   (label "D8" (at 172.72 187.96 0) (fields_autoplaced)
+    (effects (font (size 1.27 1.27)) (justify left bottom))
+  )
+  (label "+5Vmmu" (at 163.83 38.1 0) (fields_autoplaced)
     (effects (font (size 1.27 1.27)) (justify left bottom))
   )
@@
         )
       )
-    )
-  )
-  (symbol (lib_id "power:+5VD") (at 171.45 38.1 0) (unit 1)
-    (in_bom yes) (on_board yes) (dnp no)
-    (property "Reference" "#PWR0116" (at 171.45 41.91 0)
-      (effects (font (size 1.27 1.27)) hide)
-    )
-    (property "Value" "+5VD" (at 171.45 34.544 0)
-      (effects (font (size 1.27 1.27)))
-    )
-    (property "Footprint" "" (at 171.45 38.1 0)
-      (effects (font (size 1.27 1.27)) hide)
-    )
-    (property "Datasheet" "" (at 171.45 38.1 0)
-      (effects (font (size 1.27 1.27)) hide)
-    )
-    (pin "1")
-    (instances
-      (project "motherboard"
-        (path "/61fe4c73-be59-4519-98f1-a634322a841d/00000000-0000-0000-0000-000062c842ff"
-          (reference "#PWR0116") (unit 1)
-        )
-      )
