File: subsheet_202.kicad_sch (KiCad schematic)
At the start: 54 parts, among them J6 DIN13S, Q10 2N3904, Q2 2N3904, Q3 2N3904, Q4 2N3904, Q5 2N3904, U31 ST_SHIFTER_PHY

Commit message: finition de la fiche, rajout de pwr_flag sur presque tous les points filtrés
Changed lines of the file:
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@@
   (junction (at 97.79 105.41) (diameter 0) (color 0 0 0 0)
+  )
+  (junction (at 83.82 64.77) (diameter 0) (color 0 0 0 0)
   )
   (junction (at 191.77 69.85) (diameter 0) (color 0 0 0 0)
@@
       (effects (font (size 1.27 1.27)) hide)
     )
+    (pin "1")
+  )
+  (symbol (lib_id "power:PWR_FLAG") (at 83.82 64.77 270) (unit 1)
+    (in_bom yes) (on_board yes)
+    (property "Reference" "#FLG?" (id 0) (at 85.725 64.77 0)
+      (effects (font (size 1.27 1.27)) hide)
+    )
+    (property "Value" "PWR_FLAG" (id 1) (at 86.36 64.77 90)
+      (effects (font (size 1.27 1.27)) (justify left))
+    )
+    (property "Footprint" "" (id 2) (at 83.82 64.77 0)
+      (effects (font (size 1.27 1.27)) hide)
+    )
+    (property "Datasheet" "~" (id 3) (at 83.82 64.77 0)
+      (effects (font (size 1.27 1.27)) hide)
+    )

Commit message: fixed symbols causing DRC errors, fixed renamed symbol 'FerriteBead_small'
Parts:
- L17, L21: symbol Device:Ferrite_Bead_Small -> Device:FerriteBead_Small
Changed lines of the file:
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@@
     (pin "1")
   )
-  (symbol (lib_id "Device:Ferrite_Bead_Small") (at 77.47 57.15 270) (unit 1)
+  (symbol (lib_id "Device:FerriteBead_Small") (at 77.47 57.15 270) (unit 1)
     (in_bom yes) (on_board yes)
     (property "Reference" "L21" (id 0) (at 71.12 55.88 90)
@@
     (pin "1")
   )
-  (symbol (lib_id "Device:Ferrite_Bead_Small") (at 133.35 30.48 270) (unit 1)
+  (symbol (lib_id "Device:FerriteBead_Small") (at 133.35 30.48 270) (unit 1)
     (in_bom yes) (on_board yes)
     (property "Reference" "L17" (id 0) (at 128.27 29.21 90)
