File: subsheet_203.kicad_sch (KiCad schematic)
At the start: 15 parts, among them J1 Cartridge port, U2 27C512_PHY, U3 27C512_PHY, U4 27C512_PHY, U5 27C512_PHY, U6 27C512_PHY, U7 27C512_PHY

Commit message: fixed symbols causing DRC errors, fixed renamed symbol 'FerriteBead_small'
Parts:
- L23: symbol Device:Ferrite_Bead_Small -> Device:FerriteBead_Small
Changed lines of the file:
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@@
     )
   )
-  (symbol (lib_id "27c512:27C512_PHY") (at 43.18 67.31 0) (unit 1)
+  (symbol (lib_name "27C512_PHY_2") (lib_id "27c512:27C512_PHY") (at 43.18 67.31 0) (unit 1)
     (in_bom yes) (on_board yes)
     (property "Reference" "U4" (id 0) (at 33.02 43.18 0)
@@
     (pin "1")
   )
-  (symbol (lib_id "27c512:27C512_PHY") (at 43.18 118.11 0) (unit 1)
+  (symbol (lib_name "27C512_PHY_4") (lib_id "27c512:27C512_PHY") (at 43.18 118.11 0) (unit 1)
     (in_bom yes) (on_board yes)
     (property "Reference" "U3" (id 0) (at 33.02 93.98 0)
@@
     (pin "1")
   )
-  (symbol (lib_id "27c512:27C512_PHY") (at 119.38 67.31 0) (unit 1)
+  (symbol (lib_name "27C512_PHY_3") (lib_id "27c512:27C512_PHY") (at 119.38 67.31 0) (unit 1)
     (in_bom yes) (on_board yes)
     (property "Reference" "U7" (id 0) (at 109.22 43.18 0)
@@
     (pin "1")
   )
-  (symbol (lib_id "27c512:27C512_PHY") (at 119.38 118.11 0) (unit 1)
+  (symbol (lib_name "27C512_PHY_5") (lib_id "27c512:27C512_PHY") (at 119.38 118.11 0) (unit 1)
     (in_bom yes) (on_board yes)
     (property "Reference" "U6" (id 0) (at 109.22 93.98 0)
@@
     (pin "1")
   )
-  (symbol (lib_id "27c512:27C512_PHY") (at 119.38 168.91 0) (unit 1)
+  (symbol (lib_name "27C512_PHY_1") (lib_id "27c512:27C512_PHY") (at 119.38 168.91 0) (unit 1)
     (in_bom yes) (on_board yes)
     (property "Reference" "U5" (id 0) (at 109.22 144.78 0)
@@
     (pin "1")
   )
-  (symbol (lib_id "Device:Ferrite_Bead_Small") (at 171.45 132.08 270) (unit 1)
+  (symbol (lib_id "Device:FerriteBead_Small") (at 171.45 132.08 270) (unit 1)
     (in_bom yes) (on_board yes)
     (property "Reference" "L23" (id 0) (at 165.1 130.81 90)
