File: subsheet_300.kicad_sch (KiCad schematic)
At the start: 0 parts

Commit message: done 32mhz clock and modulator clock
Parts:
- added C52: 33pF, commons-passives_THT:Passive_THT_capacitor_mlcc_W2.54mm_L12.70mm, symbol Device:C_Small
- added C56: 68pF, commons-passives_THT:Passive_THT_capacitor_mlcc_W2.54mm_L12.70mm, symbol Device:C_Small
- added C63: 8.2pF, commons-passives_THT:Passive_THT_capacitor_mlcc_W2.54mm_L12.70mm, symbol Device:C_Small
- added C66, C77: 0.1uF, commons-passives_THT:Passive_THT_capacitor_mlcc_W2.54mm_L12.70mm, symbol Device:C_Small
- added C73: 0.47uF, commons-passives_THT:Passive_THT_capacitor_mlcc_W2.54mm_L12.70mm, symbol Device:C_Small
- added C74: 4700pF, commons-passives_THT:Passive_THT_capacitor_mlcc_W2.54mm_L12.70mm, symbol Device:C_Small
- added C76, C?: 1SV69, symbol Device:D_Capacitance
- added C?: 0.022uF, commons-passives_THT:Passive_THT_capacitor_mlcc_W2.54mm_L12.70mm, symbol Device:C_Small
- added L19: see table, symbol Device:L_Small
- added L20: 0.27uH, symbol Device:L_Small
- added L22: 1uH, symbol Device:L_Small
- added Q11, Q6, Q?: 2N3904, symbol Device:Q_NPN_CBE
- added Q7, Q9: 2N3906, symbol Device:Q_PNP_CBE
- added R109: 150, symbol Device:R_Small_US
- added R112, R94: 100, symbol Device:R_Small_US
- added R113: 220, symbol Device:R_Small_US
- added R141: 2K2, symbol Device:R_Small_US
- added R67: 33K, symbol Device:R_Small_US
- added R68: 6K8, symbol Device:R_Small_US
- added R69, R70: 100K, symbol Device:R_Small_US
- added R72: 470, symbol Device:R_Small_US
- added R73: 27, symbol Device:R_Small_US
- added R84: 560, symbol Device:R_Small_US
- added R85: 5K6, symbol Device:R_Small_US
- added R86: 4K7, symbol Device:R_Small_US
- added R88: 1K5, symbol Device:R_Small_US
- added U41: 74LS74 DUAL FLIP-FLOPS, Package_DIP:DIP-14_W7.62mm_LongPads, symbol 74x74:74LS74_DUAL_POSITIVE-EDGE-TRIGGERED_D_FLIP-FLOPS_WITH_PRESET_CLEAR_AND_CO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
- added Y2, Y3: see table, symbol Device:Crystal_Small
Connections:
- new net: C63.1, C73.1, L19.1, L20.2, Q6.1 (C), R68.2
- new net: C52.1, C63.2, L19.2, Q?.1 (C), R67.1
- new net: Q?.2 (B), R68.1, R85.2, Y2.2
- new net: C76.1 (K), L22.1, R86.1
- new net: L22.2, R86.2, Y2.1
- new net: C52.2, Q6.2 (B), R67.2
- new net: C77.1, Q9.2 (B), R72.1, R88.2, R94.2
- new net: C?.1, R69.1, R70.1
- new net: Q11.1 (C), R141.1, R69.2
- new net: C56.1, Q?.3 (E), R84.2
- new net: C?.1 (K), R70.2
- new net: Q11.2 (B), U41.6 (~{1Q})
- new net: Q9.1 (C), R112.2, Y3.2
- new net: Q7.2 (B), R94.1, Y3.1
- new net: Q7.3 (E), Q9.3 (E), R73.1
- new net: R72.2, R73.2
- new net +12V: R141.2
- new net +5V: C66.1, C74.1, L20.1, U41.1 (~{1CLR}), U41.14 (VCC), U41.4 (~{1PRE})
- new net 32MHZ: Q6.3 (E), R109.2
- new net GND: C56.2, C66.2, C73.2, C74.2, C76.2 (A), C77.2, C?.2, C?.2 (A), Q11.3 (E), R109.1, R112.1, R113.1, R84.1, R85.1, R88.1, U41.10 (~{2PRE}), U41.11 (2CLK), U41.12 (2D), U41.13 (~{2CLR}), U41.7 (GND)
- new net LINE_PHASE: U41.3 (1CLK)
- new net MODCLOCK: Q7.1 (C), R113.2, U41.2 (1D)
- no-connect marks 0 -> 3
Other:
- note added: "ASSY N0. -001 -002,-003,-005 -004"
- note added: "From U35"
- note added: "L19 1uH 0.82uH 1uH"
- note added: "NTSC PAL NO MODULATOR"
- note added: "PCB ASSY NO. * CA070052-001 * CA070052-002 * CA070052-003 * CA070052-005"
- note added: "Reference table"
- note added: "With modulator"
- note added: "Without modulator : PCB ASSY NO. CA070052-004"
- note added: "Without modulator C76 is a 22pF non polarized capacitor"
- note added: "Y2 32.0424 MHz 32.084988 MHz 32.084988 MHz"
- note added: "Y3 3.579545 MHz 4.433618 MHz"

Commit message: added missing wires, and annotation
Parts:
- gave numbers to parts that had none: 1
Connections:
- net at C63.1, C73.1, L19.1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: now also R72.2, R73.2
- net at C76.1 (K), L22.1, R86.1: now also CR8.1 (K), R70.2
Changed lines of the file:
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@@
   (junction (at 165.1 34.29) (diameter 0) (color 0 0 0 0)
   )
+  (junction (at 50.8 34.29) (diameter 0) (color 0 0 0 0)
+  )
   (junction (at 165.1 50.8) (diameter 0) (color 0 0 0 0)
   )
@@
   (junction (at 127 63.5) (diameter 0) (color 0 0 0 0)
   )
+  (junction (at 50.8 74.93) (diameter 0) (color 0 0 0 0)
+  )
   (junction (at 139.7 41.91) (diameter 0) (color 0 0 0 0)
   )
@@
   (junction (at 59.69 134.62) (diameter 0) (color 0 0 0 0)
   )
+  (junction (at 72.39 74.93) (diameter 0) (color 0 0 0 0)
+  )
   (junction (at 85.09 83.82) (diameter 0) (color 0 0 0 0)
+  )
+  (junction (at 72.39 48.26) (diameter 0) (color 0 0 0 0)
   )
   (junction (at 139.7 104.14) (diameter 0) (color 0 0 0 0)
@@
     (stroke (width 0) (type default) (color 0 0 0 0))
   )
+  (wire (pts (xy 50.8 74.93) (xy 59.69 74.93))
+    (stroke (width 0) (type default) (color 0 0 0 0))
+  )
   (wire (pts (xy 25.4 26.67) (xy 25.4 35.56))
     (stroke (width 0) (type default) (color 0 0 0 0))
   )
-  (wire (pts (xy 59.69 48.26) (xy 77.47 48.26))
+  (wire (pts (xy 59.69 48.26) (xy 72.39 48.26))
     (stroke (width 0) (type default) (color 0 0 0 0))
   )
@@
     (stroke (width 0) (type default) (color 0 0 0 0))
   )
+  (wire (pts (xy 72.39 48.26) (xy 72.39 74.93))
+    (stroke (width 0) (type default) (color 0 0 0 0))
+  )
   (wire (pts (xy 104.14 121.92) (xy 72.39 121.92))
     (stroke (width 0) (type default) (color 0 0 0 0))
@@
     (stroke (width 0) (type default) (color 0 0 0 0))
   )
+  (wire (pts (xy 72.39 48.26) (xy 77.47 48.26))
+    (stroke (width 0) (type default) (color 0 0 0 0))
+  )
   (wire (pts (xy 46.99 83.82) (xy 46.99 82.55))
     (stroke (width 0) (type default) (color 0 0 0 0))
@@
     (stroke (width 0) (type default) (color 0 0 0 0))
   )
-  (wire (pts (xy 38.1 34.29) (xy 104.14 34.29))
+  (wire (pts (xy 38.1 34.29) (xy 50.8 34.29))
     (stroke (width 0) (type default) (color 0 0 0 0))
   )
@@
     (stroke (width 0) (type default) (color 0 0 0 0))
   )
-  (wire (pts (xy 40.64 74.93) (xy 59.69 74.93))
+  (wire (pts (xy 40.64 74.93) (xy 50.8 74.93))
     (stroke (width 0) (type default) (color 0 0 0 0))
   )
@@
     (stroke (width 0) (type default) (color 0 0 0 0))
   )
+  (wire (pts (xy 50.8 34.29) (xy 50.8 74.93))
+    (stroke (width 0) (type default) (color 0 0 0 0))
+  )
   (wire (pts (xy 177.8 83.82) (xy 177.8 134.62))
     (stroke (width 0) (type default) (color 0 0 0 0))
@@
   )
   (wire (pts (xy 139.7 38.1) (xy 139.7 41.91))
+    (stroke (width 0) (type default) (color 0 0 0 0))
+  )
+  (wire (pts (xy 50.8 34.29) (xy 104.14 34.29))
     (stroke (width 0) (type default) (color 0 0 0 0))
   )
@@
   )
   (text "Without modulator\nC76 is a 22pF non\npolarized capacitor"
-    (at 57.15 57.15 0)
-    (effects (font (size 1.27 1.27)) (justify right bottom))
+    (at 54.61 46.99 0)
+    (effects (font (size 1.27 1.27)) (justify left bottom))
   )
   (text "\nNTSC\nPAL\nNO MODULATOR" (at 33.02 191.77 180)
@@
   (symbol (lib_id "Device:D_Capacitance") (at 72.39 80.01 270) (unit 1)
     (in_bom yes) (on_board yes)
-    (property "Reference" "C?" (id 0) (at 73.66 77.47 90)
-      (effects (font (size 1.27 1.27)) (justify left))
-    )
+    (property "Reference" "CR8" (id 0) (at 73.66 77.47 90)
+      (effects (font (size 1.27 1.27)) (justify left))
+    )

Commit message: fixed some DRC errors
Parts:
- gave numbers to parts that had none: 2
Changed lines of the file:
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@@
   (symbol (lib_id "Device:C_Small") (at 85.09 88.9 0) (unit 1)
     (in_bom yes) (on_board yes)
-    (property "Reference" "C?" (id 0) (at 87.63 87.63 0)
+    (property "Reference" "C64" (id 0) (at 87.63 87.63 0)
       (effects (font (size 1.27 1.27)) (justify left))
     )
@@
   (symbol (lib_id "Device:Q_NPN_CBE") (at 114.3 48.26 0) (unit 1)
     (in_bom yes) (on_board yes)
-    (property "Reference" "Q?" (id 0) (at 119.38 46.99 0)
+    (property "Reference" "Q2" (id 0) (at 119.38 46.99 0)
       (effects (font (size 1.27 1.27)) (justify left))
     )

Commit message: fixed some DRC errors
Parts:
- renumbered Q2 to Q8
Changed lines of the file:
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@@
   (symbol (lib_id "Device:Q_NPN_CBE") (at 114.3 48.26 0) (unit 1)
     (in_bom yes) (on_board yes)
-    (property "Reference" "Q2" (id 0) (at 119.38 46.99 0)
+    (property "Reference" "Q8" (id 0) (at 119.38 46.99 0)
       (effects (font (size 1.27 1.27)) (justify left))
     )

Commit message: assigning footprints
Parts:
- C76: footprint (none) -> commons-passives_THT:Passive_THT_capacitor_W2.54mm_L12.70mm
- CR8: footprint (none) -> commons-passives_THT:Passive_THT_diode_W2.54mm_L12.70mm
Changed lines of the file:
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@@
       (effects (font (size 1.27 1.27)) (justify left))
     )
-    (property "Footprint" "" (id 2) (at 72.39 80.01 0)
+    (property "Footprint" "commons-passives_THT:Passive_THT_diode_W2.54mm_L12.70mm" (id 2) (at 72.39 80.01 0)
       (effects (font (size 1.27 1.27)) hide)
     )
@@
       (effects (font (size 1.27 1.27)) (justify left))
     )
-    (property "Footprint" "" (id 2) (at 59.69 54.61 0)
-      (effects (font (size 1.27 1.27)) hide)
-    )
+    (property "Footprint" "commons-passives_THT:Passive_THT_capacitor_W2.54mm_L12.70mm" (id 2) (at 59.69 54.61 0)
+      (effects (font (size 1.27 1.27)) hide)
+    )

Commit message: assign footprints of remaining Resistors
Parts:
- R109, R112, R113, R141, R67, R68, R69, R70, R72, R73, R84, R85, R86, R88, R94: footprint (none) -> commons-passives_THT:Passive_THT_resistor_W2.54mm_L12.70mm
Changed lines of the file:
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@@
       (effects (font (size 1.27 1.27)) (justify right))
     )
-    (property "Footprint" "" (id 2) (at 106.68 58.42 0)
+    (property "Footprint" "commons-passives_THT:Passive_THT_resistor_W2.54mm_L12.70mm" (id 2) (at 106.68 58.42 0)
       (effects (font (size 1.27 1.27)) hide)
     )
@@
       (effects (font (size 1.27 1.27)) (justify right))
     )
-    (property "Footprint" "" (id 2) (at 165.1 58.42 0)
+    (property "Footprint" "commons-passives_THT:Passive_THT_resistor_W2.54mm_L12.70mm" (id 2) (at 165.1 58.42 0)
       (effects (font (size 1.27 1.27)) hide)
     )
@@
       (effects (font (size 1.27 1.27)) (justify right))
     )
-    (property "Footprint" "" (id 2) (at 146.05 41.91 0)
+    (property "Footprint" "commons-passives_THT:Passive_THT_resistor_W2.54mm_L12.70mm" (id 2) (at 146.05 41.91 0)
       (effects (font (size 1.27 1.27)) hide)
     )
@@
       (effects (font (size 1.27 1.27)) (justify right))
     )
-    (property "Footprint" "" (id 2) (at 114.3 83.82 0)
+    (property "Footprint" "commons-passives_THT:Passive_THT_resistor_W2.54mm_L12.70mm" (id 2) (at 114.3 83.82 0)
       (effects (font (size 1.27 1.27)) hide)
     )
@@
       (effects (font (size 1.27 1.27)) (justify right))
     )
-    (property "Footprint" "" (id 2) (at 85.09 78.74 0)
+    (property "Footprint" "commons-passives_THT:Passive_THT_resistor_W2.54mm_L12.70mm" (id 2) (at 85.09 78.74 0)
       (effects (font (size 1.27 1.27)) hide)
     )
@@
       (effects (font (size 1.27 1.27)) (justify right))
     )
-    (property "Footprint" "" (id 2) (at 46.99 120.65 0)
+    (property "Footprint" "commons-passives_THT:Passive_THT_resistor_W2.54mm_L12.70mm" (id 2) (at 46.99 120.65 0)
       (effects (font (size 1.27 1.27)) hide)
     )
@@
       (effects (font (size 1.27 1.27)) (justify right))
     )
-    (property "Footprint" "" (id 2) (at 40.64 78.74 0)
+    (property "Footprint" "commons-passives_THT:Passive_THT_resistor_W2.54mm_L12.70mm" (id 2) (at 40.64 78.74 0)
       (effects (font (size 1.27 1.27)) hide)
     )
@@
       (effects (font (size 1.27 1.27)) (justify right))
     )
-    (property "Footprint" "" (id 2) (at 59.69 78.74 0)
+    (property "Footprint" "commons-passives_THT:Passive_THT_resistor_W2.54mm_L12.70mm" (id 2) (at 59.69 78.74 0)
       (effects (font (size 1.27 1.27)) hide)
     )
@@
       (effects (font (size 1.27 1.27)) (justify right))
     )
-    (property "Footprint" "" (id 2) (at 34.29 99.06 0)
+    (property "Footprint" "commons-passives_THT:Passive_THT_resistor_W2.54mm_L12.70mm" (id 2) (at 34.29 99.06 0)
       (effects (font (size 1.27 1.27)) hide)
     )
@@
       (effects (font (size 1.27 1.27)) (justify right))
     )
-    (property "Footprint" "" (id 2) (at 34.29 134.62 0)
+    (property "Footprint" "commons-passives_THT:Passive_THT_resistor_W2.54mm_L12.70mm" (id 2) (at 34.29 134.62 0)
       (effects (font (size 1.27 1.27)) hide)
     )
@@
       (effects (font (size 1.27 1.27)) (justify right))
     )
-    (property "Footprint" "" (id 2) (at 49.53 138.43 0)
+    (property "Footprint" "commons-passives_THT:Passive_THT_resistor_W2.54mm_L12.70mm" (id 2) (at 49.53 138.43 0)
       (effects (font (size 1.27 1.27)) hide)
     )
@@
       (effects (font (size 1.27 1.27)) (justify right))
     )
-    (property "Footprint" "" (id 2) (at 85.09 50.8 0)
+    (property "Footprint" "commons-passives_THT:Passive_THT_resistor_W2.54mm_L12.70mm" (id 2) (at 85.09 50.8 0)
       (effects (font (size 1.27 1.27)) hide)
     )
@@
       (effects (font (size 1.27 1.27)) (justify right))
     )
-    (property "Footprint" "" (id 2) (at 116.84 58.42 0)
+    (property "Footprint" "commons-passives_THT:Passive_THT_resistor_W2.54mm_L12.70mm" (id 2) (at 116.84 58.42 0)
       (effects (font (size 1.27 1.27)) hide)
     )
@@
       (effects (font (size 1.27 1.27)) (justify right))
     )
-    (property "Footprint" "" (id 2) (at 177.8 78.74 0)
+    (property "Footprint" "commons-passives_THT:Passive_THT_resistor_W2.54mm_L12.70mm" (id 2) (at 177.8 78.74 0)
       (effects (font (size 1.27 1.27)) hide)
     )
@@
       (effects (font (size 1.27 1.27)) (justify right))
     )
-    (property "Footprint" "" (id 2) (at 104.14 38.1 0)
-      (effects (font (size 1.27 1.27)) hide)
-    )
+    (property "Footprint" "commons-passives_THT:Passive_THT_resistor_W2.54mm_L12.70mm" (id 2) (at 104.14 38.1 0)
+      (effects (font (size 1.27 1.27)) hide)
+    )
