File: subsheet_300.kicad_sch (KiCad schematic)
At the start: 36 parts, among them Q11 2N3904, Q6 2N3904, Q7 2N3906, Q8 2N3904, Q9 2N3906, U41 74LS74 DUAL FLIP-FLOPS, Y2 see table, Y3 see table

Commit message: assigned footprint for all remaining standard passives
Parts:
- L19, L20, L22: footprint (none) -> commons-passives_THT:Passive_THT_inductor_W5.08mm_L15.24mm
- Q11, Q6, Q8: footprint (none) -> Package_TO_SOT_THT:TO-92L_Inline_Wide; symbol Device:Q_NPN_CBE -> Device:Q_NPN_EBC
- Q7, Q9: footprint (none) -> Package_TO_SOT_THT:TO-92L_Inline_Wide
- Y2, Y3: footprint (none) -> Crystal:Crystal_HC50_Horizontal
Connections:
- net 32MHZ: now also Q6.1 (E); no longer Q6.3 (E)
- net GND: now also Q11.1 (E); no longer Q11.3 (E)
- net at C63.1, C73.1, L19.1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: now also Q6.3 (C); no longer Q6.1 (C)
- net at C52.1, C63.2, L19.2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: now also Q8.3 (C); no longer Q8.1 (C)
- net at R141.1, R69.2: now also Q11.3 (C); no longer Q11.1 (C)
- net at C56.1, R84.2: now also Q8.1 (E); no longer Q8.3 (E)
Changed lines of the file:
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@@
       (effects (font (size 1.27 1.27)) (justify left))
     )
-    (property "Footprint" "" (id 2) (at 128.27 38.1 0)
+    (property "Footprint" "commons-passives_THT:Passive_THT_inductor_W5.08mm_L15.24mm" (id 2) (at 128.27 38.1 0)
       (effects (font (size 1.27 1.27)) hide)
     )
@@
       (effects (font (size 1.27 1.27)) (justify right))
     )
-    (property "Footprint" "" (id 2) (at 85.09 45.72 0)
+    (property "Footprint" "commons-passives_THT:Passive_THT_inductor_W5.08mm_L15.24mm" (id 2) (at 85.09 45.72 0)
       (effects (font (size 1.27 1.27)) hide)
     )
@@
       (effects (font (size 1.27 1.27)) (justify left))
     )
-    (property "Footprint" "" (id 2) (at 34.29 116.84 0)
+    (property "Footprint" "Crystal:Crystal_HC50_Horizontal" (id 2) (at 34.29 116.84 0)
       (effects (font (size 1.27 1.27)) hide)
     )
@@
       (effects (font (size 1.27 1.27)) (justify right))
     )
-    (property "Footprint" "" (id 2) (at 36.83 91.44 0)
+    (property "Footprint" "Package_TO_SOT_THT:TO-92L_Inline_Wide" (id 2) (at 36.83 91.44 0)
       (effects (font (size 1.27 1.27)) hide)
     )
@@
     (property "Reference" "Y2" (id 0) (at 99.06 45.72 0))
     (property "Value" "see table" (id 1) (at 99.06 50.8 0))
-    (property "Footprint" "" (id 2) (at 99.06 48.26 0)
+    (property "Footprint" "Crystal:Crystal_HC50_Horizontal" (id 2) (at 99.06 48.26 0)
       (effects (font (size 1.27 1.27)) hide)
     )
@@
     (pin "2")
   )
-  (symbol (lib_id "Device:Q_NPN_CBE") (at 175.26 139.7 0) (unit 1)
+  (symbol (lib_id "Device:Q_NPN_EBC") (at 175.26 139.7 0) (unit 1)
     (in_bom yes) (on_board yes)
     (property "Reference" "Q11" (id 0) (at 180.34 138.43 0)
@@
       (effects (font (size 1.27 1.27)) (justify left))
     )
-    (property "Footprint" "" (id 2) (at 180.34 137.16 0)
+    (property "Footprint" "Package_TO_SOT_THT:TO-92L_Inline_Wide" (id 2) (at 180.34 137.16 0)
       (effects (font (size 1.27 1.27)) hide)
     )
@@
     (pin "1")
   )
-  (symbol (lib_id "Device:Q_NPN_CBE") (at 162.56 41.91 0) (unit 1)
+  (symbol (lib_id "Device:Q_NPN_EBC") (at 162.56 41.91 0) (unit 1)
     (in_bom yes) (on_board yes)
     (property "Reference" "Q6" (id 0) (at 167.64 40.64 0)
@@
       (effects (font (size 1.27 1.27)) (justify left))
     )
-    (property "Footprint" "" (id 2) (at 167.64 39.37 0)
+    (property "Footprint" "Package_TO_SOT_THT:TO-92L_Inline_Wide" (id 2) (at 167.64 39.37 0)
       (effects (font (size 1.27 1.27)) hide)
     )
@@
       (effects (font (size 1.27 1.27)) (justify right))
     )
-    (property "Footprint" "" (id 2) (at 44.45 91.44 0)
+    (property "Footprint" "Package_TO_SOT_THT:TO-92L_Inline_Wide" (id 2) (at 44.45 91.44 0)
       (effects (font (size 1.27 1.27)) hide)
     )
@@
       (effects (font (size 1.27 1.27)) (justify left))
     )
-    (property "Footprint" "" (id 2) (at 38.1 30.48 0)
+    (property "Footprint" "commons-passives_THT:Passive_THT_inductor_W5.08mm_L15.24mm" (id 2) (at 38.1 30.48 0)
       (effects (font (size 1.27 1.27)) hide)
     )
@@
     (pin "2")
   )
-  (symbol (lib_id "Device:Q_NPN_CBE") (at 114.3 48.26 0) (unit 1)
+  (symbol (lib_id "Device:Q_NPN_EBC") (at 114.3 48.26 0) (unit 1)
     (in_bom yes) (on_board yes)
     (property "Reference" "Q8" (id 0) (at 119.38 46.99 0)
@@
       (effects (font (size 1.27 1.27)) (justify left))
     )
-    (property "Footprint" "" (id 2) (at 119.38 45.72 0)
-      (effects (font (size 1.27 1.27)) hide)
-    )
+    (property "Footprint" "Package_TO_SOT_THT:TO-92L_Inline_Wide" (id 2) (at 119.38 45.72 0)
+      (effects (font (size 1.27 1.27)) hide)
+    )

Commit message: Fixed 32Mhz clock/modulator clock circuit : mention C67, forgotten R140
Parts:
- added R140: 2K2, commons-passives_THT:Passive_THT_resistor_W2.54mm_L12.70mm, symbol Device:R_Small_US
Connections:
- net at U41.6 (~{1Q}): now also R140.1; no longer Q11.2 (B)
- new net: Q11.2 (B), R140.2
Other:
- note added: "C67"
- note added: "On the PCB, there is a C67 between the base and the emitter of Q8. I can't find it on the schematic and on the equivalent circuit in later models (STF, STe). Thus, I choose to discard it."
- moved on the sheet: C56, R84, R85

Commit message: pcb session : acsi port, floppy disc drive port, parts of 32Mhz clock and modulator clock -- 2023-08-16T08:43+02:00
Connections:
- net at Q8.2 (B), R68.1, R85.2: now also Y2.1; no longer Y2.2
- net at L22.2, R86.2: now also Y2.2; no longer Y2.1
Other:
- moved on the sheet: Y2
Changed lines of the file:
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@@
     (pin "2")
   )
-  (symbol (lib_id "Device:Crystal_Small") (at 99.06 48.26 0) (unit 1)
+  (symbol (lib_id "Device:Crystal_Small") (at 99.06 48.26 180) (unit 1)
     (in_bom yes) (on_board yes)
     (property "Reference" "Y2" (id 0) (at 99.06 45.72 0))

Commit message: pcb session : done positionning, but traces will not match -- 2023-08-16T16:57+02:00
Connections:
- net at Q9.1 (C), R112.2: now also Y3.1; no longer Y3.2
- net at Q7.2 (B), R94.1: now also Y3.2; no longer Y3.1
Other:
- moved on the sheet: Y3
Changed lines of the file:
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@@
     (pin "2")
   )
-  (symbol (lib_id "Device:Crystal_Small") (at 34.29 116.84 0) (unit 1)
+  (symbol (lib_id "Device:Crystal_Small") (at 34.29 116.84 180) (unit 1)
     (in_bom yes) (on_board yes)
     (property "Reference" "Y3" (id 0) (at 31.75 115.57 0)
+      (effects (font (size 1.27 1.27)) (justify left))
+    )
+    (property "Value" "see table" (id 1) (at 36.83 115.57 0)
       (effects (font (size 1.27 1.27)) (justify right))
     )
-    (property "Value" "see table" (id 1) (at 36.83 115.57 0)
-      (effects (font (size 1.27 1.27)) (justify left))
-    )
     (property "Footprint" "Crystal:Crystal_HC50_Horizontal" (id 2) (at 34.29 116.84 0)
