File: subsheet_103.kicad_sch (KiCad schematic)
At the start: 28 parts, among them J5 DB25 Parallel Port, Q1 2N3904, U19 YM2149, U40 QUAD 2-INPUT NOR GATES

Commit message: fixed : forgotten annotation of L74~L83 of the parallel port
Parts:
- gave numbers to parts that had none: 10
Changed lines of the file:
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@@
   (symbol (lib_id "Device:Filter_EMI_LCL") (at 101.6 233.68 0) (unit 1)
     (in_bom yes) (on_board yes)
-    (property "Reference" "L?" (id 0) (at 99.06 228.6 0)
+    (property "Reference" "L82" (id 0) (at 99.06 228.6 0)
       (effects (font (size 1.27 1.27)) (justify right))
     )
@@
   (symbol (lib_id "Device:Filter_EMI_LCL") (at 116.84 182.88 0) (unit 1)
     (in_bom yes) (on_board yes)
-    (property "Reference" "L?" (id 0) (at 114.3 177.8 0)
+    (property "Reference" "L77" (id 0) (at 114.3 177.8 0)
       (effects (font (size 1.27 1.27)) (justify right))
     )
@@
   (symbol (lib_id "Device:Filter_EMI_LCL") (at 101.6 152.4 0) (unit 1)
     (in_bom yes) (on_board yes)
-    (property "Reference" "L?" (id 0) (at 99.06 147.32 0)
+    (property "Reference" "L74" (id 0) (at 99.06 147.32 0)
       (effects (font (size 1.27 1.27)) (justify right))
     )
@@
   (symbol (lib_id "Device:Filter_EMI_LCL") (at 101.6 172.72 0) (unit 1)
     (in_bom yes) (on_board yes)
-    (property "Reference" "L?" (id 0) (at 99.06 167.64 0)
+    (property "Reference" "L76" (id 0) (at 99.06 167.64 0)
       (effects (font (size 1.27 1.27)) (justify right))
     )
@@
   (symbol (lib_id "Device:Filter_EMI_LCL") (at 101.6 213.36 0) (unit 1)
     (in_bom yes) (on_board yes)
-    (property "Reference" "L?" (id 0) (at 99.06 208.28 0)
+    (property "Reference" "L80" (id 0) (at 99.06 208.28 0)
       (effects (font (size 1.27 1.27)) (justify right))
     )
@@
   (symbol (lib_id "Device:Filter_EMI_LCL") (at 101.6 193.04 0) (unit 1)
     (in_bom yes) (on_board yes)
-    (property "Reference" "L?" (id 0) (at 99.06 187.96 0)
+    (property "Reference" "L78" (id 0) (at 99.06 187.96 0)
       (effects (font (size 1.27 1.27)) (justify right))
     )
@@
   (symbol (lib_id "Device:Filter_EMI_LCL") (at 116.84 243.84 0) (unit 1)
     (in_bom yes) (on_board yes)
-    (property "Reference" "L?" (id 0) (at 114.3 238.76 0)
+    (property "Reference" "L83" (id 0) (at 114.3 238.76 0)
       (effects (font (size 1.27 1.27)) (justify right))
     )
@@
   (symbol (lib_id "Device:Filter_EMI_LCL") (at 116.84 203.2 0) (unit 1)
     (in_bom yes) (on_board yes)
-    (property "Reference" "L?" (id 0) (at 114.3 198.12 0)
+    (property "Reference" "L79" (id 0) (at 114.3 198.12 0)
       (effects (font (size 1.27 1.27)) (justify right))
     )
@@
   (symbol (lib_id "Device:Filter_EMI_LCL") (at 116.84 162.56 0) (unit 1)
     (in_bom yes) (on_board yes)
-    (property "Reference" "L?" (id 0) (at 114.3 157.48 0)
+    (property "Reference" "L75" (id 0) (at 114.3 157.48 0)
       (effects (font (size 1.27 1.27)) (justify right))
     )
@@
   (symbol (lib_id "Device:Filter_EMI_LCL") (at 116.84 223.52 0) (unit 1)
     (in_bom yes) (on_board yes)
-    (property "Reference" "L?" (id 0) (at 114.3 218.44 0)
-      (effects (font (size 1.27 1.27)) (justify right))
-    )
+    (property "Reference" "L81" (id 0) (at 114.3 218.44 0)
+      (effects (font (size 1.27 1.27)) (justify right))
+    )

Commit message: fixed some DRC errors
Connections:
- no-connect marks 6 -> 10
Changed lines of the file:
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@@
   (no_connect (at 170.18 215.9))
   (no_connect (at 119.38 99.06))
+  (no_connect (at 170.18 182.88))
+  (no_connect (at 170.18 187.96))
+  (no_connect (at 170.18 172.72))
+  (no_connect (at 170.18 177.8))
   (wire (pts (xy 83.82 241.3) (xy 76.2 241.3))
     (stroke (width 0) (type default) (color 0 0 0 0))
@@
   (symbol (lib_id "power:+5V") (at 76.2 241.3 0) (unit 1)
     (in_bom yes) (on_board yes)
-    (property "Reference" "#PWR?" (id 0) (at 76.2 245.11 0)
+    (property "Reference" "#PWR0300" (id 0) (at 76.2 245.11 0)
       (effects (font (size 1.27 1.27)) hide)
     )
@@
   (symbol (lib_id "power:GND") (at 134.62 53.34 0) (unit 1)
     (in_bom yes) (on_board yes)
-    (property "Reference" "#PWR?" (id 0) (at 134.62 59.69 0)
+    (property "Reference" "#PWR0287" (id 0) (at 134.62 59.69 0)
       (effects (font (size 1.27 1.27)) hide)
     )
@@
   (symbol (lib_id "power:GND") (at 74.93 63.5 0) (unit 1)
     (in_bom yes) (on_board yes)
-    (property "Reference" "#PWR?" (id 0) (at 74.93 69.85 0)
+    (property "Reference" "#PWR0284" (id 0) (at 74.93 69.85 0)
       (effects (font (size 1.27 1.27)) hide)
     )
@@
   (symbol (lib_id "power:GND") (at 149.86 53.34 0) (unit 1)
     (in_bom yes) (on_board yes)
-    (property "Reference" "#PWR?" (id 0) (at 149.86 59.69 0)
+    (property "Reference" "#PWR0293" (id 0) (at 149.86 59.69 0)
       (effects (font (size 1.27 1.27)) hide)
     )
@@
   (symbol (lib_id "power:GND") (at 161.29 207.01 0) (unit 1)
     (in_bom yes) (on_board yes)
-    (property "Reference" "#PWR?" (id 0) (at 161.29 213.36 0)
+    (property "Reference" "#PWR0307" (id 0) (at 161.29 213.36 0)
       (effects (font (size 1.27 1.27)) hide)
     )
@@
   (symbol (lib_id "power:GND") (at 116.84 185.42 0) (unit 1)
     (in_bom yes) (on_board yes)
-    (property "Reference" "#PWR?" (id 0) (at 116.84 191.77 0)
+    (property "Reference" "#PWR0313" (id 0) (at 116.84 191.77 0)
       (effects (font (size 1.27 1.27)) hide)
     )
@@
   (symbol (lib_id "power:GND") (at 167.64 240.03 0) (unit 1)
     (in_bom yes) (on_board yes)
-    (property "Reference" "#PWR?" (id 0) (at 167.64 246.38 0)
+    (property "Reference" "#PWR0306" (id 0) (at 167.64 246.38 0)
       (effects (font (size 1.27 1.27)) hide)
     )
@@
   (symbol (lib_id "power:+5V") (at 127 102.87 0) (unit 1)
     (in_bom yes) (on_board yes)
-    (property "Reference" "#PWR?" (id 0) (at 127 106.68 0)
+    (property "Reference" "#PWR0296" (id 0) (at 127 106.68 0)
       (effects (font (size 1.27 1.27)) hide)
     )
@@
   (symbol (lib_id "power:GND") (at 140.97 63.5 0) (unit 1)
     (in_bom yes) (on_board yes)
-    (property "Reference" "#PWR?" (id 0) (at 140.97 69.85 0)
+    (property "Reference" "#PWR0288" (id 0) (at 140.97 69.85 0)
       (effects (font (size 1.27 1.27)) hide)
     )
@@
   (symbol (lib_id "power:GND") (at 116.84 165.1 0) (unit 1)
     (in_bom yes) (on_board yes)
-    (property "Reference" "#PWR?" (id 0) (at 116.84 171.45 0)
+    (property "Reference" "#PWR0314" (id 0) (at 116.84 171.45 0)
       (effects (font (size 1.27 1.27)) hide)
     )
@@
   (symbol (lib_id "power:GND") (at 101.6 236.22 0) (unit 1)
     (in_bom yes) (on_board yes)
-    (property "Reference" "#PWR?" (id 0) (at 101.6 242.57 0)
+    (property "Reference" "#PWR0301" (id 0) (at 101.6 242.57 0)
       (effects (font (size 1.27 1.27)) hide)
     )
@@
   (symbol (lib_id "power:GND") (at 161.29 201.93 0) (unit 1)
     (in_bom yes) (on_board yes)
-    (property "Reference" "#PWR?" (id 0) (at 161.29 208.28 0)
+    (property "Reference" "#PWR0311" (id 0) (at 161.29 208.28 0)
       (effects (font (size 1.27 1.27)) hide)
     )
@@
   (symbol (lib_id "power:GND") (at 167.64 142.24 0) (unit 1)
     (in_bom yes) (on_board yes)
-    (property "Reference" "#PWR?" (id 0) (at 167.64 148.59 0)
+    (property "Reference" "#PWR0289" (id 0) (at 167.64 148.59 0)
       (effects (font (size 1.27 1.27)) hide)
     )
@@
   (symbol (lib_id "power:GND") (at 110.49 53.34 0) (unit 1)
     (in_bom yes) (on_board yes)
-    (property "Reference" "#PWR?" (id 0) (at 110.49 59.69 0)
+    (property "Reference" "#PWR0292" (id 0) (at 110.49 59.69 0)
       (effects (font (size 1.27 1.27)) hide)
     )
@@
   (symbol (lib_id "power:GND") (at 101.6 195.58 0) (unit 1)
     (in_bom yes) (on_board yes)
-    (property "Reference" "#PWR?" (id 0) (at 101.6 201.93 0)
+    (property "Reference" "#PWR0303" (id 0) (at 101.6 201.93 0)
       (effects (font (size 1.27 1.27)) hide)
     )
@@
   (symbol (lib_id "power:GND") (at 161.29 191.77 0) (unit 1)
     (in_bom yes) (on_board yes)
-    (property "Reference" "#PWR?" (id 0) (at 161.29 198.12 0)
+    (property "Reference" "#PWR0310" (id 0) (at 161.29 198.12 0)
       (effects (font (size 1.27 1.27)) hide)
     )
@@
   (symbol (lib_id "power:GND") (at 116.84 205.74 0) (unit 1)
     (in_bom yes) (on_board yes)
-    (property "Reference" "#PWR?" (id 0) (at 116.84 212.09 0)
+    (property "Reference" "#PWR0315" (id 0) (at 116.84 212.09 0)
       (effects (font (size 1.27 1.27)) hide)
     )
@@
   (symbol (lib_id "power:GND") (at 116.84 226.06 0) (unit 1)
     (in_bom yes) (on_board yes)
-    (property "Reference" "#PWR?" (id 0) (at 116.84 232.41 0)
+    (property "Reference" "#PWR0312" (id 0) (at 116.84 232.41 0)
       (effects (font (size 1.27 1.27)) hide)
     )
@@
   (symbol (lib_id "power:GND") (at 116.84 246.38 0) (unit 1)
     (in_bom yes) (on_board yes)
-    (property "Reference" "#PWR?" (id 0) (at 116.84 252.73 0)
+    (property "Reference" "#PWR0299" (id 0) (at 116.84 252.73 0)
       (effects (font (size 1.27 1.27)) hide)
     )
@@
   (symbol (lib_id "power:GND") (at 161.29 213.36 0) (unit 1)
     (in_bom yes) (on_board yes)
-    (property "Reference" "#PWR?" (id 0) (at 161.29 219.71 0)
+    (property "Reference" "#PWR0308" (id 0) (at 161.29 219.71 0)
       (effects (font (size 1.27 1.27)) hide)
     )
@@
   (symbol (lib_id "power:+5V") (at 115.57 22.86 0) (unit 1)
     (in_bom yes) (on_board yes)
-    (property "Reference" "#PWR?" (id 0) (at 115.57 26.67 0)
+    (property "Reference" "#PWR0295" (id 0) (at 115.57 26.67 0)
       (effects (font (size 1.27 1.27)) hide)
     )
@@
   (symbol (lib_id "power:GND") (at 101.6 175.26 0) (unit 1)
     (in_bom yes) (on_board yes)
-    (property "Reference" "#PWR?" (id 0) (at 101.6 181.61 0)
+    (property "Reference" "#PWR0304" (id 0) (at 101.6 181.61 0)
       (effects (font (size 1.27 1.27)) hide)
     )
@@
   (symbol (lib_id "power:+5V") (at 127 95.25 0) (unit 1)
     (in_bom yes) (on_board yes)
-    (property "Reference" "#PWR?" (id 0) (at 127 99.06 0)
+    (property "Reference" "#PWR0285" (id 0) (at 127 99.06 0)
       (effects (font (size 1.27 1.27)) hide)
     )
@@
   (symbol (lib_id "power:+5V") (at 123.19 63.5 0) (unit 1)
     (in_bom yes) (on_board yes)
-    (property "Reference" "#PWR?" (id 0) (at 123.19 67.31 0)
+    (property "Reference" "#PWR0286" (id 0) (at 123.19 67.31 0)
       (effects (font (size 1.27 1.27)) hide)
     )
@@
   (symbol (lib_id "power:GND") (at 181.61 115.57 0) (unit 1)
     (in_bom yes) (on_board yes)
-    (property "Reference" "#PWR?" (id 0) (at 181.61 121.92 0)
+    (property "Reference" "#PWR0298" (id 0) (at 181.61 121.92 0)
       (effects (font (size 1.27 1.27)) hide)
     )
@@
   (symbol (lib_id "power:GND") (at 129.54 142.24 0) (unit 1)
     (in_bom yes) (on_board yes)
-    (property "Reference" "#PWR?" (id 0) (at 129.54 148.59 0)
+    (property "Reference" "#PWR0290" (id 0) (at 129.54 148.59 0)
       (effects (font (size 1.27 1.27)) hide)
     )
@@
   (symbol (lib_id "power:GND") (at 101.6 215.9 0) (unit 1)
     (in_bom yes) (on_board yes)
-    (property "Reference" "#PWR?" (id 0) (at 101.6 222.25 0)
+    (property "Reference" "#PWR0302" (id 0) (at 101.6 222.25 0)
       (effects (font (size 1.27 1.27)) hide)
     )
@@
   (symbol (lib_id "power:GND") (at 101.6 154.94 0) (unit 1)
     (in_bom yes) (on_board yes)
-    (property "Reference" "#PWR?" (id 0) (at 101.6 161.29 0)
+    (property "Reference" "#PWR0305" (id 0) (at 101.6 161.29 0)
       (effects (font (size 1.27 1.27)) hide)
     )
@@
   (symbol (lib_id "power:GND") (at 144.78 104.14 0) (unit 1)
     (in_bom yes) (on_board yes)
-    (property "Reference" "#PWR?" (id 0) (at 144.78 110.49 0)
+    (property "Reference" "#PWR0297" (id 0) (at 144.78 110.49 0)
       (effects (font (size 1.27 1.27)) hide)
     )
@@
   (symbol (lib_id "power:GND") (at 161.29 196.85 0) (unit 1)
     (in_bom yes) (on_board yes)
-    (property "Reference" "#PWR?" (id 0) (at 161.29 203.2 0)
+    (property "Reference" "#PWR0309" (id 0) (at 161.29 203.2 0)
       (effects (font (size 1.27 1.27)) hide)
     )
@@
   (symbol (lib_id "power:GND") (at 170.18 22.86 0) (unit 1)
     (in_bom yes) (on_board yes)
-    (property "Reference" "#PWR?" (id 0) (at 170.18 29.21 0)
+    (property "Reference" "#PWR0294" (id 0) (at 170.18 29.21 0)
       (effects (font (size 1.27 1.27)) hide)
     )
@@
   (symbol (lib_id "power:+5V") (at 163.83 115.57 0) (unit 1)
     (in_bom yes) (on_board yes)
-    (property "Reference" "#PWR?" (id 0) (at 163.83 119.38 0)
-      (effects (font (size 1.27 1.27)) hide)
-    )
+    (property "Reference" "#PWR0291" (id 0) (at 163.83 119.38 0)
+      (effects (font (size 1.27 1.27)) hide)
+    )

Commit message: fixed some DRC errors
Parts:
- gave numbers to parts that had none: 1
- renumbered C32 to C60
Changed lines of the file:
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@@
   (symbol (lib_id "Device:C_Small") (at 173.99 115.57 90) (unit 1)
     (in_bom yes) (on_board yes)
-    (property "Reference" "C32" (id 0) (at 172.72 114.3 90)
+    (property "Reference" "C60" (id 0) (at 172.72 114.3 90)
       (effects (font (size 1.27 1.27)) (justify left))
     )
@@
   (symbol (lib_id "Device:C_Small") (at 133.35 63.5 90) (unit 1)
     (in_bom yes) (on_board yes)
-    (property "Reference" "C?" (id 0) (at 132.08 62.23 90)
-      (effects (font (size 1.27 1.27)) (justify left))
-    )
+    (property "Reference" "C32" (id 0) (at 132.08 62.23 90)
+      (effects (font (size 1.27 1.27)) (justify left))
+    )

Commit message: fixed symbols causing DRC errors, fixed renamed symbol 'FerriteBead_small'
Parts:
- L31: symbol Device:Ferrite_Bead_Small -> Device:FerriteBead_Small
Changed lines of the file:
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@@
     (pin "2")
   )
-  (symbol (lib_id "Device:Ferrite_Bead_Small") (at 123.19 22.86 270) (unit 1)
+  (symbol (lib_id "Device:FerriteBead_Small") (at 123.19 22.86 270) (unit 1)
     (in_bom yes) (on_board yes)
     (property "Reference" "L31" (id 0) (at 118.11 21.59 90)

Commit message: assign footprints of remaining Resistors
Parts:
- R107, R111, R38, R39, R40, R41: footprint (none) -> commons-passives_THT:Passive_THT_resistor_W2.54mm_L12.70mm
Changed lines of the file:
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@@
       (effects (font (size 1.27 1.27)) (justify right))
     )
-    (property "Footprint" "" (id 2) (at 149.86 48.26 0)
+    (property "Footprint" "commons-passives_THT:Passive_THT_resistor_W2.54mm_L12.70mm" (id 2) (at 149.86 48.26 0)
       (effects (font (size 1.27 1.27)) hide)
     )
@@
       (effects (font (size 1.27 1.27)) (justify right))
     )
-    (property "Footprint" "" (id 2) (at 134.62 48.26 0)
+    (property "Footprint" "commons-passives_THT:Passive_THT_resistor_W2.54mm_L12.70mm" (id 2) (at 134.62 48.26 0)
       (effects (font (size 1.27 1.27)) hide)
     )
@@
       (effects (font (size 1.27 1.27)) (justify right))
     )
-    (property "Footprint" "" (id 2) (at 130.81 27.94 0)
+    (property "Footprint" "commons-passives_THT:Passive_THT_resistor_W2.54mm_L12.70mm" (id 2) (at 130.81 27.94 0)
       (effects (font (size 1.27 1.27)) hide)
     )
@@
       (effects (font (size 1.27 1.27)) (justify right))
     )
-    (property "Footprint" "" (id 2) (at 86.36 241.3 0)
+    (property "Footprint" "commons-passives_THT:Passive_THT_resistor_W2.54mm_L12.70mm" (id 2) (at 86.36 241.3 0)
       (effects (font (size 1.27 1.27)) hide)
     )
@@
       (effects (font (size 1.27 1.27)) (justify right))
     )
-    (property "Footprint" "" (id 2) (at 149.86 27.94 0)
+    (property "Footprint" "commons-passives_THT:Passive_THT_resistor_W2.54mm_L12.70mm" (id 2) (at 149.86 27.94 0)
       (effects (font (size 1.27 1.27)) hide)
     )
@@
       (effects (font (size 1.27 1.27)) (justify right))
     )
-    (property "Footprint" "" (id 2) (at 110.49 45.72 0)
-      (effects (font (size 1.27 1.27)) hide)
-    )
+    (property "Footprint" "commons-passives_THT:Passive_THT_resistor_W2.54mm_L12.70mm" (id 2) (at 110.49 45.72 0)
+      (effects (font (size 1.27 1.27)) hide)
+    )

Commit message: assigned footprint for all remaining standard passives
Parts:
- C31, C34: footprint commons-passives_THT:Passive_THT_capacitor_mlcc_W2.54mm_L12.70mm -> Capacitor_THT:C_Radial_D6.3mm_H11.0mm_P2.50mm
- C33: footprint (none) -> Capacitor_THT:CP_Radial_D6.3mm_P2.50mm
- L74, L75, L76, L77, L78, L79, L80, L81, L82, L83: footprint (none) -> commons-passives_THT:Passive_THT_EMI_filter_W5.08mm_L7.62mm
- Q1: footprint (none) -> Package_TO_SOT_THT:TO-92L_Inline_Wide; symbol Device:Q_NPN_CBE -> Device:Q_NPN_EBC
Connections:
- net at Q1.1 (E): now also C33.1, R41.2; no longer R40.1
- new net: Q1.3 (C), R40.1
Changed lines of the file:
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@@
       (effects (font (size 1.27 1.27)) (justify right))
     )
-    (property "Footprint" "commons-passives_THT:Passive_THT_capacitor_mlcc_W2.54mm_L12.70mm" (id 2) (at 121.92 38.1 0)
+    (property "Footprint" "Capacitor_THT:C_Radial_D6.3mm_H11.0mm_P2.50mm" (id 2) (at 121.92 38.1 0)
       (effects (font (size 1.27 1.27)) hide)
     )
@@
     (pin "2")
   )
-  (symbol (lib_id "Device:Q_NPN_CBE") (at 147.32 38.1 0) (unit 1)
+  (symbol (lib_id "Device:Q_NPN_EBC") (at 147.32 38.1 0) (unit 1)
     (in_bom yes) (on_board yes)
     (property "Reference" "Q1" (id 0) (at 152.4 36.83 0)
@@
       (effects (font (size 1.27 1.27)) (justify left))
     )
-    (property "Footprint" "" (id 2) (at 152.4 35.56 0)
+    (property "Footprint" "Package_TO_SOT_THT:TO-92L_Inline_Wide" (id 2) (at 152.4 35.56 0)
       (effects (font (size 1.27 1.27)) hide)
     )
@@
       (effects (font (size 1.27 1.27)) (justify left))
     )
-    (property "Footprint" "" (id 2) (at 101.6 233.68 90)
+    (property "Footprint" "commons-passives_THT:Passive_THT_EMI_filter_W5.08mm_L7.62mm" (id 2) (at 101.6 233.68 90)
       (effects (font (size 1.27 1.27)) hide)
     )
@@
       (effects (font (size 1.27 1.27)) (justify left))
     )
-    (property "Footprint" "" (id 2) (at 116.84 182.88 90)
+    (property "Footprint" "commons-passives_THT:Passive_THT_EMI_filter_W5.08mm_L7.62mm" (id 2) (at 116.84 182.88 90)
       (effects (font (size 1.27 1.27)) hide)
     )
@@
       (effects (font (size 1.27 1.27)) (justify left))
     )
-    (property "Footprint" "" (id 2) (at 101.6 152.4 90)
+    (property "Footprint" "commons-passives_THT:Passive_THT_EMI_filter_W5.08mm_L7.62mm" (id 2) (at 101.6 152.4 90)
       (effects (font (size 1.27 1.27)) hide)
     )
@@
       (effects (font (size 1.27 1.27)) (justify left))
     )
-    (property "Footprint" "" (id 2) (at 101.6 172.72 90)
+    (property "Footprint" "commons-passives_THT:Passive_THT_EMI_filter_W5.08mm_L7.62mm" (id 2) (at 101.6 172.72 90)
       (effects (font (size 1.27 1.27)) hide)
     )
@@
       (effects (font (size 1.27 1.27)) (justify right))
     )
-    (property "Footprint" "" (id 2) (at 163.83 44.45 0)
+    (property "Footprint" "Capacitor_THT:CP_Radial_D6.3mm_P2.50mm" (id 2) (at 163.83 44.45 0)
       (effects (font (size 1.27 1.27)) hide)
     )
@@
       (effects (font (size 1.27 1.27)) (justify left))
     )
-    (property "Footprint" "" (id 2) (at 101.6 213.36 90)
+    (property "Footprint" "commons-passives_THT:Passive_THT_EMI_filter_W5.08mm_L7.62mm" (id 2) (at 101.6 213.36 90)
       (effects (font (size 1.27 1.27)) hide)
     )
@@
       (effects (font (size 1.27 1.27)) (justify left))
     )
-    (property "Footprint" "" (id 2) (at 101.6 193.04 90)
+    (property "Footprint" "commons-passives_THT:Passive_THT_EMI_filter_W5.08mm_L7.62mm" (id 2) (at 101.6 193.04 90)
       (effects (font (size 1.27 1.27)) hide)
     )
@@
       (effects (font (size 1.27 1.27)) (justify right))
     )
-    (property "Footprint" "commons-passives_THT:Passive_THT_capacitor_mlcc_W2.54mm_L12.70mm" (id 2) (at 54.61 38.1 0)
+    (property "Footprint" "Capacitor_THT:C_Radial_D6.3mm_H11.0mm_P2.50mm" (id 2) (at 54.61 38.1 0)
       (effects (font (size 1.27 1.27)) hide)
     )
@@
       (effects (font (size 1.27 1.27)) (justify left))
     )
-    (property "Footprint" "" (id 2) (at 116.84 243.84 90)
+    (property "Footprint" "commons-passives_THT:Passive_THT_EMI_filter_W5.08mm_L7.62mm" (id 2) (at 116.84 243.84 90)
       (effects (font (size 1.27 1.27)) hide)
     )
@@
       (effects (font (size 1.27 1.27)) (justify left))
     )
-    (property "Footprint" "" (id 2) (at 116.84 203.2 90)
+    (property "Footprint" "commons-passives_THT:Passive_THT_EMI_filter_W5.08mm_L7.62mm" (id 2) (at 116.84 203.2 90)
       (effects (font (size 1.27 1.27)) hide)
     )
@@
       (effects (font (size 1.27 1.27)) (justify left))
     )
-    (property "Footprint" "" (id 2) (at 116.84 162.56 90)
+    (property "Footprint" "commons-passives_THT:Passive_THT_EMI_filter_W5.08mm_L7.62mm" (id 2) (at 116.84 162.56 90)
       (effects (font (size 1.27 1.27)) hide)
     )
@@
       (effects (font (size 1.27 1.27)) (justify left))
     )
-    (property "Footprint" "" (id 2) (at 116.84 223.52 90)
-      (effects (font (size 1.27 1.27)) hide)
-    )
+    (property "Footprint" "commons-passives_THT:Passive_THT_EMI_filter_W5.08mm_L7.62mm" (id 2) (at 116.84 223.52 90)
+      (effects (font (size 1.27 1.27)) hide)
+    )
