File: subsheet_103.kicad_sch (KiCad schematic)
At the start: 28 parts, among them J5 DB25 Parallel Port, Q1 2N3904, U19 YM2149, U40 QUAD 2-INPUT NOR GATES

Commit message: assign dsub footprints and midi ports
Parts:
- J5: footprint (none) -> Connector_Dsub:DSUB-25_Female_Horizontal_P2.77x2.84mm_EdgePinOffset4.94mm_Housed_MountingHolesOffset7.48mm
Changed lines of the file:
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@@
     (property "Reference" "J5" (id 0) (at 177.8 163.83 0))
     (property "Value" "DB25 Parallel Port" (id 1) (at 177.8 165.735 0))
-    (property "Footprint" "" (id 2) (at 177.8 200.66 0)
+    (property "Footprint" "Connector_Dsub:DSUB-25_Female_Horizontal_P2.77x2.84mm_EdgePinOffset4.94mm_Housed_MountingHolesOffset7.48mm" (id 2) (at 177.8 200.66 0)
       (effects (font (size 1.27 1.27)) hide)
     )
