File: subsheet_204.kicad_sch (KiCad schematic)
At the start: 3 parts, among them U12 ST_GLUE_PHY

Commit message: Fixes U12 -- #48 and #49 are wired to DATA[8] and DATA[9] respectively
Connections:
- net D0 renamed D8
- net D1 renamed D9
Changed lines of the file:
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@@
     (effects (font (size 1.27 1.27)) (justify right bottom))
   )
-  (label "D0" (at 148.59 123.19 0) (fields_autoplaced)
+  (label "D8" (at 148.59 123.19 0) (fields_autoplaced)
     (effects (font (size 1.27 1.27)) (justify left bottom))
   )
@@
     (effects (font (size 1.27 1.27)) (justify left bottom))
   )
-  (label "D1" (at 148.59 120.65 0) (fields_autoplaced)
+  (label "D9" (at 148.59 120.65 0) (fields_autoplaced)
     (effects (font (size 1.27 1.27)) (justify left bottom))
   )
